File: Eagle Projects/SolarForce Prototypes/CAN_ProtoBoard_home.brd (EAGLE design)
At the start: 50 x 50 mm, 41 parts, among them Q1 16MHz, U1 MCP2551

Commit message: Used wrong package for MCP2515.. SO not TSSOP!! Changed and fixxed...
Parts:
- U$1: device RobThePyro:TSSOP20 -> RobThePyro:SO-18W
- moved CLKOUT 4.05 mm to (24.4, 22.5)
- moved RX1BF 1.79 mm to (11.7, 7.30)
- moved RX0BF 1.79 mm to (14.2, 7.30)
- moved U$1 1.25 mm to (19.2, 14.7), turned to 180 degrees
- moved R5 0.86 mm to (26.9, 13.7)
- moved C4 0.42 mm to (26.5, 9.53)
Connections:
- net +5V: now also U$1.18; no longer U$1.20
- net CS: now also U$1.16; no longer U$1.18
- net GND: now also U$1.9; no longer U$1.10
- net INT: now also U$1.12; no longer U$1.13
- net N$1: now also U$1.8; no longer U$1.9
- net N$2: now also U$1.7; no longer U$1.8
- net N$5: now also U$1.17; no longer U$1.19
- net RX0BF: now also U$1.11; no longer U$1.12
- net RX1BF: now also U$1.10; no longer U$1.11
- net SCK: now also U$1.13; no longer U$1.14
- net SI: now also U$1.14; no longer U$1.16
- net SO: now also U$1.15; no longer U$1.17
- net TX2RTS: now also U$1.6; no longer U$1.7
Routing:
- net N$21: track 0.00 -> 6.00 mm
- net N$20: track 0.00 -> 6.00 mm
- net N$19: track 0.00 -> 6.00 mm
- net N$18: track 0.00 -> 6.00 mm
- net INT: track 23.7 -> 19.3 mm
- net N$17: track 10.0 -> 6.00 mm
- net N$15: track 10.0 -> 6.00 mm
- net N$14: track 10.0 -> 6.00 mm
- net N$13: track 10.0 -> 6.00 mm
- net +5V: track 122.4 -> 119.7 mm
- net SCK: track 9.04 -> 6.54 mm
- net CLKOUT: track 2.27 -> 4.75 mm
- net CS: track 10.6 -> 8.14 mm
- net N$1: track 11.0 -> 8.75 mm
- net RX1BF: track 5.85 -> 3.61 mm
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