File: Eagle Projects/SolarForce Prototypes/CAN_ProtoBoard_Pro_Mini.brd (EAGLE design)
At the start: 50 x 50 mm, 45 parts, among them Q1 16MHz, U1 MCP2551

Commit message: Working on protopanels
Parts:
- removed !INT, CLKOUT, RX, RX0BF, RX1BF, TX, TX0RTS, TX1RTS, TX2RTS, VBAT, VREF: (no value), pinhead:1X01
- removed C11: 100uF, resistor:PANASONIC_D
- removed C6: 560pF, resistor:C0805K
- removed DB9M: (no value), SparkFun-Connectors:DB9_MALE
- removed IO: (no value), pinhead:1X10
- removed JLINE, KLINE: (no value), pinhead:1X03
- removed R8, R9: 100E, resistor:R0805
- removed SJ1: Term, SparkFun-Retired:SJ_2S-TRACE
- removed U1: MCP2551, SparkFun-DigitalIC:SO08
- added JP5, JP8: (no value), pinhead:1X02
- added JP6: (no value), pinhead:1X12
- added JP7: AVR_SPI_PRG_6PTH, SparkFun-Connectors:2X3
- added Q2: (no value), crystal:HC49UP
- added U2: MCP2551PDIP, RobThePyro:DIL08
- C5: value 560pF -> (none); device resistor:C0805K -> resistor:E5-8,5
- JP4: device pinhead:1X02 -> pinhead:1X12
- LED1, LED2, LED3, LED4: device led:CHIPLED_0805 -> led:LED3MM
- moved JP3 44.2 mm to (36.1, 15.7), turned to 270 degrees
- moved R7 34.6 mm to (6.83, 38.6), flipped to the bottom
- moved JP4 29.6 mm to (22.1, 2.03)
- moved CANSCREW 29.3 mm to (13.1, 44.5), turned to 180 degrees
- moved Q1 28.7 mm to (38.1, 44.4)
- moved C4 28.3 mm to (20.3, 37.1), flipped to the bottom, turned to 180 degrees
- moved CAN 28.2 mm to (8.66, 33.8), turned to 0 degrees
- moved C1 27.5 mm to (35.0, 48.5), flipped to the bottom, turned to 0 degrees
- moved C2 27.4 mm to (39.6, 48.5), flipped to the bottom, turned to 180 degrees
- moved JP1 25.4 mm to (22.1, 20.8)
- moved U$1 25.3 mm to (33.3, 35.7), flipped to the bottom, turned to 90 degrees
- moved R5 21.9 mm to (40.4, 30.9), flipped to the bottom
- moved R6 21.2 mm to (1.65, 27.8), flipped to the bottom, turned to 90 degrees
- moved R2 20.2 mm to (3.94, 27.8), flipped to the bottom, turned to 90 degrees
- moved LED3 17.3 mm to (27.7, 43.7), turned to 270 degrees
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Connections:
- removed net CLKOUT: CLKOUT.1, U$1.3
- removed net D10: JP1.12
- removed net D11: JP1.11
- removed net D12: JP1.10
- removed net D13: JP1.9
- removed net D2: JP2.5
- removed net J+: DB9M.7, JLINE.3
- removed net J-: DB9M.6, JLINE.2
- removed net K: DB9M.4, KLINE.3
- removed net L: DB9M.8, KLINE.2
- removed net N$10: U1.5, VREF.1
- removed net N$11: C5.2, R8.1
- removed net N$12: C6.2, R9.1
- removed net N$16: IO.3
- removed net RX0BF: RX0BF.1, U$1.11
- removed net RX1BF: RX1BF.1, U$1.10
- removed net TX0RTS: TX0RTS.1, U$1.4
- removed net TX1RTS: TX1RTS.1, U$1.5
- removed net TX2RTS: TX2RTS.1, U$1.6
- removed net VBAT: DB9M.9, VBAT.1
- removed net VCC: JP1.4
- new net @RST: JP2.3, JP4.3
- new net A6: JP3.2
- new net A7: JP3.1
- net +5V: now also C5.+, JP1.4, JP6.4, JP7.2, JP8.1, U2.3; no longer C11.+, IO.10, IO.2, U1.3
- net A0: now also JP6.8
- net A1: now also JP6.7
- net A2: now also JP6.6
- net A3: now also JP6.5
- net CANH: now also JP5.1, U2.7; no longer DB9M.3, R9.2, SJ1.1, U1.7
- net CANL: now also U2.6; no longer DB9M.5, R8.2, U1.6
- net CS: now also JP1.12, JP6.12; no longer IO.8
- net D3: now also JP4.6
- net D4: now also JP4.7
- net D5: now also JP4.8
- net D6: now also JP4.9
- net D7: now also JP4.10
- net D8: now also JP4.11
- net D9: now also JP4.12
- net GND: now also C5.-, JP3.3, JP4.4, JP6.2, JP7.6, JP8.2, LED1.K, U2.2; no longer C11.-, C5.1, C6.1, DB9M.2, IO.1, IO.9, JLINE.1, KLINE.1, LED1.C, U1.2
- net INT: now also JP2.5, JP4.5, LED4.K; no longer !INT.1, IO.4, LED4.C
- net N$1: now also Q2.2
- net N$2: now also Q2.1
- net N$8: now also U2.8; no longer U1.8
- net N$9: now also JP5.2; no longer SJ1.2
- net RAW: now also JP6.1
- net RST: now also JP6.3, JP7.5; no longer JP2.3
- net RXCAN: now also LED2.K, U2.4; no longer LED2.C, RX.1, U1.4
- net RXI: now also JP4.2
- net SCK: now also JP1.9, JP6.9, JP7.3; no longer IO.5
- net SI: now also JP1.11, JP6.11, JP7.4; no longer IO.6
- net SO: now also JP1.10, JP6.10, JP7.1; no longer IO.7
- net TXCAN: now also LED3.K, U2.1; no longer LED3.C, TX.1, U1.1
- net TXO: now also JP4.1
Routing:
- net INT: track 19.3 -> 90.6 mm
- net RST: track 0.00 -> 69.6 mm
- net GND: track 43.6 -> 94.3 mm, vias 5 -> 10
- net J-: track 31.0 -> 0.00 mm
- net CANL: track 67.4 -> 37.0 mm
- net CANH: track 55.2 -> 27.0 mm
- net SO: track 7.59 -> 35.6 mm
- net J+: track 27.5 -> 0.00 mm
- net SCK: track 6.54 -> 28.4 mm
- net +5V: track 119.7 -> 139.3 mm
- net L: track 19.1 -> 0.00 mm
- net SI: track 7.08 -> 23.1 mm
- net N$7: track 1.94 -> 15.4 mm
- net K: track 13.1 -> 0.00 mm
- net TX0RTS: track 12.1 -> 0.00 mm
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Other:
- board text removed: "5V"
- board text removed: "CAN BUS"
- board text removed: "CS"
- board text removed: "Demo Board"
- board text removed: "INT"
- board text removed: "J-"
- board text removed: "R Mawbey | UKZN | 2015"
- board text removed: "SCK"
- board text removed: "SI"
- board text removed: "SO"
