File: Eagle Projects/SolarForce Prototypes/CAN_ProtoBoard_Pro_Mini.sch (EAGLE design)
At the start: 45 parts, among them Q1 16MHz, U1 MCP2551

Commit message: Working on protopanels
Parts:
- removed !INT, CLKOUT, RX, RX0BF, RX1BF, TX, TX0RTS, TX1RTS, TX2RTS, VBAT, VREF: (no value), pinhead:PINHD-1X1
- removed C11: 100uF, resistor:CPOL-USD
- removed C6: 560pF, resistor:C-EUC0805K
- removed DB9M: (no value), SparkFun-Connectors:DB9MALE
- removed IO: (no value), pinhead:PINHD-1X10
- removed JLINE, KLINE: (no value), pinhead:PINHD-1X3
- removed R8, R9: 100E, resistor:R-US_R0805
- removed SJ1: Term, SparkFun-Retired:SOLDERJUMPERTRACE
- removed U1: MCP2551, SparkFun-DigitalIC:MCP2551
- added JP5, JP8: (no value), pinhead:PINHD-1X2
- added JP6: (no value), pinhead:PINHD-1X12
- added JP7: AVR_SPI_PRG_6PTH, SparkFun-Connectors:AVR_SPI_PRG_6PTH
- added Q2: (no value), crystal:CRYSTALHC49UP
- added U2: MCP2551PDIP, RobThePyro:MCP2551PDIP
- C5: value 560pF -> (none); device resistor:C-EUC0805K -> resistor:CPOL-USE5-8.5
- JP4: device pinhead:PINHD-1X2 -> pinhead:PINHD-1X12
- LED1, LED2, LED3, LED4: device led:LEDCHIPLED_0805 -> led:LED3MM
Connections:
- removed net CLKOUT: CLKOUT.1, U$1G$1.CLKOUT
- removed net D10: JP1.12
- removed net D11: JP1.11
- removed net D12: JP1.10
- removed net D13: JP1.9
- removed net D2: JP2.5
- removed net J+: DB9M.7, JLINE.3
- removed net J-: DB9M.6, JLINE.2
- removed net K: DB9M.4, KLINE.3
- removed net L: DB9M.8, KLINE.2
- removed net N$10: U1.VREF, VREF.1
- removed net N$11: C5.2, R8.1
- removed net N$12: C6.2, R9.1
- removed net N$16: IO.3
- removed net RX0BF: RX0BF.1, U$1G$1.!RX0BF
- removed net RX1BF: RX1BF.1, U$1G$1.!RX1BF
- removed net TX0RTS: TX0RTS.1, U$1G$1.!TX0RTS
- removed net TX1RTS: TX1RTS.1, U$1G$1.!TX1RTS
- removed net TX2RTS: TX2RTS.1, U$1G$1.!TX2RTS
- removed net VBAT: DB9M.9, VBAT.1
- removed net VCC: JP1.4
- new net @RST: JP2.3, JP4.3
- new net A6: JP3.2
- new net A7: JP3.1
- net +5V: now also C5.+, JP1.4, JP6.4, JP7.2, JP8.1, U2.VDD; no longer C11.+, IO.10, IO.2, U1.VDD
- net A0: now also JP6.8
- net A1: now also JP6.7
- net A2: now also JP6.6
- net A3: now also JP6.5
- net CANH: now also JP5.1, U2.CANH; no longer DB9M.3, R9.2, SJ1.1, U1.CANH
- net CANL: now also U2.CANL; no longer DB9M.5, R8.2, U1.CANL
- net CS: now also JP1.12, JP6.12; no longer IO.8
- net D3: now also JP4.6
- net D4: now also JP4.7
- net D5: now also JP4.8
- net D6: now also JP4.9
- net D7: now also JP4.10
- net D8: now also JP4.11
- net D9: now also JP4.12
- net GND: now also C5.-, JP3.3, JP4.4, JP6.2, JP7.6, JP8.2, U2.VSS; no longer C11.-, C5.1, C6.1, DB9M.2, IO.1, IO.9, JLINE.1, KLINE.1, U1.VSS
- net INT: now also JP2.5, JP4.5; no longer !INT.1, IO.4
- net N$1: now also Q2.2
- net N$2: now also Q2.1
- net N$8: now also U2.RS; no longer U1.RS
- net N$9: now also JP5.2; no longer SJ1.2
- net RAW: now also JP6.1
- net RST: now also JP6.3, JP7.5; no longer JP2.3
- net RXCAN: now also U2.RXD; no longer RX.1, U1.RXD
- net RXI: now also JP4.2
- net SCK: now also JP1.9, JP6.9, JP7.3; no longer IO.5
- net SI: now also JP1.11, JP6.11, JP7.4; no longer IO.6
- net SO: now also JP1.10, JP6.10, JP7.1; no longer IO.7
- net TXCAN: now also U2.TXD; no longer TX.1, U1.TXD
- net TXO: now also JP4.1
Other:
- moved on the sheet: JP2, JP3
