File: Eagle Projects/Ben/CAN Interface/CAN Interface.brd (EAGLE design)
At the start: 100 x 80 mm, 28 parts, among them Q1 16MHz, Q3 16MHz, Q4 16MHz, U1 ATMEGA328P_TQFP, U2 MCP2551

Commit message: Working on PCB's and Generic CAN interface
Parts:
- removed C5, C6: 100nF, resistor:C0805K
- removed JP1: AVRISP6, atmel-avr:HDR-75869-131
- removed JP2: CAN_Interface, pinhead:1X04
- removed JP3: GFX_LCD, adafruit:1X20
- removed Q3: 16MHz, crystal:HC49/S
- removed Q4: 16MHz, crystal:HC49UP
- removed R6, R7: 100k, resistor:R0805
- removed U2: MCP2551, SparkFun:SO08
- C1, C2: device resistor:C0805 -> resistor:C0805K
- C3, C4: value 22pF -> 100nF
- Q1: device special:QS -> crystal:HC49/S
- Q2: value (none) -> 16MHz; device SparkFun:SOT23 -> crystal:HC49UP
- R1: value 50k -> 1k
- R4, R5: value 1k -> 100k
- U1: value ATMEGA328P_TQFP -> MCP2551; device SparkFun-DigitalIC:TQFP32-08 -> SparkFun:SO08
- moved R2 62.0 mm to (35.3, 15.7), turned to 270 degrees
- moved C1 59.0 mm to (16.0, 24.1), turned to 180 degrees
- moved R1 54.4 mm to (32.8, 15.7), turned to 270 degrees
- moved Q1 53.8 mm to (19.3, 28.4), turned to 180 degrees
- moved Q2 51.4 mm to (19.3, 28.4), turned to 180 degrees
- moved C2 39.9 mm to (22.6, 24.1)
- moved R3 34.8 mm to (13.7, 19.6), turned to 90 degrees
- moved C4 31.6 mm to (30.0, 15.7), turned to 270 degrees
- moved C3 30.0 mm to (37.3, 19.6), turned to 0 degrees
- moved R4 29.7 mm to (31.2, 12.7), turned to 0 degrees
- moved U$1 25.1 mm to (22.6, 17.3)
- moved LED3 25.1 mm to (13.7, 15.0)
- moved LED1 25.1 mm to (30.7, 21.1)
- moved LED2 25.1 mm to (33.3, 21.1)
- moved Z1 25.1 mm to (35.3, 32.3)
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Connections:
- removed net LCD_CS: JP3.4, U1.12
- removed net LCD_PWM: R2.2, U1.13
- removed net N$2: C2.2, Q1.2, U1.8
- removed net N$3: C3.1, Q3.2, Q4.2, U$1.8
- removed net N$5: Q2.1, R2.1
- removed net N$6: C4.1, Q3.1, Q4.1, U$1.7
- removed net RST: JP1.5, R1.1, U1.29
- removed net SS: JP2.1, U1.14
- net +5V: now also C3.2, C4.2, R2.2, R4.1, U1.3; no longer C5.2, C6.2, JP1.2, JP3.17, JP3.19, JP3.2, R4.2, R5.2, R6.1, U1.18, U1.20, U1.4, U1.6, U2.3
- net CANH: now also U1.7; no longer U2.7
- net CANL: now also U1.6; no longer U2.6
- net CANRST: now also R4.2; no longer R6.2
- net CANSTBY: now also R5.1, U1.8; no longer R7.1, U2.8
- net GND: now also C1.2, C2.2, C3.1, C4.1, R5.2, U1.2; no longer C1.1, C2.1, C3.2, C4.2, C5.1, C6.1, JP1.6, JP3.1, JP3.15, Q2.2, R7.2, U1.21, U1.3, U1.5, U2.2
- net MISO: no longer JP1.1, JP2.3, U1.16
- net MOSI: no longer JP1.4, JP2.2, JP3.5, U1.15
- net N$1: now also C2.1, Q2.1, U$1.7; no longer C1.2, U1.7
- net N$4: now also C1.1, Q1.2, Q2.2, U$1.8; no longer JP3.20, Q2.3
- net N$7: now also R1.1; no longer R3.1
- net N$8: now also R2.1; no longer R4.1
- net N$9: now also R3.1; no longer R5.1
- net RXCAN: now also U1.4; no longer U2.4
- net SCK: no longer JP1.3, JP2.4, JP3.6, U1.17
- net TXCAN: now also U1.1; no longer U2.1
Routing:
- net N$4: track 0.00 -> 10.3 mm
- net N$3: track 10.3 -> 0.00 mm
- net N$1: track 0.00 -> 10.0 mm
- net N$6: track 10.0 -> 0.00 mm
- net SCK: track 0.00 -> 1.56 mm
- net MOSI: track 0.00 -> 1.56 mm
- net MISO: track 0.00 -> 1.56 mm
