File: Eagle Projects/Ben/Display Node/Display_Node.sch (EAGLE design)
At the start: 32 parts, among them Q1 16MHz, Q3 16MHz, Q4 16MHz, Q5 16MHz, U1 ATMEGA328P_TQFP, U2 MCP2551, X1 5566-6, X2 5566-6

Commit message: Moar Layout on display
Parts:
- removed Q2: (no value), SparkFun:TRANSISTOR_NPNSOT23
- added Q6, Q7: 2N7002, transistor-fet:2N7002
- added R8: 100E, resistor:R-US_R0805
- R2: value 1k -> 100E
Connections:
- new net N$11: Q6.S, U$3.SCK/E
- new net N$12: Q6.G, R8.2
- new net N$13: U1.PD3(INT1)
- new net N$16: U1.PD2(INT0)
- new net N$17: U1.PD0(RXD)
- new net N$18: U1.PD1(TXD)
- new net SCKCNTRL: R8.1, U1.PD6(AIN0)
- net GND: now also Q7.S; no longer Q2.E
- net N$4: now also Q7.D; no longer Q2.C
- net N$5: now also Q7.G; no longer Q2.B
- net SCK: now also Q6.D; no longer U$3.SCK/E
Other:
- moved on the sheet: R2
Changed lines of the file:
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@@
 <part name="GND1" library="supply1" deviceset="GND" device=""/>
 <part name="GND2" library="supply1" deviceset="GND" device=""/>
-<part name="Q2" library="SparkFun" deviceset="TRANSISTOR_NPN" device="SOT23"/>
 <part name="GND4" library="supply1" deviceset="GND" device=""/>
-<part name="R2" library="resistor" deviceset="R-US_" device="R0805" value="1k"/>
+<part name="R2" library="resistor" deviceset="R-US_" device="R0805" value="100E"/>
 <part name="JP1" library="atmel-avr" deviceset="AVR-ISP6-" device="75869-131" value="AVRISP6"/>
 <part name="GND6" library="supply1" deviceset="GND" device=""/>
@@
 <part name="JP2" library="pinhead" deviceset="PINHD-1X2" device=""/>
 <part name="Q5" library="crystal" deviceset="CRYSTAL" device="HC49UP" value="16MHz"/>
+<part name="Q6" library="transistor-fet" deviceset="2N7002*" device=""/>
+<part name="R8" library="resistor" deviceset="R-US_" device="R0805" value="100E"/>
+<part name="Q7" library="transistor-fet" deviceset="2N7002*" device=""/>
 </parts>
 <sheets>
@@
 <instance part="GND1" gate="1" x="-66.04" y="58.42"/>
 <instance part="GND2" gate="1" x="-50.8" y="33.02"/>
-<instance part="Q2" gate="G$1" x="93.98" y="48.26"/>
 <instance part="GND4" gate="1" x="96.52" y="38.1"/>
-<instance part="R2" gate="G$1" x="81.28" y="48.26" rot="R180"/>
+<instance part="R2" gate="G$1" x="81.28" y="45.72" rot="R180"/>
 <instance part="JP1" gate="G$1" x="73.66" y="0" rot="R90"/>
 <instance part="GND6" gate="1" x="83.82" y="10.16" rot="R90"/>
@@
 <instance part="JP2" gate="G$1" x="73.66" y="25.4"/>
 <instance part="Q5" gate="G$1" x="-48.26" y="68.58" rot="R90"/>
+<instance part="Q6" gate="G$1" x="83.82" y="73.66" rot="MR270"/>
+<instance part="R8" gate="G$1" x="86.36" y="86.36" rot="R270"/>
+<instance part="Q7" gate="G$1" x="96.52" y="48.26"/>
 </instances>
 <busses>
@@
 </segment>
 <segment>
-<pinref part="Q2" gate="G$1" pin="E"/>
 <pinref part="GND4" gate="1" pin="GND"/>
 <wire x1="96.52" y1="43.18" x2="96.52" y2="40.64" width="0.1524" layer="91"/>
+<pinref part="Q7" gate="G$1" pin="S"/>
 </segment>
 <segment>
@@
 <net name="N$4" class="0">
 <segment>
-<pinref part="Q2" gate="G$1" pin="C"/>
 <wire x1="106.68" y1="55.88" x2="96.52" y2="55.88" width="0.1524" layer="91"/>
 <wire x1="96.52" y1="55.88" x2="96.52" y2="53.34" width="0.1524" layer="91"/>
 <pinref part="U$3" gate="G$1" pin="K-"/>
+<pinref part="Q7" gate="G$1" pin="D"/>
 </segment>
 </net>
 <net name="N$5" class="0">
 <segment>
-<pinref part="Q2" gate="G$1" pin="B"/>
 <pinref part="R2" gate="G$1" pin="1"/>
-<wire x1="91.44" y1="48.26" x2="86.36" y2="48.26" width="0.1524" layer="91"/>
+<pinref part="Q7" gate="G$1" pin="G"/>
+<wire x1="86.36" y1="45.72" x2="91.44" y2="45.72" width="0.1524" layer="91"/>
 </segment>
 </net>
@@
 </segment>
 <segment>
-<pinref part="U$3" gate="G$1" pin="SCK/E"/>
-<wire x1="106.68" y1="73.66" x2="99.06" y2="73.66" width="0.1524" layer="91"/>
-<label x="91.44" y="73.66" size="1.778" layer="95"/>
+<pinref part="Q6" gate="G$1" pin="D"/>
+<wire x1="78.74" y1="73.66" x2="73.66" y2="73.66" width="0.1524" layer="91"/>
+<label x="68.58" y="73.66" size="1.778" layer="95"/>
 </segment>
 </net>
@@
 <segment>
 <pinref part="R2" gate="G$1" pin="2"/>
-<wire x1="76.2" y1="48.26" x2="71.12" y2="48.26" width="0.1524" layer="91"/>
-<label x="68.58" y="50.8" size="1.778" layer="95"/>
+<wire x1="76.2" y1="45.72" x2="71.12" y2="45.72" width="0.1524" layer="91"/>
+<label x="63.5" y="48.26" size="1.778" layer="95"/>
 </segment>
 </net>
@@
 <segment>
 <pinref part="U$3" gate="G$1" pin="!RST"/>
-<wire x1="106.68" y1="66.04" x2="91.44" y2="66.04" width="0.1524" layer="91"/>
-<label x="83.82" y="66.04" size="1.778" layer="95"/>
+<wire x1="106.68" y1="66.04" x2="101.6" y2="66.04" width="0.1524" layer="91"/>
+<label x="99.06" y="66.04" size="1.778" layer="95"/>
 </segment>
 </net>
@@
 </segment>
 </net>
+<net name="N$11" class="0">
+<segment>
+<pinref part="Q6" gate="G$1" pin="S"/>
+<pinref part="U$3" gate="G$1" pin="SCK/E"/>
+<wire x1="88.9" y1="73.66" x2="106.68" y2="73.66" width="0.1524" layer="91"/>
+</segment>
+</net>
+<net name="N$12" class="0">
+<segment>
+<pinref part="Q6" gate="G$1" pin="G"/>
+<pinref part="R8" gate="G$1" pin="2"/>
+<wire x1="86.36" y1="78.74" x2="86.36" y2="81.28" width="0.1524" layer="91"/>
+</segment>
+</net>
+<net name="SCKCNTRL" class="0">
+<segment>
+<pinref part="R8" gate="G$1" pin="1"/>
+<wire x1="86.36" y1="91.44" x2="86.36" y2="96.52" width="0.1524" layer="91"/>
+<label x="86.36" y="99.06" size="1.778" layer="95" rot="R90"/>
+</segment>
+<segment>
+<pinref part="U1" gate="U$1" pin="PD6(AIN0)"/>
+<wire x1="2.54" y1="58.42" x2="7.62" y2="58.42" width="0.1524" layer="91"/>
+<label x="10.16" y="58.42" size="1.778" layer="95"/>
+</segment>
+</net>
+<net name="N$13" class="0">
+<segment>
+<pinref part="U1" gate="U$1" pin="PD3(INT1)"/>
+<wire x1="2.54" y1="66.04" x2="7.62" y2="66.04" width="0.1524" layer="91"/>
+<label x="10.16" y="66.04" size="1.778" layer="95"/>
+</segment>
+</net>
+<net name="N$16" class="0">
+<segment>
+<pinref part="U1" gate="U$1" pin="PD2(INT0)"/>
+<wire x1="2.54" y1="68.58" x2="7.62" y2="68.58" width="0.1524" layer="91"/>
+<label x="10.16" y="68.58" size="1.778" layer="95"/>
+</segment>
+</net>
+<net name="N$17" class="0">
+<segment>
+<pinref part="U1" gate="U$1" pin="PD0(RXD)"/>
+<wire x1="2.54" y1="73.66" x2="7.62" y2="73.66" width="0.1524" layer="91"/>
+</segment>
+</net>
+<net name="N$18" class="0">
+<segment>
+<pinref part="U1" gate="U$1" pin="PD1(TXD)"/>
+<wire x1="2.54" y1="71.12" x2="7.62" y2="71.12" width="0.1524" layer="91"/>
+</segment>
+</net>

Commit message: Birds Tweeting. Shit. Bed Time..
Parts:
- added LED4, LED5: (no value), led:LEDCHIP-LED0805
- added R10, R9: 1k, resistor:R-US_R0805
- added S1: RESET, SparkFun:TAC_SWITCHSMD
- added X3: C-GRID-10-70553, con-molex:C-GRID-10-70553
- added X4: C-GRID-06-70553, con-molex:C-GRID-06-70553
Connections:
- removed net N$17: U1.PD0(RXD)
- removed net N$18: U1.PD1(TXD)
- new net A0: U1.PC4(ADC4/SDA), X3-5.S
- new net A1: U1.PC5(ADC5/SCL), X3-6.S
- new net BTN1: U1.PD2(INT0), X3-1.S
- new net BTN2: U1.PD3(INT1), X3-2.S
- new net BTN3: U1.PD4(XCK/T0), X3-3.S
- new net BTN4: U1.PD5(T1), X3-4.S
- new net CRUISE1: U1.PC0(ADC0), X4-1.S
- new net CRUISE2: U1.PC1(ADC1), X4-2.S
- new net CRUISE3: U1.PC2(ADC2), X4-3.S
- new net CRUISE4: U1.PC3(ADC3), X4-4.S
- new net LED1: LED4.C, U1.PD0(RXD), X3-7.S
- new net LED2: LED5.C, U1.PD1(TXD), X3-8.S
- new net N$23: X4-5.S
- new net N$24: X4-6.S
- net +5V: now also R10.1, R9.1, X3-9.S
- net GND: now also S1.3, S1.4, X3-10.S
- net N$13: now also LED4.A, R9.2; no longer U1.PD3(INT1)
- net N$16: now also LED5.A, R10.2; no longer U1.PD2(INT0)
- net RST: now also S1.1, S1.2
