File: Eagle Projects/Ben/Display Node/Display_Node.sch (EAGLE design)
At the start: 90 parts, among them Q1 16MHz, Q3 16MHz, Q4 16MHz, Q5 16MHz, Q6 2N7002, Q7 2N7002, U1 ATMEGA328P_TQFP, U2 MCP2551, X1 5566-6, X2 5566-6

Commit message: Board Rework
Parts:
- removed JP2: (no value), pinhead:PINHD-1X2
- removed LED4, LED5: (no value), led:LEDCHIP-LED0805
- removed LED6, LED7: (no value), led:LED5MM
- removed R10, R9: 1k, resistor:R-US_R0805
- added D1: (no value), diode:SCHOTTKY-DIODESMD
- added LED8: F50360, led:F50360
- added R23, R24, R25: 1k, resistor:R-US_R0805
- added SG1: F/CM12P, buzzer:F/CM12P
Connections:
- removed net LCD_RST: U$3.!RST
- removed net N$13: LED4.A, LED7.A, R9.2
- removed net N$16: LED5.A, LED6.A, R10.2
- removed net SCKCNTRL: R8.1, U1.PD6(AIN0)
- new net LED3: R25.2, U1.PC4(ADC4/SDA)
- new net N$30: SG1.2, U1.PD6(AIN0)
- new net N$31: LED8.RC, R23.1
- new net N$32: LED8.GC, R24.1
- new net N$33: LED8.BC, R25.1
- new net N$36: U1.PC5(ADC5/SCL)
- net +5V: now also D1.C, LED8.BA, LED8.GA, LED8.RA, SG1.1, U$3.!RST; no longer JP2.1, R10.1, R9.1
- net A0: now also U1.ADC6; no longer U1.PC4(ADC4/SDA)
- net A1: now also U1.ADC7; no longer U1.PC5(ADC5/SCL)
- net LCD_CS: now also R8.1
- net LED1: now also R23.2; no longer LED4.C, LED7.C
- net LED2: now also R24.2; no longer LED5.C, LED6.C
- net N$10: now also D1.A; no longer JP2.2

Commit message: Experimenting with ideas...
Parts:
- added C23, C24: 22pF, resistor:C-EUC0805
- added Q2: 16MHz, special:XTAL/S
- added Q8: 16MHz, crystal:CRYSTALHC49UP
- added R9: 50k, resistor:R-US_R0805
- added S6: RESET, SparkFun:TAC_SWITCHSMD
- added U3: ATMEGA328P_TQFP, SparkFun-DigitalIC:ATMEGA328P_TQFP
Connections:
- new net MISO2: U3.PB4(MISO)
- new net MISOU: U1.PD0(RXD), U3.PD0(RXD)
- new net MOSI2: U$3.MOSI/RW, U3.PB3(MOSI/OC2)
- new net MOSIU: U1.PD1(TXD), U3.PD1(TXD)
- new net N$34: C23.2, Q2.1, Q8.2, U3.PB6(XTAL1/TOSC1)
- new net N$35: C24.2, Q2.2, Q8.1, U3.PB7(XTAL2/TOSC2)
- new net RST1: R9.1, S6.1, S6.2
- new net SCK2: Q6.D, U3.PB5(SCK)
- new net SCKU: U1.PD4(XCK/T0), U3.PD4(XCK/T0)
- net +5V: now also R9.2
- net BTN3: no longer U1.PD4(XCK/T0)
- net GND: now also C23.1, C24.1, S6.3, S6.4
- net LCD_CS: now also U3.PD7(AIN1); no longer U1.PD7(AIN1)
- net LCD_PWM: now also U3.PB1(OC1A); no longer U1.PB1(OC1A)
- net LED1: no longer U1.PD0(RXD)
- net LED2: no longer U1.PD1(TXD)
- net MOSI: no longer U$3.MOSI/RW
- net SCK: no longer Q6.D
