File: Eagle Projects/Ben/Display Node/Display_Node.brd (EAGLE design)
At the start: 93 x 90 mm, 62 parts, among them Q1 16MHz, Q3 16MHz, Q4 16MHz, Q5 16MHz, Q6 2N7002, Q7 2N7002, U1 ATMEGA328P_TQFP, U2 MCP2551, X1 5566-6, X2 5566-6

Commit message: Working on boards and moar code...
Parts:
- added C11, C12, C13, C14, C15, C16, C17, C18, C19, C20, C21, C22: 10nF, resistor:C0805
- added R15, R16, R17, R18, R19, R20, R21, R22: 470E, resistor:R0805
- added U$12, U$13, U$14, U$15, U$16, U$17, U$18, U$19: DRTR5V0U1SO, RobThePyro:SOT23
Connections:
- new net N$22: R18.1, U$4.P$3
- new net N$23: R17.1, U$4.P$4
- new net N$24: R16.1, U$4.P$5
- new net N$25: R15.1, U$4.P$6
- new net N$26: R19.1, U$5.P$4
- new net N$27: R20.1, U$5.P$3
- new net N$28: R21.1, U$5.P$2
- new net N$29: R22.1, U$5.P$1
- net +5V: now also U$12.2, U$13.2, U$14.2, U$15.2, U$16.2, U$17.2, U$18.2, U$19.2
- net A0: now also C22.1, R22.2, U$19.1; no longer U$5.P$1
- net A1: now also C21.1, R21.2, U$18.1; no longer U$5.P$2
- net BTN1: now also C14.1
- net BTN2: now also C13.1
- net BTN3: now also C12.1
- net BTN4: now also C11.1
- net CRUISE1: now also C18.1, R18.2, U$15.1; no longer U$4.P$3
- net CRUISE2: now also C17.1, R17.2, U$14.1; no longer U$4.P$4
- net CRUISE3: now also C16.1, R16.2, U$13.1; no longer U$4.P$5
- net CRUISE4: now also C15.1, R15.2, U$12.1; no longer U$4.P$6
- net GND: now also C11.2, C12.2, C13.2, C14.2, C15.2, C16.2, C17.2, C18.2, C19.2, C20.2, C21.2, C22.2, U$12.3, U$13.3, U$14.3, U$15.3, U$16.3, U$17.3, U$18.3, U$19.3
- net LED1: now also C20.1, R20.2, U$17.1; no longer U$5.P$3
- net LED2: now also C19.1, R19.2, U$16.1; no longer U$5.P$4
Routing:
- net LED2: track 76.1 -> 2.67 mm
- net CRUISE4: track 27.7 -> 0.00 mm
- net BTN3: track 54.5 -> 71.8 mm, vias 0 -> 1
- net CRUISE2: track 29.7 -> 13.1 mm
- net CRUISE1: track 32.2 -> 16.0 mm
- net CRUISE3: track 27.8 -> 12.5 mm
- net GND: track 111.6 -> 121.0 mm
- net N$26: track 0.00 -> 4.47 mm
- net LED1: track 73.4 -> 69.9 mm
- net BTN4: track 94.6 -> 96.9 mm
- net BTN2: track 31.7 -> 32.9 mm
- net BTN1: track 26.4 -> 27.0 mm

Commit message: Display Node Done?
Parts:
- moved C17 66.3 mm to (65.0, 15.2)
- moved C15 65.4 mm to (65.1, 22.9)
- moved C18 61.5 mm to (67.3, 11.5)
- moved C22 46.7 mm to (67.0, 26.8), turned to 0 degrees
- moved C21 38.3 mm to (65.9, 30.4)
- moved C19 37.5 mm to (66.9, 38.6)
- moved C16 26.5 mm to (67.2, 19.2)
- moved C20 19.3 mm to (67.2, 34.5), turned to 0 degrees
- moved R18 9.08 mm to (78.7, 11.2)
- moved R17 7.54 mm to (78.7, 15.3)
- moved R16 5.76 mm to (78.8, 19.6)
- moved R2 5.65 mm to (62.3, 9.67)
- moved R15 4.15 mm to (78.8, 23.7)
- moved R21 2.95 mm to (79.6, 36.0), turned to 180 degrees
- moved R22 1.40 mm to (78.8, 32.6)
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Routing:
- net LED2: track 2.67 -> 104.8 mm
- net +5V: track 313.7 -> 366.2 mm, vias 4 -> 12
- net GND: track 121.0 -> 165.6 mm, vias 11 -> 19
- net LED1: track 69.9 -> 104.0 mm
- net CRUISE4: track 0.00 -> 24.9 mm
- net A0: track 11.6 -> 28.9 mm
- net A1: track 9.29 -> 26.3 mm
- net CRUISE2: track 13.1 -> 29.7 mm
- net BTN4: track 96.9 -> 80.7 mm
- net CRUISE1: track 16.0 -> 32.1 mm
- net CRUISE3: track 12.5 -> 25.9 mm
- net N$22: track 0.00 -> 11.3 mm
- net N$23: track 0.00 -> 9.06 mm
- net N$5: track 4.53 -> 12.4 mm
- net N$24: track 0.00 -> 7.41 mm
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