File: Eagle Projects/SolarEV_RxBoard/RxBrd.brd (EAGLE design)
At the start: 80 x 80.1 mm, 50 parts, among them U2 ATMEGA32U4-XUAU, X1 USBPTH, Y2 16MHz

Commit message: There is now a PCB for the Rx board. Comments and criticism welcome.
Parts:
- removed JP2: PhotovoltaicCell Connect, pinhead:1X02
- added X2: 5566-6, con-molex:5566-6
- JP1: value Anemometer Connect -> (none); device pinhead:1X02 -> jumper:JP1
- moved D6 128.0 mm to (65.8, 46.7), turned to 90 degrees
- moved D5 122.7 mm to (65.8, 40.9), turned to 90 degrees
- moved ON4 119.8 mm to (56.4, 62.0), turned to 180 degrees
- moved R2 115.5 mm to (52.8, 62.2), turned to 270 degrees
- moved JP3 112.1 mm to (64.3, 4.32)
- moved D3 106.1 mm to (63.0, 49.0), turned to 270 degrees
- moved R1 105.5 mm to (41.9, 15.7), turned to 90 degrees
- moved ON3 105.4 mm to (49.5, 54.4), turned to 90 degrees
- moved C4 105.0 mm to (46.0, 14.5)
- moved D4 104.1 mm to (53.3, 41.9), turned to 270 degrees
- moved S1 100.2 mm to (57.9, 49.3), turned to 270 degrees
- moved ON2 99.5 mm to (49.5, 56.4), turned to 90 degrees
- moved ON6 96.8 mm to (55.1, 4.32), turned to 180 degrees
- moved C6 96.0 mm to (38.6, 52.8)
- moved R9 95.3 mm to (59.7, 62.2), turned to 90 degrees
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Connections:
- removed net RF_TRANSCEIVER_CONNECTED_OK: ON4.C, U2.1
- new net N$13: ON4.C, U2.33
- net +5V: now also X2.2; no longer JP1.2
- net GND: now also X2.6; no longer JP2.2
- net N$1: now also U2.32, X2.5; no longer JP1.1, U2.25
- net N$4: now also X2.3; no longer JP2.1
- net RX_LED: now also U2.18
- net TX_LED: now also U2.19
Routing:
- net +5V: track 0.00 -> 259.0 mm, vias 0 -> 3
- net GND: track 0.00 -> 204.5 mm, vias 0 -> 6
- net VUSB: track 0.00 -> 88.6 mm, vias 0 -> 2
- net TX_LED: track 0.00 -> 51.1 mm
- net N$8: track 0.00 -> 50.1 mm
- net N$7: track 0.00 -> 48.6 mm
- net AVCC: track 0.00 -> 48.6 mm
- net N$5: track 0.00 -> 47.9 mm, vias 0 -> 2
- net RX_LED: track 0.00 -> 45.2 mm
- net N$1: track 0.00 -> 43.4 mm, vias 0 -> 1
- net N$4: track 0.00 -> 42.0 mm, vias 0 -> 1
- net XTAL2: track 0.00 -> 29.8 mm
- net XTAL1: track 0.00 -> 27.9 mm
- net N$10: track 0.00 -> 26.7 mm, vias 0 -> 1
- net N$13: track 0.00 -> 24.7 mm
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Other:
- board text added: "SS Patel 212513168 Support Vehicle Aggredator Board Electronic/Computer Engineering Design 3 UKZN 2015"
