File: Eagle Projects/SolarEV_RxBoard/RxBrd.sch (EAGLE design)
At the start: 50 parts, among them U2 ATMEGA32U4-XUAU, X1 USBPTH, Y2 16MHz

Commit message: There is now a PCB for the Rx board. Comments and criticism welcome.
Parts:
- removed JP2: PhotovoltaicCell Connect, pinhead:PINHD-1X2
- added X2: 5566-6, con-molex:5566-6
- JP1: value Anemometer Connect -> (none); device pinhead:PINHD-1X2 -> jumper:JP1E
Connections:
- removed net RF_TRANSCEIVER_CONNECTED_OK: ON4.C, U2.(INT6/AIN0)PE6
- new net N$13: ON4.C, U2.(#HWB)PE2
- net +5V: now also X2-2.S; no longer JP1.2
- net GND: now also X2-6.S; no longer JP2.2
- net N$1: now also U2.(ICP3/CLK0/OC4A)PC7, X2-5.S; no longer JP1.1, U2.(ICP1/ADC8)PD4
- net N$4: now also X2-3.S; no longer JP2.1
- net RX_LED: now also U2.(OC0B/SCL/INT0)PD0
- net TX_LED: now also U2.(SDA/INT1)PD1
Other:
- note added: "Photovolt"
Changed lines of the file:
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@@
 <?xml version="1.0" encoding="utf-8"?>
 <!DOCTYPE eagle SYSTEM "eagle.dtd">
-<eagle version="7.2.0">
+<eagle version="7.1.0">
 <drawing>
 <settings>
@@
 <part name="U$4" library="MyPOW" deviceset="+5V" device=""/>
 <part name="GND1" library="supply1" deviceset="GND" device=""/>
-<part name="JP1" library="pinhead" deviceset="PINHD-1X2" device="" value="Anemometer Connect"/>
 <part name="D3" library="diode" deviceset="MBR0540" device=""/>
 <part name="D4" library="diode" deviceset="MBR0540" device=""/>
 <part name="GND3" library="supply1" deviceset="GND" device=""/>
-<part name="JP2" library="pinhead" deviceset="PINHD-1X2" device="" value="PhotovoltaicCell Connect"/>
 <part name="U$2" library="MyPOW" deviceset="+5V" device=""/>
 <part name="D5" library="diode" deviceset="MBR0540" device=""/>
@@
 <part name="ON6" library="led" deviceset="LED" device="CHIPLED_0805" value="Yellow"/>
 <part name="X1" library="SparkFun" deviceset="USB" device="PTH"/>
+<part name="X2" library="con-molex" deviceset="5566-6" device=""/>
+<part name="JP1" library="jumper" deviceset="JP1E" device=""/>
 </parts>
 <sheets>
@@
 <text x="-165.1" y="-93.98" size="3.81" layer="94" ratio="10" rot="MR0">USB</text>
 <text x="142.24" y="-15.24" size="3.81" layer="94" ratio="10" rot="MR0">ATmega32U4</text>
+<text x="193.04" y="-27.94" size="1.778" layer="91">Photovolt</text>
 </plain>
 <instances>
@@
 <instance part="U$4" gate="G$1" x="71.12" y="-48.26"/>
 <instance part="GND1" gate="1" x="86.36" y="-101.6"/>
-<instance part="JP1" gate="G$1" x="205.74" y="-68.58" rot="R90"/>
 <instance part="D3" gate="G$1" x="195.58" y="-63.5" rot="R90"/>
 <instance part="D4" gate="G$1" x="195.58" y="-76.2" rot="R90"/>
 <instance part="GND3" gate="1" x="195.58" y="-86.36"/>
-<instance part="JP2" gate="G$1" x="205.74" y="-22.86" rot="R90"/>
 <instance part="U$2" gate="G$1" x="185.42" y="-10.16"/>
 <instance part="D5" gate="G$1" x="185.42" y="-17.78" rot="R90"/>
@@
 <instance part="ON6" gate="G$1" x="167.64" y="-66.04" rot="R270"/>
 <instance part="X1" gate="G$1" x="-152.4" y="-116.84" rot="R180"/>
+<instance part="X2" gate="-1" x="279.4" y="-58.42"/>
+<instance part="X2" gate="-2" x="208.28" y="-60.96"/>
+<instance part="X2" gate="-3" x="172.72" y="-22.86" rot="R90"/>
+<instance part="X2" gate="-4" x="279.4" y="-66.04"/>
+<instance part="X2" gate="-5" x="205.74" y="-71.12"/>
+<instance part="X2" gate="-6" x="182.88" y="-40.64" rot="R180"/>
+<instance part="JP1" gate="A" x="27.94" y="-30.48"/>
 </instances>
 <busses>
@@
 <wire x1="205.74" y1="-55.88" x2="205.74" y2="-50.8" width="0.1524" layer="91"/>
 <wire x1="205.74" y1="-50.8" x2="223.52" y2="-50.8" width="0.1524" layer="91"/>
-<pinref part="JP1" gate="G$1" pin="2"/>
-<wire x1="205.74" y1="-55.88" x2="205.74" y2="-71.12" width="0.1524" layer="91"/>
+<wire x1="205.74" y1="-55.88" x2="205.74" y2="-60.96" width="0.1524" layer="91"/>
 <junction x="205.74" y="-55.88"/>
 <junction x="223.52" y="-50.8"/>
@@
 <junction x="187.96" y="-55.88"/>
 <junction x="187.96" y="-63.5"/>
+<pinref part="X2" gate="-2" pin="S"/>
 </segment>
 <segment>
@@
 <pinref part="D6" gate="G$1" pin="A"/>
 <pinref part="GND5" gate="1" pin="GND"/>
-<wire x1="185.42" y1="-38.1" x2="185.42" y2="-43.18" width="0.1524" layer="91"/>
-<pinref part="JP2" gate="G$1" pin="2"/>
-<wire x1="205.74" y1="-25.4" x2="205.74" y2="-43.18" width="0.1524" layer="91"/>
-<wire x1="205.74" y1="-43.18" x2="185.42" y2="-43.18" width="0.1524" layer="91"/>
-<junction x="185.42" y="-43.18"/>
+<wire x1="185.42" y1="-38.1" x2="185.42" y2="-40.64" width="0.1524" layer="91"/>
+<pinref part="X2" gate="-6" pin="S"/>
+<wire x1="185.42" y1="-40.64" x2="185.42" y2="-43.18" width="0.1524" layer="91"/>
+<junction x="185.42" y="-40.64"/>
 </segment>
 <segment>
@@
 </segment>
 </net>
-<net name="N$1" class="0">
-<segment>
-<pinref part="U2" gate="G$1" pin="(ICP1/ADC8)PD4"/>
-<wire x1="152.4" y1="-71.12" x2="195.58" y2="-71.12" width="0.1524" layer="91"/>
-<pinref part="JP1" gate="G$1" pin="1"/>
-<pinref part="D3" gate="G$1" pin="A"/>
-<wire x1="195.58" y1="-71.12" x2="203.2" y2="-71.12" width="0.1524" layer="91"/>
-<wire x1="195.58" y1="-66.04" x2="195.58" y2="-71.12" width="0.1524" layer="91"/>
-<pinref part="D4" gate="G$1" pin="C"/>
-<wire x1="195.58" y1="-71.12" x2="195.58" y2="-73.66" width="0.1524" layer="91"/>
-<junction x="195.58" y="-71.12"/>
-<junction x="152.4" y="-71.12"/>
-</segment>
-</net>
 <net name="N$4" class="0">
 <segment>
-<wire x1="152.4" y1="-25.4" x2="185.42" y2="-25.4" width="0.1524" layer="91"/>
-<pinref part="JP2" gate="G$1" pin="1"/>
+<wire x1="152.4" y1="-25.4" x2="172.72" y2="-25.4" width="0.1524" layer="91"/>
 <pinref part="D5" gate="G$1" pin="A"/>
-<wire x1="185.42" y1="-25.4" x2="203.2" y2="-25.4" width="0.1524" layer="91"/>
+<wire x1="172.72" y1="-25.4" x2="185.42" y2="-25.4" width="0.1524" layer="91"/>
 <wire x1="185.42" y1="-20.32" x2="185.42" y2="-25.4" width="0.1524" layer="91"/>
 <pinref part="D6" gate="G$1" pin="C"/>
@@
 <pinref part="U2" gate="G$1" pin="(PCINT6/OC1B/OC4B/ADC13)PB6"/>
 <junction x="152.4" y="-25.4"/>
+<pinref part="X2" gate="-3" pin="S"/>
+<junction x="172.72" y="-25.4"/>
 </segment>
 </net>
@@
 </segment>
 </net>
-<net name="RF_TRANSCEIVER_CONNECTED_OK" class="0">
-<segment>
-<pinref part="ON4" gate="G$1" pin="C"/>
-<pinref part="U2" gate="G$1" pin="(INT6/AIN0)PE6"/>
-<wire x1="162.56" y1="-55.88" x2="152.4" y2="-55.88" width="0.1524" layer="91"/>
-<label x="157.48" y="-53.34" size="1.778" layer="95"/>
-</segment>
-</net>
 <net name="N$12" class="0">
 <segment>
@@
 <segment>
 <pinref part="ON5" gate="G$1" pin="C"/>
-<wire x1="162.56" y1="-63.5" x2="152.4" y2="-63.5" width="0.1524" layer="91"/>
+<wire x1="162.56" y1="-63.5" x2="160.02" y2="-63.5" width="0.1524" layer="91"/>
 <label x="154.94" y="-63.5" size="1.778" layer="95"/>
+<pinref part="U2" gate="G$1" pin="(SDA/INT1)PD1"/>
+<wire x1="152.4" y1="-78.74" x2="160.02" y2="-78.74" width="0.1524" layer="91"/>
+<wire x1="160.02" y1="-78.74" x2="160.02" y2="-71.12" width="0.1524" layer="91" curve="180"/>
+<wire x1="160.02" y1="-63.5" x2="160.02" y2="-71.12" width="0.1524" layer="91"/>
+<junction x="152.4" y="-78.74"/>
 </segment>
 </net>
@@
 <segment>
 <pinref part="ON6" gate="G$1" pin="C"/>
-<wire x1="162.56" y1="-66.04" x2="152.4" y2="-66.04" width="0.1524" layer="91"/>
 <label x="154.94" y="-68.58" size="1.778" layer="95"/>
-</segment>
-</net>
+<pinref part="U2" gate="G$1" pin="(OC0B/SCL/INT0)PD0"/>
+<wire x1="152.4" y1="-81.28" x2="162.56" y2="-81.28" width="0.1524" layer="91"/>
+<wire x1="162.56" y1="-81.28" x2="162.56" y2="-78.74" width="0.1524" layer="91"/>
+<wire x1="162.56" y1="-78.74" x2="162.56" y2="-71.12" width="0.1524" layer="91" curve="180"/>
+<wire x1="162.56" y1="-71.12" x2="162.56" y2="-66.04" width="0.1524" layer="91"/>
+<junction x="152.4" y="-81.28"/>
+</segment>
+</net>
+<net name="N$1" class="0">
+<segment>
+<wire x1="193.04" y1="-53.34" x2="193.04" y2="-58.42" width="0.1524" layer="91" curve="180"/>
+<pinref part="U2" gate="G$1" pin="(ICP3/CLK0/OC4A)PC7"/>
+<wire x1="152.4" y1="-48.26" x2="193.04" y2="-48.26" width="0.1524" layer="91"/>
+<wire x1="193.04" y1="-53.34" x2="193.04" y2="-48.26" width="0.1524" layer="91"/>
+<wire x1="193.04" y1="-58.42" x2="193.04" y2="-71.12" width="0.1524" layer="91"/>
+<pinref part="D3" gate="G$1" pin="A"/>
+<wire x1="195.58" y1="-71.12" x2="203.2" y2="-71.12" width="0.1524" layer="91"/>
+<wire x1="195.58" y1="-66.04" x2="195.58" y2="-71.12" width="0.1524" layer="91"/>
+<pinref part="D4" gate="G$1" pin="C"/>
+<wire x1="195.58" y1="-71.12" x2="195.58" y2="-73.66" width="0.1524" layer="91"/>
+<junction x="195.58" y="-71.12"/>
+<wire x1="193.04" y1="-71.12" x2="195.58" y2="-71.12" width="0.1524" layer="91"/>
+<junction x="152.4" y="-48.26"/>
+<pinref part="X2" gate="-5" pin="S"/>
+</segment>
+</net>
+<net name="N$13" class="0">
+<segment>
+<pinref part="U2" gate="G$1" pin="(#HWB)PE2"/>
+<wire x1="152.4" y1="-58.42" x2="157.48" y2="-58.42" width="0.1524" layer="91"/>
+<wire x1="157.48" y1="-58.42" x2="157.48" y2="-55.88" width="0.1524" layer="91"/>
+<pinref part="ON4" gate="G$1" pin="C"/>
+<wire x1="157.48" y1="-55.88" x2="162.56" y2="-55.88" width="0.1524" layer="91"/>
+<junction x="152.4" y="-58.42"/>
+</segment>
+</net>
