File: Eagle Projects/SolarEV_RxBoard/RxBrd_v2.brd (EAGLE design)
At the start: 80 x 80.1 mm, 50 parts, among them U2 ATMEGA32U4-XUAU, X1 USBPTH, Y2 16MHz

Commit message: Rx Board Rev 2
Parts:
- removed JP2: PhotovoltaicCell Connect, pinhead:1X02
- added X2: 5566-6, con-molex:5566-6
- JP1: value Anemometer Connect -> (none); device pinhead:1X02 -> jumper:JP1
- moved D6 136.0 mm to (71.6, 34.3), turned to 90 degrees
- moved D5 132.6 mm to (71.6, 24.1), turned to 90 degrees
- moved ON4 119.8 mm to (56.4, 62.0), turned to 180 degrees
- moved JP3 116.2 mm to (68.3, 3.81)
- moved R2 115.5 mm to (52.8, 62.2), turned to 270 degrees
- moved D4 112.3 mm to (59.9, 34.8), turned to 270 degrees
- moved D3 110.5 mm to (66.5, 43.4), turned to 270 degrees
- moved R1 107.9 mm to (41.4, 8.13), turned to 90 degrees
- moved C4 107.0 mm to (48.3, 15.0)
- moved ON3 105.4 mm to (49.5, 54.4), turned to 90 degrees
- moved S1 101.3 mm to (58.7, 46.5), turned to 270 degrees
- moved ON2 99.5 mm to (49.5, 56.4), turned to 90 degrees
- moved ON6 96.8 mm to (55.1, 4.32), turned to 180 degrees
- moved C6 96.6 mm to (38.1, 61.7)
- moved R9 95.3 mm to (59.7, 62.2), turned to 90 degrees
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Connections:
- removed net RF_TRANSCEIVER_CONNECTED_OK: ON4.C, U2.1
- new net N$13: ON4.C, U2.33
- net +5V: now also X2.2; no longer JP1.2
- net GND: now also X2.6; no longer JP2.2
- net N$1: now also U2.32, X2.5; no longer JP1.1, U2.25
- net N$4: now also X2.3; no longer JP2.1
- net RX_LED: now also U2.18
- net TX_LED: now also U2.19
Routing:
- net GND: track 0.00 -> 325.3 mm, vias 0 -> 6
- net +5V: track 0.00 -> 324.3 mm, vias 0 -> 6
- net VUSB: track 0.00 -> 93.5 mm
- net N$4: track 0.00 -> 65.7 mm, vias 0 -> 2
- net N$5: track 0.00 -> 52.5 mm, vias 0 -> 2
- net N$1: track 0.00 -> 49.3 mm
- net N$8: track 0.00 -> 47.2 mm
- net N$7: track 0.00 -> 45.3 mm
- net AVCC: track 0.00 -> 45.2 mm
- net TX_LED: track 0.00 -> 42.4 mm
- net XTAL1: track 0.00 -> 40.8 mm
- net RX_LED: track 0.00 -> 39.5 mm
- net XTAL2: track 0.00 -> 38.8 mm
- net MOSI: track 0.00 -> 29.6 mm
- net MISO: track 0.00 -> 27.9 mm
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Other:
- board text added: "SS Patel 212513168 Support Vehicle Aggredator Board Electronic/Computer Engineering Design 3 UKZN 2015"
