File: Eagle Projects/SolarEV_RxBoard/RxBrd_v2.brd (EAGLE design)
At the start: 80 x 80.1 mm, 49 parts, among them U2 ATMEGA32U4-XUAU, X1 USBPTH, X2 5566-6, Y2 16MHz

Commit message: fixed up patels board :D
Parts:
- removed S1: RESET, SparkFun:TACTILE_SWITCH_SMD
- added C10, C11: 100n, resistor:C0805
- added R13, R14, R15, R16: 1k, resistor:R0805
- moved C2 35.6 mm to (45.0, 50.5)
- moved R8 34.8 mm to (7.24, 23.5), turned to 0 degrees
- moved C8 28.3 mm to (7.24, 26.8), turned to 180 degrees
- moved C9 21.7 mm to (7.24, 30.1), turned to 180 degrees
- moved F1 11.3 mm to (15.6, 32.4), turned to 90 degrees
- moved R4 9.78 mm to (17.4, 43.8)
- moved R5 9.78 mm to (17.4, 41.3)
- moved D3 6.68 mm to (59.9, 42.4)
- moved Z1 4.91 mm to (15.5, 39.2), turned to 180 degrees
- moved Z2 2.68 mm to (15.5, 46.1), turned to 180 degrees
- moved S3 2.30 mm to (12.7, 21.1), turned to 90 degrees
- moved C7 2.09 mm to (22.6, 37.6), turned to 90 degrees
- moved ON4 0.89 mm to (57.3, 62.0)
- moved ON 0.76 mm to (57.1, 56.6)
Connections:
- removed net N$23: ICSP.5, S3.1, S3.2
- new net N$15: R15.1, X2.5
- new net RST: ICSP.5, R6.1, S3.1, S3.2, U2.13
- net GND: now also C10.2, C11.2, R14.2, R16.2; no longer S1.1, S1.2
- net N$1: now also C11.1, R15.2, R16.1; no longer X2.5
- net N$4: now also R13.1; no longer D5.A, D6.C, U2.30
- net N$5: now also C10.1, D5.A, D6.C, R13.2, R14.1, U2.30; no longer R6.1, S1.3, S1.4, U2.13
Routing:
- net +5V: track 322.6 -> 409.8 mm, vias 6 -> 0
- net RST: track 0.00 -> 77.6 mm
- net N$4: track 65.7 -> 11.2 mm, vias 2 -> 0
- net VUSB: track 93.5 -> 55.9 mm
- net N$1: track 49.3 -> 29.6 mm
- net N$15: track 0.00 -> 18.6 mm
- net GND: track 335.6 -> 317.1 mm
- net N$23: track 15.7 -> 0.00 mm
- net RD-: track 7.23 -> 17.1 mm
- net D+: track 20.4 -> 10.6 mm, vias 1 -> 0
- net RD+: track 7.83 -> 17.3 mm
- net D-: track 16.3 -> 8.90 mm
- net N$5: track 52.5 -> 55.8 mm, vias 2 -> 0
- net UCAP: track 11.2 -> 14.2 mm
- net PC_CONNECTED_OK: track 16.4 -> 18.6 mm
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
Commit message: final rx board (i think) is still called rev2 xD
on other side, minor software tweaks but they're nonfunctional atm
Routing:
- net +5V: track 409.8 -> 408.8 mm
Other:
- board text added: "+"
- board text added: "-"
- board text added: "ON"
- board text added: "PC OK WS OK PVC OK"
- board text added: "PVC"
- board text added: "RF OK"
- board text added: "TX/RX"
- board text added: "WS"
Changed lines of the file:
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@@
 <?xml version="1.0" encoding="utf-8"?>
 <!DOCTYPE eagle SYSTEM "eagle.dtd">
-<eagle version="7.2.0">
+<eagle version="7.1.0">
 <drawing>
 <settings>
@@
 <hole x="77" y="77" drill="3.2"/>
 <hole x="3" y="77" drill="3.2"/>
-<text x="16.002" y="67.818" size="1.778" layer="1">SS Patel 212513168
+<text x="6.858" y="68.453" size="1.778" layer="1">SS Patel 212513168
 Support Vehicle Aggredator Board
 Electronic/Computer Engineering Design 3
 UKZN 2015</text>
+<text x="76.327" y="67.564" size="1.778" layer="1">+</text>
+<text x="68.707" y="63.881" size="1.778" layer="1" rot="R90">-</text>
+<text x="47.371" y="2.921" size="1.27" layer="1">TX/RX</text>
+<text x="73.914" y="58.674" size="1.27" layer="1" rot="R270">WS</text>
+<text x="73.914" y="54.864" size="1.27" layer="1" rot="R270">PVC</text>
+<text x="41.529" y="59.944" size="1.27" layer="1">PC OK
+WS OK
+PVC OK</text>
+<text x="59.817" y="67.564" size="1.27" layer="1">RF OK</text>
+<text x="56.769" y="49.149" size="1.27" layer="1">ON</text>
 </plain>
 <attributes>
@@
 <wire x1="59.69" y1="61.38" x2="67.056" y2="61.38" width="0.4064" layer="1"/>
 <wire x1="67.056" y1="61.38" x2="67.144" y2="61.38" width="0.4064" layer="1"/>
-<wire x1="67.144" y1="61.38" x2="67.945" y2="60.579" width="0.8128" layer="1"/>
-<wire x1="67.945" y1="60.579" x2="68.326" y2="60.198" width="0.8128" layer="1"/>
+<wire x1="67.144" y1="61.38" x2="68.326" y2="60.198" width="0.8128" layer="1"/>
 <wire x1="68.326" y1="60.198" x2="75.394" y2="60.198" width="0.8128" layer="1"/>
 <wire x1="75.394" y1="60.198" x2="77.172" y2="58.42" width="0.8128" layer="1"/>
@@
 <wire x1="60.706" y1="1.778" x2="64.77" y2="5.842" width="0.8128" layer="1"/>
 <wire x1="64.77" y1="5.842" x2="75.184" y2="5.842" width="0.8128" layer="1"/>
-<wire x1="75.184" y1="5.842" x2="78.74" y2="9.398" width="0.8128" layer="1"/>
-<wire x1="78.74" y1="9.398" x2="78.74" y2="21.082" width="0.8128" layer="1"/>
-<wire x1="78.74" y1="21.082" x2="77.47" y2="22.352" width="0.8128" layer="1"/>
+<wire x1="75.184" y1="5.842" x2="78.486" y2="9.271" width="0.8128" layer="1"/>
+<wire x1="78.486" y1="9.271" x2="78.486" y2="21.336" width="0.8128" layer="1"/>
+<wire x1="78.486" y1="21.336" x2="77.47" y2="22.352" width="0.8128" layer="1"/>
 <wire x1="77.47" y1="22.352" x2="76.454" y2="22.352" width="0.8128" layer="1"/>
 <wire x1="76.454" y1="22.352" x2="74.93" y2="20.828" width="0.8128" layer="1"/>
@@
 <wire x1="2.032" y1="15.367" x2="12.065" y2="5.334" width="0.8128" layer="1"/>
 <wire x1="12.065" y1="5.334" x2="16.383" y2="5.334" width="0.8128" layer="1"/>
-<wire x1="66.548" y1="60.872" x2="67.056" y2="61.38" width="0.8128" layer="1"/>
 <wire x1="16.383" y1="5.334" x2="16.383" y2="5.234" width="0.4064" layer="1"/>
 <wire x1="16.383" y1="5.234" x2="16.537" y2="5.08" width="0.4064" layer="1"/>
@@
 <contactref element="R5" pad="1"/>
 <contactref element="X1" pad="D+"/>
-<wire x1="16.549" y1="41.275" x2="12.192" y2="41.275" width="0.4064" layer="1"/>
-<wire x1="12.192" y1="41.275" x2="11.938" y2="41.021" width="0.4064" layer="1"/>
-<wire x1="11.938" y1="41.021" x2="9.879" y2="41.021" width="0.4064" layer="1"/>
-<wire x1="9.879" y1="41.021" x2="8.6" y2="42.3" width="0.4064" layer="1"/>
 <wire x1="16.494" y1="39.243" x2="16.494" y2="41.22" width="0.4064" layer="1"/>
 <wire x1="16.494" y1="41.22" x2="16.549" y2="41.275" width="0.4064" layer="1"/>
+<wire x1="16.494" y1="41.22" x2="11.502" y2="41.22" width="0.4064" layer="1"/>
+<wire x1="11.502" y1="41.22" x2="11.303" y2="41.021" width="0.4064" layer="1"/>
+<wire x1="9.779" y1="41.021" x2="11.303" y2="41.021" width="0.254" layer="1"/>
+<wire x1="9.779" y1="41.021" x2="9.017" y2="41.783" width="0.4064" layer="1"/>
+<wire x1="9.017" y1="41.783" x2="9.017" y2="41.883" width="0.4064" layer="1"/>
+<wire x1="9.017" y1="41.883" x2="8.6" y2="42.3" width="0.4064" layer="1"/>
 </signal>
 <signal name="XUSB" class="3">

Commit message: Potato!
Parts:
- removed ICSP: ICSP, SmartPrj:2X03
- added Q2: (no value), crystal:HC49/S
- JP1: value (none) -> AVR-ISP6-75869-131; device jumper:JP1 -> atmel-avr:HDR-75869-131
- moved JP1 34.2 mm to (20.6, 21.3), turned to 90 degrees
- moved R1 22.2 mm to (39.8, 30.2), turned to 180 degrees
- moved C4 5.46 mm to (45.1, 19.4), turned to 180 degrees
- moved C3 5.00 mm to (36.3, 19.3), turned to 0 degrees
- moved Y2 1.55 mm to (40.6, 19.4)
Connections:
- net GND: now also JP1.6; no longer ICSP.6
- net MISO: now also JP1.1; no longer ICSP.1
- net MOSI: now also JP1.4; no longer ICSP.4
- net N$10: now also JP1.2; no longer ICSP.2
- net RST: now also JP1.5; no longer ICSP.5
- net SCK: now also JP1.3; no longer ICSP.3
- net XTAL1: now also Q2.1
- net XTAL2: now also Q2.2
Routing:
- net GND: track 317.1 -> 275.1 mm, vias 6 -> 5
- net XTAL2: track 39.0 -> 25.9 mm
- net XTAL1: track 41.6 -> 29.7 mm
- net +5V: track 408.8 -> 406.9 mm
- net RST: track 77.6 -> 77.1 mm
Other:
- board text added: "5V"
- board text added: "Gnd"
- board text added: "RX"
- board text added: "Tx"
- board text added: "USB"

Commit message: Fixed patties board
Connections:
- net GND: now also U2.33
- net N$13: now also U2.31; no longer U2.33
Routing:
- net GND: track 275.1 -> 289.2 mm
- net N$13: track 24.0 -> 29.2 mm
