File: Eagle Projects/RF Tx Board/Tx_328p.sch (EAGLE design)
At the start: 45 parts, among them Q3 16MHz, Q4 16MHz, U1 ATMEGA328P_TQFP, U2 MCP2551, X1 5566-6, X2 5566-6

Commit message: More Tx board routing
Parts:
- removed TELEMETRY: (no value), pinhead:PINHD-1X5
- added U$3: HEADER-5WAY, con-TE-EP:HEADER-5WAY
Connections:
- net GND: now also U$3.P$1; no longer TELEMETRY.5
- net TX0: now also U$3.P$4; no longer TELEMETRY.2
- net VCC: now also U$3.P$5; no longer TELEMETRY.1
Other:
- moved on the sheet: C2
Changed lines of the file:
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@@
 <part name="P+3" library="supply1" deviceset="VCC" device=""/>
 <part name="GND3" library="supply1" deviceset="GND" device=""/>
-<part name="TELEMETRY" library="pinhead" deviceset="PINHD-1X5" device=""/>
 <part name="U1" library="SparkFun-DigitalIC" deviceset="ATMEGA328P_TQFP" device="" value="ATMEGA328P_TQFP"/>
 <part name="R2" library="resistor" deviceset="R-US_" device="M0805" value="50k"/>
@@
 <part name="X1" library="con-molex" deviceset="5566-6" device=""/>
 <part name="X2" library="con-molex" deviceset="5566-6" device=""/>
+<part name="U$3" library="con-TE-EP" deviceset="HEADER-5WAY" device=""/>
 </parts>
 <sheets>
 <sheet>
 <plain>
-<text x="190.5" y="131.064" size="1.778" layer="91">Vcc
+<text x="193.04" y="131.064" size="1.778" layer="91">Vcc
 Rx
 Tx
@@
 <instance part="P+3" gate="VCC" x="172.72" y="149.86"/>
 <instance part="GND3" gate="1" x="182.88" y="99.06"/>
-<instance part="TELEMETRY" gate="A" x="187.96" y="137.16"/>
 <instance part="U1" gate="U$1" x="96.52" y="60.96"/>
 <instance part="R2" gate="G$1" x="63.5" y="91.44"/>
@@
 <instance part="P+5" gate="VCC" x="205.74" y="114.3"/>
 <instance part="GND5" gate="1" x="205.74" y="96.52"/>
-<instance part="C2" gate="G$1" x="203.2" y="139.7"/>
-<instance part="P+6" gate="VCC" x="203.2" y="147.32"/>
-<instance part="GND6" gate="1" x="203.2" y="129.54"/>
+<instance part="C2" gate="G$1" x="210.82" y="139.7"/>
+<instance part="P+6" gate="VCC" x="210.82" y="147.32"/>
+<instance part="GND6" gate="1" x="210.82" y="129.54"/>
 <instance part="C5" gate="G$1" x="213.36" y="35.56"/>
 <instance part="P+7" gate="VCC" x="213.36" y="43.18"/>
@@
 <instance part="X2" gate="-5" x="180.34" y="-7.62" rot="R90"/>
 <instance part="X2" gate="-6" x="182.88" y="-7.62" rot="R90"/>
+<instance part="U$3" gate="G$1" x="190.5" y="137.16"/>
 </instances>
 <busses>
@@
 </segment>
 <segment>
-<pinref part="TELEMETRY" gate="A" pin="5"/>
 <wire x1="185.42" y1="132.08" x2="177.8" y2="132.08" width="0.1524" layer="91"/>
 <pinref part="GND4" gate="1" pin="GND"/>
@@
 <junction x="177.8" y="132.08"/>
 <pinref part="R1" gate="G$1" pin="2"/>
+<pinref part="U$3" gate="G$1" pin="P$1"/>
 </segment>
 <segment>
@@
 <pinref part="GND6" gate="1" pin="GND"/>
 <pinref part="C2" gate="G$1" pin="2"/>
-<wire x1="203.2" y1="132.08" x2="203.2" y2="134.62" width="0.1524" layer="91"/>
+<wire x1="210.82" y1="132.08" x2="210.82" y2="134.62" width="0.1524" layer="91"/>
 </segment>
 <segment>
@@
 <segment>
 <pinref part="P+3" gate="VCC" pin="VCC"/>
-<pinref part="TELEMETRY" gate="A" pin="1"/>
 <wire x1="172.72" y1="142.24" x2="172.72" y2="147.32" width="0.1524" layer="91"/>
 <wire x1="185.42" y1="142.24" x2="172.72" y2="142.24" width="0.1524" layer="91"/>
+<pinref part="U$3" gate="G$1" pin="P$5"/>
 </segment>
 <segment>
@@
 <pinref part="C2" gate="G$1" pin="1"/>
 <pinref part="P+6" gate="VCC" pin="VCC"/>
-<wire x1="203.2" y1="142.24" x2="203.2" y2="144.78" width="0.1524" layer="91"/>
+<wire x1="210.82" y1="142.24" x2="210.82" y2="144.78" width="0.1524" layer="91"/>
 </segment>
 <segment>
@@
 </segment>
 <segment>
-<pinref part="TELEMETRY" gate="A" pin="2"/>
 <wire x1="185.42" y1="139.7" x2="172.72" y2="139.7" width="0.1524" layer="91"/>
 <label x="162.56" y="139.7" size="1.778" layer="95"/>
@@
 <pinref part="RX_3DR_LED" gate="G$1" pin="A"/>
 <wire x1="172.72" y1="137.16" x2="160.02" y2="137.16" width="0.1524" layer="91"/>
-</segment>
-</net>
+<pinref part="U$3" gate="G$1" pin="P$4"/>
+</segment>
+</net>
