File: Eagle Projects/RF Tx Board/Tx_328p.brd (EAGLE design)
At the start: 80 x 80 mm, 45 parts, among them Q3 16MHz, Q4 16MHz, U1 ATMEGA328P_TQFP, U2 MCP2551, X1 5566-6, X2 5566-6

Commit message: More Tx board routing
Parts:
- removed TELEMETRY: (no value), pinhead:1X05
- added U$3: HEADER-5WAY, con-TE-EP:1744426-5
Connections:
- net GND: now also U$3.P$1; no longer TELEMETRY.5
- net TX0: now also U$3.P$4; no longer TELEMETRY.2
- net VCC: now also U$3.P$5; no longer TELEMETRY.1
Routing:
- net TX0: track 18.1 -> 53.9 mm
- net RX0: track 45.3 -> 75.6 mm
- net GND: track 61.7 -> 92.0 mm, vias 7 -> 9
- net VCC: track 213.6 -> 243.1 mm
- net N$8: track 0.00 -> 22.5 mm, vias 0 -> 4
- net N$9: track 20.2 -> 36.1 mm
- net CANH: track 62.0 -> 55.2 mm
Other:
- board text added: "212503024 | Design 3"
- board text added: "SOLAR EV TX BOARD"
- board text added: "UKZN | Matthew de Neef"
- board text removed: "Tx Rx"

Commit message: Sorted Matts Board :)
Parts:
- removed ., .., R1, R3: 1k, rcl:M0805
- removed RX_3DR_LED, RX_LED, TX_LED, TX_LED_GPS: (no value), led:CHIP-LED0805
- removed S1: SKHMPSE010, switch:SKHMPXE010
- removed USART: (no value), pinhead:1X02
- added C10, C9: 22pF, resistor:C0805K
- added JP1: (no value), pinhead:1X02
- added U$4: HEADER-2WAY, con-TE-EP:1744426-2
- moved C1 46.5 mm to (72.6, 20.1), turned to 270 degrees
- moved C2 39.0 mm to (71.9, 30.8), turned to 180 degrees
- moved RESET 28.3 mm to (51.5, 45.9), turned to 0 degrees
- moved R2 24.9 mm to (65.5, 58.7), turned to 90 degrees
- moved C5 22.4 mm to (58.3, 55.0)
- moved Z1 10.9 mm to (4.34, 11.3), turned to 270 degrees
- moved C4 10.5 mm to (66.2, 69.2), turned to 270 degrees
- moved Z2 10.4 mm to (4.34, 15.4), turned to 90 degrees
- moved R8 9.41 mm to (7.90, 8.53), turned to 180 degrees
- moved U$3 5.84 mm to (77.2, 39.8)
- moved R7 4.84 mm to (22.4, 29.2), turned to 0 degrees
- moved U2 2.20 mm to (10.2, 13.4), turned to 90 degrees
- moved Q1 1.82 mm to (56.2, 72.4), turned to 0 degrees
- moved Q2 1.82 mm to (56.2, 72.4), turned to 0 degrees
- moved LED2 0.76 mm to (17.1, 18.1)
Connections:
- removed net +5V: R7.1
- removed net N$20: X1.5
- removed net N$21: X1.6
- removed net N$26: X2.5
- removed net N$27: X2.6
- removed net N$3: R2.2, U1.29
- removed net N$4: R3.1, TX_LED_GPS.C
- removed net N$5: R1.1, RX_3DR_LED.C
- removed net N$6: ...1, RX_LED.C
- removed net N$8: ..1, TX_LED.C
- removed net N$9: C4.1, U1.21, U1.3, U1.5
- new net N$17: ISP1.2, JP1.2
- new net SPARE1: X1.5, X2.5
- new net SPARE2: X1.6, X2.6
- net GND: now also C10.2, C9.2, U1.21, U1.3, U1.5; no longer ...2, ..2, R1.2, R3.2, S1.1, S1.2
- net N$1: now also C9.1, Q1.2, Q2.2; no longer Q1.1, Q2.1
- net N$2: now also C10.1, Q1.1, Q2.1; no longer Q1.2, Q2.2
- net RST: now also R2.2, RESET.3, RESET.4, U1.29
- net RX0: now also U$4.P$1; no longer TX_LED.A, TX_LED_GPS.A, USART.2
- net TX0: now also U$4.P$2; no longer RX_3DR_LED.A, RX_LED.A, USART.1
- net VCC: now also C4.1, JP1.1, R7.1, U1.6; no longer ISP1.2, RESET.3, RESET.4, S1.3, S1.4
Routing:
- net RST: track 0.00 -> 45.2 mm
- net N$4: track 38.5 -> 0.00 mm, vias 2 -> 0
- net N$9: track 36.1 -> 0.00 mm
- net N$3: track 33.1 -> 0.00 mm, vias 2 -> 0
- net SPARE2: track 0.00 -> 25.1 mm
- net SPARE1: track 0.00 -> 24.8 mm
- net VCC: track 243.1 -> 266.5 mm, vias 7 -> 0
- net N$8: track 22.5 -> 0.00 mm, vias 4 -> 0
- net RX0: track 75.6 -> 53.2 mm, vias 2 -> 0
- net TX0: track 53.9 -> 33.5 mm
- net N$5: track 19.2 -> 0.00 mm
- net GND: track 92.0 -> 110.0 mm, vias 9 -> 8
- net MOSI: track 68.0 -> 53.0 mm, vias 2 -> 0
- net N$17: track 0.00 -> 10.6 mm
- net CANL: track 56.5 -> 48.9 mm, vias 1 -> 0
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
Commit message: Added status LEDs for Tx board
Parts:
- added LED4, LED5: (no value), led:SML0805
- added R1, R3: (no value), resistor:M0805
- moved C7 0.63 mm to (12.3, 20.2)
- moved R5 0.52 mm to (14.5, 23.9)
- moved C8 0.51 mm to (19.7, 23.9)
- moved R4 0.44 mm to (16.9, 23.8)
Connections:
- new net LED_DIAG: LED5.C, U1.1
- new net LED_RF: LED4.C, U1.32
- new net N$4: LED4.A, R1.2
- new net N$5: LED5.A, R3.2
- net RX0: now also U$3.P$3
- net VCC: now also R1.1, R3.1
Routing:
- net VCC: track 266.5 -> 283.0 mm
- net LED_RF: track 0.00 -> 11.5 mm
- net LED_DIAG: track 0.00 -> 9.34 mm
- net RX0: track 53.2 -> 60.5 mm
- net N$4: track 0.00 -> 2.93 mm
- net N$5: track 0.00 -> 2.78 mm
- net GND: track 110.0 -> 111.1 mm
Other:
- board text added: "CAN I/O"
- board text added: "RESET"
- board text added: "RF TX USART"

Commit message: Exported BMP's
Parts:
- added JP2: (no value), pinhead:1X01
Connections:
- new net N$3: GPS.3, JP2.1
Routing:
- net VCC: track 283.0 -> 287.5 mm
- net N$3: track 0.00 -> 3.82 mm
Other:
- board text added: "5V"
- board text added: "GND"
- board text added: "PWR"
- board text added: "RXD"
- board text added: "Reset"
- board text added: "SMPS Regulator"
- board text added: "TXD"
- board text added: "Vin"
- board text added: "Vout"

Commit message: Fixed n00b mistake on board+Schematic for Tx board
Connections:
- net N$3: now also GPS.2; no longer GPS.3
- net RX0: now also GPS.3; no longer GPS.2
Routing:
- net RX0: track 60.5 -> 58.0 mm
- net N$3: track 3.82 -> 5.28 mm

Commit message: Fixed my silly on matts board
Connections:
- net CANCS: now also U1.14
- net CANINT: now also U1.13
Changed lines of the file:
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@@
 <wire x1="35.941" y1="28.448" x2="35.941" y2="25.2308" width="0.4064" layer="1"/>
 <wire x1="35.941" y1="25.2308" x2="35.9156" y2="25.2054" width="0.4064" layer="1"/>
+<contactref element="U1" pad="13"/>
+<wire x1="35.179" y1="29.21" x2="54.0994" y2="62.1" width="0" layer="19" extent="1-1"/>
 </signal>
 <signal name="CANCS">
 <contactref element="U$1" pad="16"/>
+<contactref element="U1" pad="14"/>
+<wire x1="24.4856" y1="26.6573" x2="54.0994" y2="61.3" width="0" layer="19" extent="1-1"/>
 </signal>
 <signal name="N$10">
