File: Eagle Projects/Ben/SD Node/SD_Node.sch (EAGLE design)
At the start: 33 parts, among them Q1 16MHz, Q3 16MHz, Q4 16MHz, Q5 16MHz, U1 ATMEGA328P_TQFP, U2 MCP2551, X1 5566-6, X2 5566-6

Commit message: Working on the things..
Parts:
- added JP3, JP5: (no value), pinhead:PINHD-1X1
- added LED4, LED5, LED6: (no value), led:LEDCHIP-LED0805
- added R2, R8, R9: 50k, resistor:R-US_R0805
- added U$4: SHROOM15MM, RobThePyro:SHROOM15MM
- added U$5: SHROOM5MM, RobThePyro:SHROOM5MM
Connections:
- new net N$11: R2.1, U1.PC3(ADC3)
- new net N$12: R8.1, U1.PC2(ADC2)
- new net N$13: LED6.C, R9.1
- new net N$16: JP3.1, U1.PD0(RXD)
- new net N$17: JP5.1, U1.PD1(TXD)
- new net N$4: LED4.A, R2.2
- new net N$5: LED5.A, R8.2
- net +5V: now also LED6.A
- net GND: now also LED4.C, LED5.C, R9.2
Changed lines of the file:
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@@
 <part name="P+9" library="supply1" deviceset="+5V" device=""/>
 <part name="GND4" library="supply1" deviceset="GND" device=""/>
+<part name="U$4" library="RobThePyro" deviceset="SHROOM" device="15MM"/>
+<part name="U$5" library="RobThePyro" deviceset="SHROOM" device="5MM"/>
+<part name="GND11" library="supply1" deviceset="GND" device=""/>
+<part name="LED4" library="led" deviceset="LED" device="CHIP-LED0805"/>
+<part name="LED5" library="led" deviceset="LED" device="CHIP-LED0805"/>
+<part name="R2" library="resistor" deviceset="R-US_" device="R0805" value="50k"/>
+<part name="R8" library="resistor" deviceset="R-US_" device="R0805" value="50k"/>
+<part name="JP3" library="pinhead" deviceset="PINHD-1X1" device=""/>
+<part name="JP5" library="pinhead" deviceset="PINHD-1X1" device=""/>
+<part name="LED6" library="led" deviceset="LED" device="CHIP-LED0805"/>
+<part name="R9" library="resistor" deviceset="R-US_" device="R0805" value="50k"/>
 </parts>
 <sheets>
@@
 <instance part="P+9" gate="1" x="83.82" y="83.82"/>
 <instance part="GND4" gate="1" x="83.82" y="73.66"/>
+<instance part="U$4" gate="G$1" x="154.94" y="15.24"/>
+<instance part="U$5" gate="G$1" x="162.56" y="15.24"/>
+<instance part="GND11" gate="1" x="27.94" y="76.2"/>
+<instance part="LED4" gate="G$1" x="17.78" y="88.9" rot="R90"/>
+<instance part="LED5" gate="G$1" x="17.78" y="93.98" rot="R90"/>
+<instance part="R2" gate="G$1" x="10.16" y="88.9"/>
+<instance part="R8" gate="G$1" x="10.16" y="93.98"/>
+<instance part="JP3" gate="G$1" x="12.7" y="73.66"/>
+<instance part="JP5" gate="G$1" x="12.7" y="71.12"/>
+<instance part="LED6" gate="G$1" x="-7.62" y="134.62" rot="R90"/>
+<instance part="R9" gate="G$1" x="7.62" y="134.62"/>
 </instances>
 <busses>
@@
 <segment>
 <pinref part="S1" gate="S" pin="3"/>
+<pinref part="GND15" gate="1" pin="GND"/>
+<wire x1="-43.18" y1="116.84" x2="-45.72" y2="116.84" width="0.1524" layer="91"/>
+<wire x1="-45.72" y1="116.84" x2="-48.26" y2="116.84" width="0.1524" layer="91"/>
+<wire x1="-48.26" y1="116.84" x2="-48.26" y2="111.76" width="0.1524" layer="91"/>
 <pinref part="S1" gate="S" pin="4"/>
-<wire x1="-48.26" y1="111.76" x2="-45.72" y2="111.76" width="0.1524" layer="91"/>
-<pinref part="GND15" gate="1" pin="GND"/>
-<wire x1="-43.18" y1="116.84" x2="-48.26" y2="116.84" width="0.1524" layer="91"/>
-<wire x1="-48.26" y1="116.84" x2="-48.26" y2="111.76" width="0.1524" layer="91"/>
-<junction x="-48.26" y="111.76"/>
+<wire x1="-45.72" y1="111.76" x2="-45.72" y2="116.84" width="0.1524" layer="91"/>
+<junction x="-45.72" y="116.84"/>
 </segment>
 <segment>
@@
 <pinref part="GND16" gate="1" pin="GND"/>
 <wire x1="-20.32" y1="129.54" x2="-17.78" y2="129.54" width="0.1524" layer="91"/>
-<wire x1="-17.78" y1="129.54" x2="-17.78" y2="121.92" width="0.1524" layer="91"/>
+<wire x1="-17.78" y1="129.54" x2="-17.78" y2="127" width="0.1524" layer="91"/>
 <pinref part="C8" gate="G$1" pin="1"/>
+<wire x1="-17.78" y1="124.46" x2="-17.78" y2="121.92" width="0.1524" layer="91"/>
 <wire x1="-17.78" y1="121.92" x2="-17.78" y2="116.84" width="0.1524" layer="91"/>
 <wire x1="-20.32" y1="121.92" x2="-17.78" y2="121.92" width="0.1524" layer="91"/>
 <junction x="-17.78" y="121.92"/>
+<pinref part="R9" gate="G$1" pin="2"/>
+<wire x1="12.7" y1="134.62" x2="15.24" y2="134.62" width="0.1524" layer="91"/>
+<wire x1="15.24" y1="134.62" x2="15.24" y2="127" width="0.1524" layer="91"/>
+<wire x1="15.24" y1="127" x2="-17.78" y2="127" width="0.1524" layer="91"/>
+<wire x1="-17.78" y1="127" x2="-17.78" y2="124.46" width="0.1524" layer="91"/>
 </segment>
 <segment>
@@
 <pinref part="GND4" gate="1" pin="GND"/>
 <wire x1="86.36" y1="76.2" x2="83.82" y2="76.2" width="0.1524" layer="91"/>
+</segment>
+<segment>
+<pinref part="LED5" gate="G$1" pin="C"/>
+<pinref part="LED4" gate="G$1" pin="C"/>
+<wire x1="22.86" y1="93.98" x2="22.86" y2="88.9" width="0.1524" layer="91"/>
+<pinref part="GND11" gate="1" pin="GND"/>
+<wire x1="22.86" y1="88.9" x2="27.94" y2="88.9" width="0.1524" layer="91"/>
+<wire x1="27.94" y1="88.9" x2="27.94" y2="78.74" width="0.1524" layer="91"/>
+<junction x="22.86" y="88.9"/>
 </segment>
 </net>
@@
 <wire x1="-30.48" y1="121.92" x2="-30.48" y2="129.54" width="0.1524" layer="91"/>
 <junction x="-30.48" y="129.54"/>
+<pinref part="LED6" gate="G$1" pin="A"/>
+<wire x1="-10.16" y1="134.62" x2="-30.48" y2="134.62" width="0.1524" layer="91"/>
+<junction x="-30.48" y="134.62"/>
 </segment>
 <segment>
@@
 </segment>
 </net>
+<net name="N$4" class="0">
+<segment>
+<pinref part="LED4" gate="G$1" pin="A"/>
+<pinref part="R2" gate="G$1" pin="2"/>
+</segment>
+</net>
+<net name="N$5" class="0">
+<segment>
+<pinref part="LED5" gate="G$1" pin="A"/>
+<pinref part="R8" gate="G$1" pin="2"/>
+</segment>
+</net>
+<net name="N$11" class="0">
+<segment>
+<pinref part="R2" gate="G$1" pin="1"/>
+<pinref part="U1" gate="U$1" pin="PC3(ADC3)"/>
+<wire x1="5.08" y1="88.9" x2="2.54" y2="88.9" width="0.1524" layer="91"/>
+</segment>
+</net>
+<net name="N$12" class="0">
+<segment>
+<pinref part="U1" gate="U$1" pin="PC2(ADC2)"/>
+<pinref part="R8" gate="G$1" pin="1"/>
+<wire x1="2.54" y1="91.44" x2="5.08" y2="91.44" width="0.1524" layer="91"/>
+<wire x1="5.08" y1="91.44" x2="5.08" y2="93.98" width="0.1524" layer="91"/>
+</segment>
+</net>
+<net name="N$16" class="0">
+<segment>
+<pinref part="U1" gate="U$1" pin="PD0(RXD)"/>
+<wire x1="2.54" y1="73.66" x2="10.16" y2="73.66" width="0.1524" layer="91"/>
+<pinref part="JP3" gate="G$1" pin="1"/>
+</segment>
+</net>
+<net name="N$17" class="0">
+<segment>
+<pinref part="U1" gate="U$1" pin="PD1(TXD)"/>
+<wire x1="2.54" y1="71.12" x2="10.16" y2="71.12" width="0.1524" layer="91"/>
+<pinref part="JP5" gate="G$1" pin="1"/>
+</segment>
+</net>
+<net name="N$13" class="0">
+<segment>
+<pinref part="LED6" gate="G$1" pin="C"/>
+<pinref part="R9" gate="G$1" pin="1"/>
+<wire x1="-2.54" y1="134.62" x2="2.54" y2="134.62" width="0.1524" layer="91"/>
+</segment>
+</net>
