File: Eagle Projects/Ben/SD Node/SD_Node.brd (EAGLE design)
At the start: 93 x 90 mm, 33 parts, among them Q1 16MHz, Q3 16MHz, Q4 16MHz, Q5 16MHz, U1 ATMEGA328P_TQFP, U2 MCP2551, X1 5566-6, X2 5566-6

Commit message: SD Node Done?
Parts:
- moved C2 42.2 mm to (44.9, 4.27), turned to 315 degrees
- moved C1 40.0 mm to (41.8, 7.31), turned to 135 degrees
- moved Q1 33.5 mm to (47.8, 7.56), turned to 315 degrees
- moved Q5 33.4 mm to (47.8, 7.57), turned to 135 degrees
- moved U$2 28.5 mm to (41.8, 72.9), turned to 270 degrees
- moved U$3 26.4 mm to (40.2, 35.0), turned to 90 degrees
- moved JP2 17.3 mm to (27.2, 29.1), turned to 0 degrees
- moved C8 15.7 mm to (59.0, 21.5), turned to 315 degrees
- moved S1 15.5 mm to (47.3, 24.8), turned to 270 degrees
- moved R1 12.6 mm to (39.6, 15.4), turned to 0 degrees
- moved U1 12.5 mm to (53.6, 16.7), turned to 45 degrees
- moved JP1 9.42 mm to (36.2, 22.1)
- moved C7 8.92 mm to (45.2, 16.8), turned to 225 degrees
- moved X1 6.77 mm to (8.41, 64.2)
- moved C5 6.77 mm to (18.1, 28.6)
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Routing:
- net +5V: track 76.4 -> 186.9 mm, vias 0 -> 2
- net MOSI: track 31.7 -> 92.2 mm
- net MISO: track 35.9 -> 94.7 mm, vias 2 -> 0
- net SCK: track 33.8 -> 83.6 mm
- net +12V: track 34.5 -> 77.8 mm
- net SD_CS: track 29.3 -> 53.4 mm
- net CANCS: track 22.9 -> 41.9 mm, vias 0 -> 2
- net CANINT: track 37.9 -> 56.0 mm, vias 2 -> 0
- net RST: track 43.2 -> 25.9 mm, vias 2 -> 0
- net GND: track 59.2 -> 69.1 mm, vias 7 -> 6
- net N$10: track 13.3 -> 7.90 mm
- net N$1: track 15.7 -> 14.0 mm
- net N$2: track 15.5 -> 14.8 mm
Other:
- board size 93 x 90 mm -> 67 x 75 mm

Commit message: Working on the things..
Parts:
- added JP3, JP5: (no value), pinhead:1X01
- added LED4, LED5, LED6: (no value), led:CHIP-LED0805
- added R2, R8, R9: 50k, resistor:R0805
- added U$4: SHROOM15MM, RobThePyro:SHROOM15MM
- added U$5: SHROOM5MM, RobThePyro:SHROOM
Connections:
- new net N$11: R2.1, U1.26
- new net N$12: R8.1, U1.25
- new net N$13: LED6.C, R9.1
- new net N$16: JP3.1, U1.30
- new net N$17: JP5.1, U1.31
- new net N$4: LED4.A, R2.2
- new net N$5: LED5.A, R8.2
- net +5V: now also LED6.A
- net GND: now also LED4.C, LED5.C, R9.2
Routing:
- net N$5: track 0.00 -> 25.4 mm
- net N$4: track 0.00 -> 18.0 mm
- net GND: track 69.1 -> 83.6 mm, vias 6 -> 7
- net +5V: track 186.9 -> 195.1 mm
- net N$17: track 0.00 -> 5.53 mm
- net N$11: track 0.00 -> 4.00 mm
- net N$12: track 0.00 -> 3.14 mm
- net N$16: track 0.00 -> 2.58 mm
- net N$13: track 0.00 -> 2.57 mm
- net SD_CS: track 53.4 -> 52.9 mm
Other:
- board text added: "213560382"
- board text added: "DIYElectronics.co.za"
- board text added: "R Mawbey"
- board text added: "SD Card Node Rev1.0"
- board text added: "SDCard Module"
- board text added: "SMPS Regulator"
- board text added: "SolarForce1 | UKZN | 2015"
- board text added: "Vin"
- board text added: "Vout"
- board text added: "rambo@rambo.co.za"
