File: Eagle Projects/Ben/Test Node/Test_Node.brd (EAGLE design)
At the start: 100 x 80 mm, 28 parts, among them Q1 16MHz, Q3 16MHz, Q4 16MHz, U1 ATMEGA328P_TQFP, U2 MCP2551

Commit message: Display Node Done?
Parts:
- removed JP3: GFX_LCD, adafruit:1X20
- removed Q2: (no value), SparkFun:SOT23
- added C10: 10uF, resistor:C0805
- added C11, C12, C13, C14, C15, C16, C17, C18, C19, C20, C21, C22: 10nF, resistor:C0805
- added C7, C8, C9: 100nF, resistor:C0805
- added F1: (no value), adafruit:1812
- added LED4, LED5: (no value), led:CHIP-LED0805
- added LED6, LED7: (no value), led:LED5MM
- added Q5: 16MHz, crystal:HC49UP
- added Q6, Q7: 2N7002, transistor-fet:SOT23
- added R10, R9: 1k, resistor:R0805
- added R11, R12, R13, R14, R15, R16, R17, R18, R19, R20, R21, R22: 470E, resistor:R0805
- added R8: 100E, resistor:R0805
- added S1: RESET, SparkFun:TACTILE_SWITCH_SMD
- added S2, S3: SWITCH-MOMENTARY-2PTH, SparkFun:TACTILE-PTH
- added S4: BTN3, SparkFun:TACTILE_SWITCH_SMD
- added S5: BTN4, SparkFun:TACTILE_SWITCH_SMD
- added U$10, U$11, U$12, U$13, U$14, U$15, U$16, U$17, U$18, U$19, U$8, U$9: DRTR5V0U1SO, RobThePyro:SOT23
- added U$2: SMPSBOARD, RobThePyro:SMPSBOARD
- added U$3: BYT12864FLCD, RobThePyro:BYT12864F
- added U$4: HEADER-6WAY, con-TE-EP:1744426-6
- added U$5: HEADER-5WAY, con-TE-EP:1744426-5
- added U$6: HEADER-3WAY, con-TE-EP:1744426-3
- added U$7: HEADER-2WAY, con-TE-EP:1744426-2
- added X1, X2: 5566-6, con-molex:5566-6
- JP2: value CAN_Interface -> (none); device pinhead:1X04 -> pinhead:1X02
- R2: value 1k -> 100E
- R7: value 1k -> 100k
- moved C1 99.6 mm to (50.7, 46.3), turned to 270 degrees
- moved R2 89.2 mm to (62.3, 9.67), turned to 180 degrees
- moved Q1 86.4 mm to (49.4, 41.0), turned to 180 degrees
- moved R1 73.7 mm to (52.1, 17.0), turned to 90 degrees
- moved C2 71.1 mm to (48.0, 46.3), turned to 270 degrees
- moved Z2 54.9 mm to (6.86, 37.2), turned to 90 degrees
- moved Z1 52.8 mm to (6.86, 33.2), turned to 270 degrees
- moved R7 46.8 mm to (10.4, 30.4), turned to 180 degrees
- moved U2 46.2 mm to (12.7, 35.2), turned to 90 degrees
- moved Q3 45.0 mm to (10.7, 17.2), turned to 270 degrees
- moved Q4 45.0 mm to (10.7, 17.2), turned to 270 degrees
- moved C3 39.9 mm to (15.0, 13.9), turned to 270 degrees
- moved C4 38.5 mm to (15.0, 20.5), turned to 90 degrees
- moved C5 37.6 mm to (19.6, 35.2), turned to 90 degrees
- moved LED2 36.9 mm to (18.0, 31.1), turned to 90 degrees
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Connections:
- net N$10 renamed CANSTBY
- removed net SS: JP2.1, U1.14
- new net +12V: U$2.VIN, U$4.P$2, X1.3, X2.3
- new net A0: C22.1, R22.2, U$19.1, U1.27
- new net A1: C21.1, R21.2, U$18.1, U1.28
- new net BTN1: C14.1, R14.2, U$11.1, U1.32
- new net BTN2: C13.1, R13.2, U$10.1, U1.1
- new net BTN3: C12.1, R12.2, S2.3, S4.3, S4.4, U$9.1, U1.2
- new net BTN4: C11.1, R11.2, S3.3, S5.3, S5.4, U$8.1, U1.9
- new net CRUISE1: C18.1, R18.2, U$15.1, U1.23
- new net CRUISE2: C17.1, R17.2, U$14.1, U1.24
- new net CRUISE3: C16.1, R16.2, U$13.1, U1.25
- new net CRUISE4: C15.1, R15.2, U$12.1, U1.26
- new net LCD_RST: U$3.P$4
- new net LED1: C20.1, LED4.C, LED7.K, R20.2, U$17.1, U1.30
- new net LED2: C19.1, LED5.C, LED6.K, R19.2, U$16.1, U1.31
- new net N$10: JP1.2, JP2.2
- new net N$11: Q6.2, U$3.P$15
- new net N$12: Q6.1, R8.2
- new net N$13: LED4.A, LED7.A, R9.2
- new net N$14: X1.5, X2.5
- new net N$15: X1.6, X2.6
- new net N$16: LED5.A, LED6.A, R10.2
- new net N$17: F1.2, U$7.P$2
- new net N$18: R11.1, U$6.P$3
- new net N$19: R12.1, U$6.P$2
- new net N$20: R13.1, U$6.P$1
- new net N$21: R14.1, U$5.P$5
- new net N$22: R18.1, U$4.P$3
- new net N$23: R17.1, U$4.P$4
- new net N$24: R16.1, U$4.P$5
- new net N$25: R15.1, U$4.P$6
- new net N$26: R19.1, U$5.P$4
- new net N$27: R20.1, U$5.P$3
- new net N$28: R21.1, U$5.P$2
- new net N$29: R22.1, U$5.P$1
- new net SCKCNTRL: R8.1, U1.10
- net +5V: now also C10.1, C7.2, C8.2, C9.1, F1.1, JP2.1, R10.1, R9.1, U$10.2, U$11.2, U$12.2, U$13.2, U$14.2, U$15.2, U$16.2, U$17.2, U$18.2, U$19.2, U$2.VOUT, U$3.P$19, U$3.P$2, U$8.2, U$9.2; no longer JP1.2, JP3.17, JP3.19, JP3.2
- net CANCS: now also U1.14
- net CANH: now also X1.1, X2.1
- net CANINT: now also U1.12
- net CANL: now also X1.4, X2.4
- net GND: now also C10.2, C11.2, C12.2, C13.2, C14.2, C15.2, C16.2, C17.2, C18.2, C19.2, C20.2, C21.2, C22.2, C7.1, C8.1, C9.2, Q7.2, S1.3, S1.4, S2.1, S3.1, S4.1, S4.2, S5.1, S5.2, U$10.3, U$11.3, U$12.3, U$13.3, U$14.3, U$15.3, U$16.3, U$17.3, U$18.3, U$19.3, U$2.GND, U$2.GND@, U$3.P$20, U$3.P$6, U$4.P$1, U$7.P$1, U$8.3, U$9.3, X1.2, X2.2; no longer JP3.1, JP3.15, Q2.2
- net LCD_CS: now also U$3.P$17, U1.11; no longer JP3.4, U1.12
- net MISO: no longer JP2.3
- net MOSI: now also U$3.P$16; no longer JP2.2, JP3.5
- net N$1: now also Q5.2
- net N$2: now also Q5.1
- net N$4: now also Q7.3, U$3.P$1; no longer JP3.20, Q2.3
- net N$5: now also Q7.1; no longer Q2.1
- net RST: now also S1.1, S1.2
- net SCK: now also Q6.3; no longer JP2.4, JP3.6
Routing:
- net +5V: track 44.2 -> 366.2 mm, vias 0 -> 12
- net +12V: track 0.00 -> 176.8 mm
- net GND: track 29.5 -> 165.6 mm, vias 5 -> 19
- net LED2: track 0.00 -> 104.8 mm
- net LED1: track 0.00 -> 104.0 mm
- net BTN4: track 0.00 -> 80.7 mm, vias 0 -> 2
- net BTN3: track 0.00 -> 71.5 mm, vias 0 -> 1
- net RST: track 0.00 -> 44.3 mm, vias 0 -> 2
- net MOSI: track 0.00 -> 44.2 mm
- net SCK: track 0.00 -> 40.0 mm
- net CANH: track 3.33 -> 42.5 mm
- net LCD_CS: track 0.00 -> 39.0 mm, vias 0 -> 2
- net CANL: track 3.33 -> 41.4 mm
- net MISO: track 0.00 -> 35.9 mm, vias 0 -> 2
- net CRUISE1: track 0.00 -> 32.1 mm
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- added copper zone on layer 16, net GND
Other:
- board size 100 x 80 mm -> 93 x 90 mm

Commit message: Working on the things..
Parts:
- removed C11, C12, C13, C14, C15, C16, C17, C18, C19, C20, C21, C22: 10nF, resistor:C0805
- removed F1: (no value), adafruit:1812
- removed R11, R12, R13, R14, R15, R16, R17, R18, R19, R20, R21, R22: 470E, resistor:R0805
- removed U$10, U$11, U$12, U$13, U$14, U$15, U$16, U$17, U$18, U$19, U$8, U$9: DRTR5V0U1SO, RobThePyro:SOT23
- removed U$5: HEADER-5WAY, con-TE-EP:1744426-5
- removed U$6: HEADER-3WAY, con-TE-EP:1744426-3
- removed U$7: HEADER-2WAY, con-TE-EP:1744426-2
- added SW2: EC12E_SW, switch-alps:ALPS_EC12E_SW
- U$4: value HEADER-6WAY -> HEADER-4WAY; device con-TE-EP:1744426-6 -> con-TE-EP:1744426-4
- moved U$4 11.4 mm to (84.1, 31.2)
Connections:
- removed net A0: C22.1, R22.2, U$19.1, U1.27
- removed net A1: C21.1, R21.2, U$18.1, U1.28
- removed net BTN1: C14.1, R14.2, U$11.1, U1.32
- removed net BTN2: C13.1, R13.2, U$10.1, U1.1
- removed net CRUISE1: C18.1, R18.2, U$15.1, U1.23
- removed net CRUISE2: C17.1, R17.2, U$14.1, U1.24
- removed net CRUISE3: C16.1, R16.2, U$13.1, U1.25
- removed net CRUISE4: C15.1, R15.2, U$12.1, U1.26
- removed net N$20: R13.1, U$6.P$1
- removed net N$21: R14.1, U$5.P$5
- removed net N$22: R18.1, U$4.P$3
- removed net N$23: R17.1, U$4.P$4
- removed net N$24: R16.1, U$4.P$5
- removed net N$25: R15.1, U$4.P$6
- removed net N$26: R19.1, U$5.P$4
- removed net N$27: R20.1, U$5.P$3
- removed net N$28: R21.1, U$5.P$2
- removed net N$29: R22.1, U$5.P$1
- new net RX: U$4.P$2, U1.30
- new net TX: U$4.P$3, U1.31
- net +12V: no longer U$4.P$2
- net +5V: now also U$4.P$4; no longer F1.1, U$10.2, U$11.2, U$12.2, U$13.2, U$14.2, U$15.2, U$16.2, U$17.2, U$18.2, U$19.2, U$8.2, U$9.2
- net BTN3: no longer C12.1, R12.2, U$9.1, U1.2
- net BTN4: no longer C11.1, R11.2, U$8.1
- net GND: now also SW2.C, SW2.D; no longer C11.2, C12.2, C13.2, C14.2, C15.2, C16.2, C17.2, C18.2, C19.2, C20.2, C21.2, C22.2, U$10.3, U$11.3, U$12.3, U$13.3, U$14.3, U$15.3, U$16.3, U$17.3, U$18.3, U$19.3, U$7.P$1, U$8.3, U$9.3
- net LED1: no longer C20.1, R20.2, U$17.1, U1.30
- net LED2: no longer C19.1, R19.2, U$16.1, U1.31
- net N$17: now also SW2.A, U1.1; no longer F1.2, U$7.P$2
- net N$18: now also SW2.B, U1.32; no longer R11.1, U$6.P$3
- net N$19: now also SW2.E, U1.2; no longer R12.1, U$6.P$2
Routing:
- net +5V: track 366.2 -> 284.6 mm, vias 12 -> 0
- net GND: track 165.6 -> 109.3 mm, vias 19 -> 7
- net CRUISE1: track 32.1 -> 0.00 mm
- net BTN2: track 32.0 -> 0.00 mm
- net CRUISE2: track 29.7 -> 0.00 mm
- net A0: track 28.9 -> 0.00 mm
- net LED1: track 104.0 -> 75.6 mm
- net BTN1: track 28.0 -> 0.00 mm
- net A1: track 26.3 -> 0.00 mm
- net LED2: track 104.8 -> 78.7 mm
- net CRUISE3: track 25.9 -> 0.00 mm
- net CRUISE4: track 24.9 -> 0.00 mm
- net N$22: track 11.3 -> 0.00 mm
- net N$23: track 9.06 -> 0.00 mm
- net N$24: track 7.41 -> 0.00 mm
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