File: Eagle Projects/Ben/Test Node/Test_Node.sch (EAGLE design)
At the start: 10 parts, among them Q1 16MHz, U1 ATMEGA328P_TQFP

Commit message: Working on PCB's and Generic CAN interface
Parts:
- added C3, C4: 22pF, resistor:C-EUC0805K
- added C5, C6: 100nF, resistor:C-EUC0805K
- added LED1: RX, led:LEDCHIP-LED0805
- added LED2: TX, led:LEDCHIP-LED0805
- added LED3: INT, led:LEDCHIP-LED0805
- added Q3: 16MHz, crystal:CRYSTALHC49S
- added Q4: 16MHz, crystal:CRYSTALHC49UP
- added R3, R4, R5, R7: 1k, resistor:R-US_R0805
- added R6: 100k, resistor:R-US_R0805
- added U$1: MCP2515SO, RobThePyro:MCP2515SO
- added U2: MCP2551, SparkFun:MCP2551
- added Z1, Z2: TVS-UD-SOD323, supressor:TVS-UD-SOD323
Connections:
- new net CANCS: U$1G$1.!CS
- new net CANH: U2.CANH, Z1.C
- new net CANINT: LED3.C, U$1G$1.!INT
- new net CANL: U2.CANL, Z2.C
- new net CANRST: R6.2, U$1G$1.!RESET
- new net N$10: R7.1, U2.RS
- new net N$3: C3.1, Q3.2, Q4.2, U$1G$1.OSC1
- new net N$6: C4.1, Q3.1, Q4.1, U$1G$1.OSC2
- new net N$7: LED1.A, R3.1
- new net N$8: LED2.A, R4.1
- new net N$9: LED3.A, R5.1
- new net RXCAN: LED1.C, U$1G$1.RXCAN, U2.RXD
- new net TXCAN: LED2.C, U$1G$1.TXCAN, U2.TXD
- net +5V: now also C5.2, C6.2, R3.2, R4.2, R5.2, R6.1, U$1G$2.VDD, U2.VDD
- net GND: now also C3.2, C4.2, C5.1, C6.1, R7.2, U$1G$2.VSS, U2.VSS, Z1.A, Z2.A
- net MISO: now also U$1G$1.SO
- net MOSI: now also U$1G$1.SI
- net SCK: now also U$1G$1.SCK
Other:
- note added: "CAN Interface"

Commit message: Display Node Done?
Parts:
- removed JP3: GFX_LCD, adafruit:PINHD-1X20
- removed Q2: (no value), SparkFun:TRANSISTOR_NPNSOT23
- added C10: 10uF, resistor:C-EUC0805
- added C11, C12, C13, C14, C15, C16, C17, C18, C19, C20, C21, C22: 10nF, resistor:C-EUC0805
- added C7, C8, C9: 100nF, resistor:C-EUC0805
- added F1: (no value), adafruit:PTCFUSE-1812
- added LED4, LED5: (no value), led:LEDCHIP-LED0805
- added LED6, LED7: (no value), led:LED5MM
- added Q5: 16MHz, crystal:CRYSTALHC49UP
- added Q6, Q7: 2N7002, transistor-fet:2N7002
- added R10, R9: 1k, resistor:R-US_R0805
- added R11, R12, R13, R14, R15, R16, R17, R18, R19, R20, R21, R22: 470E, resistor:R-US_R0805
- added R8: 100E, resistor:R-US_R0805
- added S1: RESET, SparkFun:TAC_SWITCHSMD
- added S2, S3: SWITCH-MOMENTARY-2PTH, SparkFun:SWITCH-MOMENTARY-2PTH
- added S4: BTN3, SparkFun:TAC_SWITCHSMD
- added S5: BTN4, SparkFun:TAC_SWITCHSMD
- added U$10, U$11, U$12, U$13, U$14, U$15, U$16, U$17, U$18, U$19, U$8, U$9: DRTR5V0U1SO, RobThePyro:DRTR5V0U1SO
- added U$2: SMPSBOARD, RobThePyro:SMPSBOARD
- added U$3: BYT12864FLCD, RobThePyro:BYT12864FLCD
- added U$4: HEADER-6WAY, con-TE-EP:HEADER-6WAY
- added U$5: HEADER-5WAY, con-TE-EP:HEADER-5WAY
- added U$6: HEADER-3WAY, con-TE-EP:HEADER-3WAY
- added U$7: HEADER-2WAY, con-TE-EP:HEADER-2WAY
- added X1, X2: 5566-6, con-molex:5566-6
- JP2: value CAN_Interface -> (none); device pinhead:PINHD-1X4 -> pinhead:PINHD-1X2
- R2: value 1k -> 100E
- R7: value 1k -> 100k
Connections:
- net N$10 renamed CANSTBY
- removed net SS: JP2.1, U1.PB2(SS/OC1B)
- new net +12V: U$2.VIN, U$4.P$2, X1-3.S, X2-3.S
- new net A0: C22.1, R22.2, U$19.I/O, U1.PC4(ADC4/SDA)
- new net A1: C21.1, R21.2, U$18.I/O, U1.PC5(ADC5/SCL)
- new net BTN1: C14.1, R14.2, U$11.I/O, U1.PD2(INT0)
- new net BTN2: C13.1, R13.2, U$10.I/O, U1.PD3(INT1)
- new net BTN3: C12.1, R12.2, S2.2, S4.3, S4.4, U$9.I/O, U1.PD4(XCK/T0)
- new net BTN4: C11.1, R11.2, S3.2, S5.3, S5.4, U$8.I/O, U1.PD5(T1)
- new net CRUISE1: C18.1, R18.2, U$15.I/O, U1.PC0(ADC0)
- new net CRUISE2: C17.1, R17.2, U$14.I/O, U1.PC1(ADC1)
- new net CRUISE3: C16.1, R16.2, U$13.I/O, U1.PC2(ADC2)
- new net CRUISE4: C15.1, R15.2, U$12.I/O, U1.PC3(ADC3)
- new net LCD_RST: U$3.!RST
- new net LED1: C20.1, LED4.C, LED7.C, R20.2, U$17.I/O, U1.PD0(RXD)
- new net LED2: C19.1, LED5.C, LED6.C, R19.2, U$16.I/O, U1.PD1(TXD)
- new net N$10: JP1.2, JP2.2
- new net N$11: Q6.S, U$3.SCK/E
- new net N$12: Q6.G, R8.2
- new net N$13: LED4.A, LED7.A, R9.2
- new net N$14: X1-5.S, X2-5.S
- new net N$15: X1-6.S, X2-6.S
- new net N$16: LED5.A, LED6.A, R10.2
- new net N$17: F1.2, U$7.P$2
- new net N$18: R11.1, U$6.P$3
- new net N$19: R12.1, U$6.P$2
- new net N$20: R13.1, U$6.P$1
- new net N$21: R14.1, U$5.P$5
- new net N$22: R18.1, U$4.P$3
- new net N$23: R17.1, U$4.P$4
- new net N$24: R16.1, U$4.P$5
- new net N$25: R15.1, U$4.P$6
- new net N$26: R19.1, U$5.P$4
- new net N$27: R20.1, U$5.P$3
- new net N$28: R21.1, U$5.P$2
- new net N$29: R22.1, U$5.P$1
- new net SCKCNTRL: R8.1, U1.PD6(AIN0)
- net +5V: now also C10.1, C7.2, C8.2, C9.1, F1.1, JP2.1, R10.1, R9.1, U$10.VCC, U$11.VCC, U$12.VCC, U$13.VCC, U$14.VCC, U$15.VCC, U$16.VCC, U$17.VCC, U$18.VCC, U$19.VCC, U$2.VOUT, U$3.A+, U$3.VDD, U$8.VCC, U$9.VCC; no longer JP1.2, JP3.17, JP3.19, JP3.2
- net CANCS: now also U1.PB2(SS/OC1B)
- net CANH: now also X1-1.S, X2-1.S
- net CANINT: now also U1.PB0(ICP)
- net CANL: now also X1-4.S, X2-4.S
- net GND: now also C10.2, C11.2, C12.2, C13.2, C14.2, C15.2, C16.2, C17.2, C18.2, C19.2, C20.2, C21.2, C22.2, C7.1, C8.1, C9.2, Q7.S, S1.3, S1.4, S2.1, S3.1, S4.1, S4.2, S5.1, S5.2, U$10.GND, U$11.GND, U$12.GND, U$13.GND, U$14.GND, U$15.GND, U$16.GND, U$17.GND, U$18.GND, U$19.GND, U$2.GND, U$2.GND@1, U$3.PSB, U$3.VSS, U$4.P$1, U$7.P$1, U$8.GND, U$9.GND, X1-2.S, X2-2.S; no longer JP3.1, JP3.15, Q2.E
- net LCD_CS: now also U$3.CS/RS, U1.PD7(AIN1); no longer JP3.4, U1.PB0(ICP)
- net MISO: no longer JP2.3
- net MOSI: now also U$3.MOSI/RW; no longer JP2.2, JP3.5
- net N$1: now also Q5.2
- net N$2: now also Q5.1
- net N$4: now also Q7.D, U$3.K-; no longer JP3.20, Q2.C
- net N$5: now also Q7.G; no longer Q2.B
- net RST: now also S1.1, S1.2
- net SCK: now also Q6.D; no longer JP2.4, JP3.6
Other:
- note added: "Power Supply"
- moved on the sheet: C3, C4, C5, C6, LED1, LED2, LED3, Q3, Q4, R2, R3, R4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

Commit message: Working on the things..
Parts:
- removed C11, C12, C13, C14, C15, C16, C17, C18, C19, C20, C21, C22: 10nF, resistor:C-EUC0805
- removed F1: (no value), adafruit:PTCFUSE-1812
- removed R11, R12, R13, R14, R15, R16, R17, R18, R19, R20, R21, R22: 470E, resistor:R-US_R0805
- removed U$10, U$11, U$12, U$13, U$14, U$15, U$16, U$17, U$18, U$19, U$8, U$9: DRTR5V0U1SO, RobThePyro:DRTR5V0U1SO
- removed U$5: HEADER-5WAY, con-TE-EP:HEADER-5WAY
- removed U$6: HEADER-3WAY, con-TE-EP:HEADER-3WAY
- removed U$7: HEADER-2WAY, con-TE-EP:HEADER-2WAY
- added SW2: EC12E_SW, switch-alps:EC12E_SW
- U$4: value HEADER-6WAY -> HEADER-4WAY; device con-TE-EP:HEADER-6WAY -> con-TE-EP:HEADER-4WAY
Connections:
- removed net A0: C22.1, R22.2, U$19.I/O, U1.PC4(ADC4/SDA)
- removed net A1: C21.1, R21.2, U$18.I/O, U1.PC5(ADC5/SCL)
- removed net BTN1: C14.1, R14.2, U$11.I/O, U1.PD2(INT0)
- removed net BTN2: C13.1, R13.2, U$10.I/O, U1.PD3(INT1)
- removed net CRUISE1: C18.1, R18.2, U$15.I/O, U1.PC0(ADC0)
- removed net CRUISE2: C17.1, R17.2, U$14.I/O, U1.PC1(ADC1)
- removed net CRUISE3: C16.1, R16.2, U$13.I/O, U1.PC2(ADC2)
- removed net CRUISE4: C15.1, R15.2, U$12.I/O, U1.PC3(ADC3)
- removed net N$20: R13.1, U$6.P$1
- removed net N$21: R14.1, U$5.P$5
- removed net N$22: R18.1, U$4.P$3
- removed net N$23: R17.1, U$4.P$4
- removed net N$24: R16.1, U$4.P$5
- removed net N$25: R15.1, U$4.P$6
- removed net N$26: R19.1, U$5.P$4
- removed net N$27: R20.1, U$5.P$3
- removed net N$28: R21.1, U$5.P$2
- removed net N$29: R22.1, U$5.P$1
- new net RX: U$4.P$2, U1.PD0(RXD)
- new net TX: U$4.P$3, U1.PD1(TXD)
- net +12V: no longer U$4.P$2
- net +5V: now also U$4.P$4; no longer F1.1, U$10.VCC, U$11.VCC, U$12.VCC, U$13.VCC, U$14.VCC, U$15.VCC, U$16.VCC, U$17.VCC, U$18.VCC, U$19.VCC, U$8.VCC, U$9.VCC
- net BTN3: no longer C12.1, R12.2, U$9.I/O, U1.PD4(XCK/T0)
- net BTN4: no longer C11.1, R11.2, U$8.I/O
- net GND: now also SW2G$1.C, SW2G$2.1; no longer C11.2, C12.2, C13.2, C14.2, C15.2, C16.2, C17.2, C18.2, C19.2, C20.2, C21.2, C22.2, U$10.GND, U$11.GND, U$12.GND, U$13.GND, U$14.GND, U$15.GND, U$16.GND, U$17.GND, U$18.GND, U$19.GND, U$7.P$1, U$8.GND, U$9.GND
- net LED1: no longer C20.1, R20.2, U$17.I/O, U1.PD0(RXD)
- net LED2: no longer C19.1, R19.2, U$16.I/O, U1.PD1(TXD)
- net N$17: now also SW2G$1.A, U1.PD3(INT1); no longer F1.2, U$7.P$2
- net N$18: now also SW2G$1.B, U1.PD2(INT0); no longer R11.1, U$6.P$3
- net N$19: now also SW2G$2.2, U1.PD4(XCK/T0); no longer R12.1, U$6.P$2
