File: Eagle Projects/Terayza/D3/MPU.brd (EAGLE design)
At the start: 100 x 80 mm, 31 parts, among them Q2 16MHz, Q3 16MHz, U1 ATMEGA328P-AU, U2 MCP2551, X1 5566-6, X2 5566-6

Commit message: MPU almost happy
Parts:
- removed JP2: AVR-ISP-6, avr-6:AVR-ISP-6
- added ISP1: AVRISP-BOX, adafruit:AVRISP-BOX
- added U$4: HEADER-2WAY, con-TE-EP:1744426-2
- moved Z2 86.3 mm to (7.11, 15.2), turned to 90 degrees
- moved Z1 84.1 mm to (7.11, 11.2), turned to 270 degrees
- moved R9 78.0 mm to (10.7, 8.38), turned to 180 degrees
- moved U2 77.6 mm to (13.0, 13.2), turned to 90 degrees
- moved C5 72.2 mm to (14.7, 19.8), turned to 180 degrees
- moved R6 67.1 mm to (16.8, 23.6), turned to 90 degrees
- moved LED2 64.9 mm to (18.8, 18.3), turned to 180 degrees
- moved R5 62.0 mm to (19.3, 23.6), turned to 90 degrees
- moved LED1 60.0 mm to (21.3, 18.3), turned to 180 degrees
- moved R8 58.7 mm to (20.8, 26.7), turned to 180 degrees
- moved C6 56.5 mm to (22.1, 23.6), turned to 90 degrees
- moved U$3 51.8 mm to (14.0, 77.5), turned to 270 degrees
- moved C4 47.3 mm to (29.5, 15.2), turned to 180 degrees
- moved Q2 46.9 mm to (32.8, 10.9), turned to 0 degrees
- moved Q3 46.9 mm to (32.8, 10.9), turned to 0 degrees
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Connections:
- net N$10 renamed SCL
- net N$11 renamed SDA
- net N$12 renamed INT
- new net OUTPUT: U$4.P$1, U1.24
- net GND: now also ISP1.6; no longer JP2.6
- net MISO: now also ISP1.1; no longer JP2.1
- net MOSI: now also ISP1.4; no longer JP2.4
- net RST: now also ISP1.5; no longer JP2.5
- net SCK: now also ISP1.3; no longer JP2.3
- net VCC: now also ISP1.2; no longer JP2.2
Routing:
- net VIN: track 0.00 -> 67.5 mm
- net CANH: track 3.33 -> 49.3 mm
- net CANL: track 3.33 -> 47.2 mm
- net SCK: track 8.76 -> 44.9 mm
- net MOSI: track 13.3 -> 46.0 mm
- net MISO: track 14.0 -> 41.0 mm
- net SPARE2: track 0.00 -> 24.5 mm
- net SPARE1: track 0.00 -> 23.5 mm
- net GND: track 34.7 -> 54.9 mm
- net N$5: track 0.00 -> 13.5 mm
- net N$7: track 34.8 -> 22.0 mm
- net N$6: track 0.00 -> 12.3 mm
- net RST: track 14.6 -> 5.98 mm
- net +5V: track 44.2 -> 50.3 mm
- net RXCAN: track 25.5 -> 30.7 mm
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Other:
- board text added: "SMPS Regulator"
- board text added: "Vin"
- board text added: "Vout"

Commit message: fixed some T things/
Routing:
- added copper zone on layer 16, net GND
Other:
- board size 100 x 80 mm -> 80 x 80 mm
Changed lines of the file:
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@@
 <?xml version="1.0" encoding="utf-8"?>
 <!DOCTYPE eagle SYSTEM "eagle.dtd">
-<eagle version="6.5.0">
+<eagle version="7.2.0">
 <drawing>
 <settings>
@@
 <setting verticaltext="up"/>
 </settings>
-<grid distance="0.05" unitdist="inch" unit="mm" style="lines" multiple="1" display="no" altdistance="0.025" altunitdist="inch" altunit="mm"/>
+<grid distance="1" unitdist="mm" unit="mm" style="lines" multiple="1" display="no" altdistance="0.635" altunitdist="mm" altunit="mm"/>
 <layers>
 <layer number="1" name="Top" color="4" fill="1" visible="yes" active="yes"/>
@@
 <layer number="43" name="vRestrict" color="2" fill="10" visible="yes" active="yes"/>
 <layer number="44" name="Drills" color="7" fill="1" visible="no" active="yes"/>
-<layer number="45" name="Holes" color="7" fill="1" visible="no" active="yes"/>
+<layer number="45" name="Holes" color="7" fill="1" visible="yes" active="yes"/>
 <layer number="46" name="Milling" color="3" fill="1" visible="no" active="yes"/>
 <layer number="47" name="Measures" color="7" fill="1" visible="no" active="yes"/>
@@
 <board>
 <plain>
-<wire x1="0" y1="0" x2="100" y2="0" width="0" layer="20"/>
-<wire x1="100" y1="0" x2="100" y2="80" width="0" layer="20"/>
-<wire x1="100" y1="80" x2="0" y2="80" width="0" layer="20"/>
+<wire x1="0" y1="0" x2="80" y2="0" width="0" layer="20"/>
+<wire x1="80" y1="0" x2="80" y2="80" width="0" layer="20"/>
+<wire x1="80" y1="80" x2="0" y2="80" width="0" layer="20"/>
 <wire x1="0" y1="80" x2="0" y2="0" width="0" layer="20"/>
-<wire x1="100" y1="-0.01" x2="0" y2="-0.01" width="0" layer="20"/>
 <text x="20.41" y="47.39" size="1.778" layer="1" rot="R90">SMPS Regulator</text>
 <text x="33.02" y="69.85" size="1.778" layer="1" rot="R90">Vin</text>
 <text x="33.02" y="39.37" size="1.778" layer="1" rot="R90">Vout</text>
+<hole x="3" y="3" drill="3.2"/>
+<hole x="77" y="3" drill="3.2"/>
+<hole x="77" y="77" drill="3.2"/>
+<hole x="3" y="77" drill="3.2"/>
 </plain>
 <attributes>
@@
 <pass name="Default">
 <param name="RoutingGrid" value="50mil"/>
+<param name="AutoGrid" value="1"/>
+<param name="Efforts" value="0"/>
+<param name="TopRouterVariant" value="1"/>
 <param name="tpViaShape" value="round"/>
 <param name="PrefDir.1" value="|"/>
@@
 <contactref element="ISP1" pad="6"/>
 <contactref element="ISP1" pad="6"/>
-<wire x1="41.8338" y1="66.3448" x2="41.0464" y2="58.1152" width="0" layer="19" extent="1-1"/>
+<polygon width="0.6096" layer="16" isolate="0.8128">
+<vertex x="0" y="0"/>
+<vertex x="80" y="0"/>
+<vertex x="80" y="80"/>
+<vertex x="0" y="80"/>
+</polygon>
 <wire x1="40.2336" y1="66.3448" x2="41.8338" y2="66.3448" width="0" layer="19" extent="1-1"/>
 <wire x1="43.18" y1="70.17" x2="41.8338" y2="66.3448" width="0" layer="19" extent="1-1"/>
-<wire x1="15.47" y1="75.47" x2="43.18" y2="70.17" width="0" layer="19" extent="1-1"/>
-<wire x1="3.6" y1="57.15" x2="15.47" y2="75.47" width="0" layer="19" extent="1-1"/>
-<wire x1="3.6" y1="35.56" x2="3.6" y2="57.15" width="0" layer="19" extent="1-1"/>
-<wire x1="15.47" y1="35.47" x2="3.6" y2="35.56" width="0" layer="19" extent="1-1"/>
-<wire x1="22.098" y1="22.622" x2="15.47" y2="35.47" width="0" layer="19" extent="1-1"/>
-<wire x1="16.764" y1="18.034" x2="22.098" y2="21.844" width="0" layer="19" extent="1-1"/>
-<wire x1="26.67" y1="15.24" x2="22.86" y2="21.082" width="0" layer="19" extent="1-1"/>
-<wire x1="7.112" y1="16.383" x2="7.112" y2="10.033" width="0" layer="19" extent="1-1"/>
-<wire x1="34.544" y1="17.3101" x2="28.464" y2="15.24" width="0" layer="19" extent="1-1"/>
-<wire x1="37.068" y1="15.24" x2="36.83" y2="15.478" width="0" layer="19" extent="1-1"/>
-<wire x1="42.6303" y1="45.85405" x2="7.112" y2="9.652" width="0" layer="19" extent="1-1"/>
-<wire x1="41.0464" y1="58.1152" x2="58.27" y2="73.62" width="0" layer="19" extent="1-1"/>
+<wire x1="41.0464" y1="58.1152" x2="41.8338" y2="66.3448" width="0" layer="19" extent="1-1"/>
+<wire x1="42.6303" y1="45.85405" x2="41.0464" y2="58.1152" width="0" layer="19" extent="1-1"/>
+<wire x1="36.83" y1="15.478" x2="37.068" y2="15.24" width="0" layer="19" extent="1-1"/>
 </signal>
 <signal name="VCC">
@@
 <wire x1="46.1264" y1="62.6364" x2="44.7548" y2="62.6364" width="0.4064" layer="1"/>
 <contactref element="ISP1" pad="5"/>
-<wire x1="39.8363" y1="45.85405" x2="48.26" y2="66.36" width="0" layer="19" extent="1-1"/>
+<wire x1="39.8363" y1="45.85405" x2="44.7548" y2="62.6364" width="0" layer="19" extent="1-1"/>
 </signal>
 <signal name="MISO">
@@
 <wire x1="37.338" y1="18.796" x2="38.288" y2="18.796" width="0.4064" layer="1"/>
 <wire x1="38.288" y1="18.796" x2="38.354" y2="18.862" width="0.4064" layer="1"/>
-<wire x1="12.827" y1="19.447" x2="13.732" y2="19.812" width="0" layer="19" extent="1-16"/>
 <wire x1="15.5702" y1="13.843" x2="17.653" y2="13.843" width="0.4064" layer="1"/>
 <wire x1="17.653" y1="13.843" x2="17.78" y2="13.97" width="0.4064" layer="1"/>
@@
 <contactref element="U1" pad="24"/>
 <contactref element="U$4" pad="P$1"/>
-<wire x1="58.27" y1="58.44" x2="43.434" y2="58.1152" width="0" layer="19" extent="1-1"/>
+<wire x1="43.434" y1="58.1152" x2="58.27" y2="58.44" width="0" layer="19" extent="1-1"/>
 </signal>
 </signals>
