File: Eagle Projects/Terayza/D3/MPU.brd (EAGLE design)
At the start: 80 x 80 mm, 32 parts, among them Q2 16MHz, Q3 16MHz, U1 ATMEGA328P-AU, U2 MCP2551, X1 5566-6, X2 5566-6

Commit message: Updates
Parts:
- removed ISP1: AVRISP-BOX, adafruit:AVRISP-BOX
- removed U$4: HEADER-2WAY, con-TE-EP:1744426-2
- removed U1: ATMEGA328P-AU, Atmel_By_element14_Batch_1-00:QFP80P900X900X120-32N
- added C7, C8: 100nF, resistor:C0805
- added JP1: AVR-ISP6-75869-131, atmel-avr:HDR-75869-131
- added LED4, LED5: (no value), led:CHIP-LED0805
- added Q4: (no value), special:QS
- added R10, R12: 560E, resistor:M0805
- added S1, S2: (no value), SparkFun:TACTILE_SWITCH_SMD
- added U3: ATMEGA328P_TQFP, SparkFun-DigitalIC:TQFP32-08
- Q1: device crystal:HC49/S -> crystal:HC49UP
- moved R2 26.6 mm to (63.3, 46.5)
- moved R4 26.6 mm to (63.3, 41.4)
- moved R3 26.6 mm to (63.3, 43.9)
- moved U$1 26.1 mm to (73.4, 46.5)
- moved Q1 23.9 mm to (31.5, 54.1)
- moved C1 23.9 mm to (21.4, 54.1)
- moved U$3 19.3 mm to (15.8, 58.2), turned to 0 degrees
- moved C2 17.3 mm to (42.1, 53.9), turned to 270 degrees
- moved R1 17.3 mm to (47.2, 50.1), turned to 270 degrees
- moved LED3 6.08 mm to (40.7, 18.8)
- moved C3 6.08 mm to (38.4, 9.62)
- moved C4 6.08 mm to (31.8, 9.62)
- moved LED1 6.08 mm to (23.7, 12.7)
- moved Q2 6.08 mm to (35.1, 5.30)
- moved Q3 6.08 mm to (35.1, 5.30)
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Connections:
- removed net OUTPUT: U$4.P$1, U1.24
- removed net VCC: ISP1.2, R1.2, U$1.P$5, U1.18, U1.20, U1.4, U1.6
- new net CANINIT: U3.13
- new net N$10: S2.1, S2.2, U3.9
- new net N$11: R1.2, U3.29
- new net N$12: LED4.A, R10.1
- new net N$14: LED5.A, R12.1
- new net N$15: LED4.C, U3.26
- new net N$17: C1.2, Q1.2, Q4.2, U3.8
- net +5V: now also C7.2, C8.2, JP1.2, R1.1, R10.2, R12.2, U$1.P$5, U3.18, U3.20, U3.4, U3.6
- net CANCS: now also U3.14
- net GND: now also C7.1, C8.1, JP1.6, S1.3, S1.4, S2.3, S2.4, U3.21, U3.3, U3.5; no longer ISP1.6, U1.21, U1.3, U1.5
- net MISO: now also JP1.1, U3.16; no longer ISP1.1, U1.16
- net MOSI: now also JP1.4, U3.15; no longer ISP1.4, U1.15
- net N$5: now also U3.28; no longer U1.28
- net N$6: now also U3.27; no longer U1.27
- net N$7: now also U3.32; no longer U1.32
- net N$8: now also LED5.C, U3.25; no longer C2.2, Q1.1, U1.7
- net N$9: now also C2.2, Q1.1, Q4.1, U3.7; no longer C1.2, Q1.2, U1.8
- net RST: now also JP1.5, S1.1, S1.2; no longer ISP1.5, R1.1, U1.29
- net SCK: now also JP1.3, U3.17; no longer ISP1.3, U1.17
Routing:
- net GND: track 54.9 -> 259.7 mm
- net +5V: track 50.3 -> 115.2 mm, vias 0 -> 2
- net CANCS: track 0.00 -> 29.0 mm
- net SCK: track 44.9 -> 19.9 mm
- net MOSI: track 46.0 -> 24.2 mm
- net N$7: track 22.0 -> 42.4 mm
- net VIN: track 67.5 -> 47.7 mm
- net N$17: track 0.00 -> 19.6 mm
- net N$10: track 0.00 -> 17.5 mm
- net MISO: track 41.0 -> 25.2 mm
- net N$11: track 0.00 -> 10.8 mm
- net RST: track 5.98 -> 16.6 mm
- net CANH: track 49.3 -> 59.6 mm
- net N$6: track 12.3 -> 20.3 mm
- net CANL: track 47.2 -> 55.1 mm
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
Commit message: Done
Parts:
- added D1: (no value), diode:SMB
- moved C7 23.5 mm to (39.7, 37.4), turned to 180 degrees
- moved C8 12.7 mm to (40.6, 51.8)
- moved S1 4.62 mm to (52.1, 29.5), turned to 45 degrees
- moved C2 2.72 mm to (40.5, 56.0)
- moved R8 1.02 mm to (23.3, 22.1)
Connections:
- removed net VOUT: U$3.VOUT
- new net N$16: D1.A, JP1.2
- net +5V: now also D1.C, U$3.VOUT; no longer JP1.2
Routing:
- net +5V: track 115.2 -> 237.8 mm, vias 2 -> 0
- net GND: track 259.7 -> 203.7 mm, vias 5 -> 6
- net N$16: track 0.00 -> 7.49 mm
- net MISO: track 25.2 -> 31.1 mm
- net CANCS: track 29.0 -> 31.6 mm
- net RST: track 16.6 -> 19.1 mm
- net N$9: track 15.8 -> 14.1 mm
- net CANRST: track 8.26 -> 8.88 mm
Other:
- board text added: "211515873"
- board text added: "MPU-6050 Board"
- board text added: "Terayza Eldridge"
- board text added: "V1"
