File: Eagle Projects/Terayza/D3/Speed.brd (EAGLE design)
At the start: 100 x 80 mm, 36 parts, among them Q2 16MHz, Q3 16MHz, U1 ATMEGA328P-AU, U2 MCP2551, X1 5566-6, X2 5566-6

Commit message: Helped with T board
Parts:
- removed JP5: AVR-ISP-6, avr-6:AVR-ISP-6
- removed U$5: DRTR5V0U1SO, RobThePyro:SOT23
- removed U1: ATMEGA328P-AU, Atmel_By_element14_Batch_1-00:QFP80P900X900X120-32N
- added C1, C9: 100nF, resistor:C0805
- added D1: (no value), diode:SMB
- added F1: MF-MSMF014-2, adafruit:1812
- added JP1: AVR-ISP6-75869-131, atmel-avr:HDR-75869-131
- added LED4, LED5: (no value), led:CHIP-LED0805
- added OK1: LTV816, optocoupler:DIL04
- added R10, R11: 560E, resistor:M0805
- added R12, R13, R14, R15: (no value), resistor:M0805
- added R16: 10K, resistor:M0805
- added S1: BTN3, SparkFun:TACTILE_SWITCH_SMD
- added S4: RST, SparkFun:TACTILE_SWITCH_SMD
- added U3: ATMEGA328P_TQFP, SparkFun-DigitalIC:TQFP32-08
- R9: value (none) -> 680E
- U$7: value HEADER-2WAY -> HEADER-4WAY; device con-TE-EP:1744426-2 -> con-TE-EP:1744426-4
- moved R9 94.0 mm to (75.4, 27.1), turned to 90 degrees
- moved C8 66.7 mm to (57.0, 26.3)
- moved Z2 53.0 mm to (5.45, 15.5)
- moved U$7 52.5 mm to (64.3, 4.32), turned to 0 degrees
- moved Z1 50.7 mm to (4.32, 13.2), turned to 0 degrees
- moved C2 50.2 mm to (25.1, 53.1)
- moved R1 47.9 mm to (44.8, 31.3), turned to 90 degrees
- moved U2 47.8 mm to (8.89, 9.14), turned to 90 degrees
- moved Q1 47.4 mm to (35.4, 54.1)
- moved C6 42.7 mm to (12.4, 14.5), turned to 180 degrees
- moved R5 39.4 mm to (14.5, 18.3), turned to 90 degrees
- moved C3 38.8 mm to (45.5, 54.6)
- moved R8 37.7 mm to (17.3, 5.33), turned to 270 degrees
- moved R4 37.3 mm to (50.8, 43.3)
- moved LED2 34.7 mm to (16.5, 13.0), turned to 180 degrees
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Connections:
- removed net PB0: R9.2, U1.12
- new net A0: R12.1, R14.2, U3.24
- new net A0IN: R12.2, U$7.P$3
- new net A1: R13.1, R15.2, U3.23
- new net A1IN: R13.2, U$7.P$2
- new net FUSEDVCC: F1.1, U$1.P$3, U$2.P$3, U$7.P$4
- new net HE1: R3.1, U3.32
- new net HE2: R4.1, U3.1
- new net MTSPD: C8.2, OK1.4, R16.1, U3.30
- new net N$10: LED5.C, U3.26
- new net N$2: D1.A, JP1.2
- new net N$5: C3.2, Q1.2, U3.7
- new net N$6: C2.2, Q1.1, U3.8
- new net N$9: LED4.C, U3.25
- net CANCS: now also U3.14
- net CANINT: now also U3.13
- net GND: now also C1.1, C9.1, JP1.6, OK1.3, R14.1, R15.1, S1.3, S1.4, S4.3, S4.4, U$7.P$1, U3.21, U3.3, U3.5; no longer JP5.6, U$5.3, U1.21, U1.3, U1.5
- net MISO: now also JP1.1, U3.16; no longer JP5.1, U1.16
- net MOSI: now also JP1.4, U3.15; no longer JP5.4, U1.15
- net N$11: now also S1.1, S1.2, U3.27; no longer U$4.VIN
- net N$12: now also OK1.2, U$6.P$2; no longer U$4.VOUT
- net N$3: no longer C8.2, U$5.1
- net N$4: now also OK1.1, R9.2; no longer U$7.P$1, U1.24
- net N$7: now also LED4.A, R10.1; no longer C3.2, Q1.2, U1.8
- net N$8: now also LED5.A, R11.1; no longer C2.2, Q1.1, U1.7
- net PD2: no longer R3.1, U1.32
- net PD3: no longer R4.1, U1.1
- net RST: now also JP1.5, S4.1, S4.2, U3.29; no longer JP5.5, U1.29
- net SCK: now also JP1.3, U3.17; no longer JP5.3, U1.17
- net VCC: now also C1.2, C9.2, D1.C, F1.2, R10.2, R11.2, R16.2, U$4.VOUT, U3.18, U3.20, U3.4, U3.6; no longer JP5.2, U$1.P$3, U$2.P$3, U$5.2, U1.18, U1.20, U1.4, U1.6
- net VIN: now also U$4.VIN
Routing:
- net FUSEDVCC: track 0.00 -> 59.0 mm
- net CANH: track 3.33 -> 49.6 mm
- net PD3: track 44.9 -> 0.00 mm
- net CANL: track 3.33 -> 46.7 mm
- net CANINT: track 8.54 -> 41.6 mm, vias 0 -> 2
- net CANCS: track 0.00 -> 31.7 mm
- net RST: track 0.00 -> 30.6 mm, vias 0 -> 2
- net MISO: track 1.56 -> 29.9 mm
- net SPARE1: track 0.00 -> 25.3 mm
- net SPARE2: track 0.00 -> 24.7 mm
- net MOSI: track 1.56 -> 25.8 mm
- net VIN: track 0.00 -> 24.2 mm
- net GND: track 29.6 -> 50.0 mm
- net SCK: track 1.56 -> 21.8 mm
- net N$3: track 0.00 -> 13.9 mm
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- added copper zone on layer 16, net GND
Other:
- board size 100 x 80 mm -> 80 x 80 mm

Commit message: Speed basically done
Parts:
- moved S1 118.5 mm to (50.9, 48.6), turned to 180 degrees
- moved R11 106.8 mm to (53.2, 41.1)
- moved R10 103.8 mm to (53.2, 43.1)
- moved LED5 95.6 mm to (49.1, 41.1), turned to 90 degrees
- moved LED4 92.5 mm to (49.0, 43.1), turned to 90 degrees
- moved C9 81.4 mm to (55.2, 26.7), turned to 90 degrees
- moved C1 76.7 mm to (56.1, 23.2), turned to 180 degrees
- moved R15 14.2 mm to (52.6, 17.7), turned to 90 degrees
- moved R12 11.9 mm to (58.5, 17.7), turned to 270 degrees
- moved R4 11.3 mm to (61.7, 46.2)
- moved R13 10.2 mm to (61.5, 17.7), turned to 270 degrees
- moved R1 9.58 mm to (37.3, 37.2)
- moved R14 8.36 mm to (55.8, 17.7), turned to 90 degrees
- moved R16 7.72 mm to (58.7, 30.7), turned to 90 degrees
- moved R3 3.86 mm to (61.8, 35.1)
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Connections:
- net A0IN: now also R13.2; no longer R12.2
- net A1IN: now also R12.2; no longer R13.2
- net GND: now also S1.1
- net N$10: now also LED4.C; no longer LED5.C
- net N$11: no longer S1.1
- net N$9: now also LED5.C; no longer LED4.C
Routing:
- net GND: track 50.0 -> 325.7 mm
- net VCC: track 0.00 -> 131.7 mm, vias 0 -> 4
- net A1: track 0.00 -> 62.2 mm
- net MTSPD: track 0.00 -> 38.3 mm
- net A0: track 0.00 -> 31.1 mm
- net HE1: track 0.00 -> 27.3 mm
- net VIN: track 24.2 -> 50.4 mm
- net HE2: track 0.00 -> 24.1 mm
- net N$6: track 0.00 -> 12.3 mm
- net N$5: track 0.00 -> 12.3 mm
- net RST: track 30.6 -> 41.3 mm
- net N$11: track 0.00 -> 8.52 mm
- net A1IN: track 0.00 -> 7.73 mm
- net A0IN: track 0.00 -> 7.56 mm
- net N$9: track 0.00 -> 6.38 mm
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
Commit message: fixed some T things/
Parts:
- added Q4: 16MHz, crystal:HC49UP
- moved C2 2.54 mm to (24.8, 55.2)
- moved C3 2.25 mm to (44.8, 55.8)
Connections:
- removed net +5V: C6.2, C7.2, R2.2, R5.2, R6.2, R7.1, U$3.18, U2.3
- net N$5: now also Q4.2
- net N$6: now also Q4.1
- net VCC: now also C6.2, C7.2, R2.2, R5.2, R6.2, R7.1, U$3.18, U2.3
Routing:
- net +5V: track 48.1 -> 0.00 mm
- net VCC: track 131.7 -> 174.6 mm
- net GND: track 325.7 -> 297.3 mm
- net N$6: track 12.3 -> 14.9 mm
- net N$5: track 12.3 -> 14.5 mm
- net A1: track 62.2 -> 64.1 mm
- net A0IN: track 7.56 -> 8.32 mm
- net A1IN: track 7.73 -> 8.48 mm
