File: Eagle Projects/Terayza/D3/Speed.brd (EAGLE design)
At the start: 80 x 80 mm, 52 parts, among them Q2 16MHz, Q3 16MHz, Q4 16MHz, U2 MCP2551, U3 ATMEGA328P_TQFP, X1 5566-6, X2 5566-6

Commit message: Speedy
Routing:
- net VCC: track 174.6 -> 242.2 mm, vias 4 -> 6
- net GND: track 297.3 -> 355.5 mm, vias 5 -> 7
- net RST: track 41.3 -> 52.9 mm
Other:
- board text added: "211515873"
- board text added: "Hall Effect Sensors"
- board text added: "Motor"
- board text added: "SMPS Regulator"
- board text added: "Speed Board V1"
- board text added: "Terayza Eldridge"
- board text added: "Vin"
- board text added: "Vout"
Changed lines of the file:
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@@
 <setting verticaltext="up"/>
 </settings>
-<grid distance="0.4" unitdist="mil" unit="mil" style="lines" multiple="1" display="yes" altdistance="0.01" altunitdist="mm" altunit="mm"/>
+<grid distance="0.05" unitdist="inch" unit="mm" style="lines" multiple="1" display="no" altdistance="0.025" altunitdist="inch" altunit="mm"/>
 <layers>
 <layer number="1" name="Top" color="4" fill="1" visible="yes" active="yes"/>
@@
 <hole x="77" y="3" drill="3.2"/>
 <hole x="3" y="3" drill="3.2"/>
-<wire x1="0" y1="-1" x2="0" y2="71" width="0.254" layer="249"/>
-<wire x1="-1" y1="70" x2="71" y2="70" width="0.254" layer="249"/>
-<wire x1="70" y1="71" x2="70" y2="-1" width="0.254" layer="249"/>
-<wire x1="71" y1="0" x2="-1" y2="0" width="0.254" layer="249"/>
+<wire x1="0" y1="-1" x2="0.030478125" y2="80.93648125" width="0.254" layer="249"/>
+<wire x1="-1.365759375" y1="80.13968125" x2="81.49528125" y2="79.9568" width="0.254" layer="249"/>
+<wire x1="80.099040625" y1="80.93648125" x2="79.936478125" y2="-1.467359375" width="0.254" layer="249"/>
+<wire x1="80.67231875" y1="-0.02031875" x2="-1" y2="0" width="0.254" layer="249"/>
 <rectangle x1="45.91811875" y1="3.672840625" x2="45.928275" y2="3.682996875" layer="200"/>
 <rectangle x1="46.009559375" y1="3.672840625" x2="46.060359375" y2="3.682996875" layer="200"/>
@@
 <rectangle x1="46.517559375" y1="15.427959375" x2="46.537878125" y2="15.438115625" layer="200"/>
 <text x="0" y="-0.0508" size="0.02031875" layer="200" font="vector">C:/Users/Terayza/Desktop/teacup.bmp</text>
+<text x="47.1932" y="69.32168125" size="1.778" layer="1" rot="R180">SMPS Regulator</text>
+<text x="24.6888" y="77.815440625" size="1.778" layer="1" rot="R180">Vin</text>
+<text x="56.11368125" y="77.38871875" size="1.778" layer="1" rot="R180">Vout</text>
+<text x="72.349359375" y="73.345040625" size="1.778" layer="1" rot="R270">Terayza Eldridge</text>
+<text x="75.478640625" y="68.1736" size="1.778" layer="1" rot="R270">211515873</text>
+<text x="1.6764" y="73.365359375" size="1.778" layer="1" rot="R270">Speed Board V1</text>
+<text x="77.24648125" y="50.6984" size="1.778" layer="1" rot="R270">Hall Effect Sensors</text>
+<text x="77.459840625" y="22.565359375" size="1.778" layer="1" rot="R270">Motor</text>
 </plain>
 <attributes>
@@
 <contactref element="C8" pad="1"/>
 <contactref element="OK1" pad="3"/>
-<wire x1="40.513" y1="33.401" x2="40.64" y2="33.401" width="0" layer="19" extent="1-16"/>
-<wire x1="40.64" y1="33.401" x2="41.656" y2="32.385" width="0" layer="19" extent="1-16"/>
-<wire x1="41.656" y1="32.385" x2="41.656" y2="28.194" width="0.4064" layer="1"/>
+<wire x1="41.656" y1="32.385" x2="41.656" y2="31.75" width="0.4064" layer="1"/>
+<wire x1="41.656" y1="31.75" x2="41.656" y2="28.194" width="0.4064" layer="1"/>
 <wire x1="41.656" y1="23.114" x2="41.656" y2="28.194" width="0.4064" layer="1"/>
 <wire x1="39.046" y1="49.2506" x2="39.046" y2="48.063" width="0.4064" layer="1"/>
@@
 <wire x1="64.77" y1="47.498" x2="63.754" y2="48.514" width="0.4064" layer="1"/>
 <wire x1="63.754" y1="48.514" x2="53.467" y2="48.514" width="0.4064" layer="1"/>
-<wire x1="34.782" y1="9.906" x2="34.544" y2="10.144" width="0" layer="19" extent="1-1"/>
 <wire x1="38.735" y1="35.179" x2="38.862" y2="35.179" width="0.4064" layer="1"/>
 <wire x1="38.862" y1="35.179" x2="41.656" y2="32.385" width="0.4064" layer="1"/>
-<wire x1="41.656" y1="32.385" x2="33.2359" y2="11.9761" width="0" layer="19" extent="1-16"/>
+<wire x1="41.656" y1="32.385" x2="41.356278125" y2="32.385" width="0.4064" layer="1"/>
+<wire x1="41.356278125" y1="32.385" x2="40.10151875" y2="31.130240625" width="0.4064" layer="1"/>
+<wire x1="40.10151875" y1="31.130240625" x2="40.10151875" y2="11.5316" width="0.4064" layer="1"/>
+<wire x1="40.10151875" y1="11.5316" x2="38.160959375" y2="9.591040625" width="0.4064" layer="1"/>
+<wire x1="38.160959375" y1="9.591040625" x2="35.096959375" y2="9.591040625" width="0.4064" layer="1"/>
+<wire x1="35.096959375" y1="9.591040625" x2="34.544" y2="10.144" width="0.4064" layer="1"/>
+<wire x1="30.988" y1="33.401" x2="32.202121875" y2="33.401" width="0.4064" layer="1"/>
+<wire x1="32.202121875" y1="33.401" x2="34.16808125" y2="31.435040625" width="0.4064" layer="1"/>
+<wire x1="34.16808125" y1="31.435040625" x2="34.16808125" y2="25.389840625" width="0.4064" layer="1"/>
+<wire x1="34.16808125" y1="25.389840625" x2="34.1376" y2="25.359359375" width="0.4064" layer="1"/>
+<via x="34.1376" y="25.359359375" extent="1-16" drill="0.9"/>
+<wire x1="34.1376" y1="25.359359375" x2="34.1376" y2="24.9021625" width="0.4064" layer="16"/>
+<wire x1="34.1376" y1="24.9021625" x2="34.62528125" y2="24.41448125" width="0.4064" layer="16"/>
+<wire x1="34.62528125" y1="24.41448125" x2="44.419521875" y2="24.41448125" width="0.4064" layer="16"/>
+<wire x1="44.419521875" y1="24.41448125" x2="44.9072" y2="24.902159375" width="0.4064" layer="16"/>
+<via x="44.9072" y="24.902159375" extent="1-16" drill="0.9"/>
+<wire x1="44.9072" y1="24.902159375" x2="44.9072" y2="28.4988" width="0.4064" layer="1"/>
+<wire x1="44.9072" y1="28.4988" x2="41.656" y2="31.75" width="0.4064" layer="1"/>
+<wire x1="60.452" y1="10.922" x2="60.512" y2="10.818" width="0" layer="19" extent="1-1"/>
+<wire x1="13.589" y1="8.509" x2="17.272" y2="4.384" width="0" layer="19" extent="1-1"/>
+<wire x1="25.08" y1="54.229" x2="37.446" y2="50.273" width="0" layer="19" extent="1-1"/>
+<wire x1="6.6" y1="31.97" x2="6.589" y2="15.466" width="0" layer="19" extent="1-1"/>
 </signal>
 <signal name="VCC">
@@
 <wire x1="34.163" y1="48.768" x2="27.305" y2="48.768" width="0.4064" layer="1"/>
 <wire x1="27.305" y1="48.768" x2="25.908" y2="47.371" width="0.4064" layer="1"/>
-<wire x1="25.908" y1="47.371" x2="25.908" y2="42.586" width="0.4064" layer="1"/>
+<wire x1="25.908" y1="47.371" x2="25.908" y2="46.99" width="0.4064" layer="1"/>
 <contactref element="U$3" pad="18"/>
 <contactref element="C6" pad="2"/>
@@
 <contactref element="U2" pad="3"/>
 <contactref element="R7" pad="1"/>
+<wire x1="25.908" y1="46.99" x2="25.908" y2="42.586" width="0.4064" layer="1"/>
 <wire x1="11.5062" y1="9.779" x2="13.335" y2="9.779" width="0.4064" layer="1"/>
 <wire x1="13.335" y1="9.779" x2="13.589" y2="10.033" width="0.4064" layer="1"/>
@@
 <wire x1="34.544" y1="13.462" x2="36.002" y2="13.462" width="0.4064" layer="1"/>
 <wire x1="36.002" y1="13.462" x2="36.068" y2="13.528" width="0.4064" layer="1"/>
-<wire x1="37.273" y1="38.177" x2="49.911" y2="35.814" width="0" layer="19" extent="1-16"/>
-<wire x1="36.068" y1="13.528" x2="53.721" y2="24.765" width="0" layer="19" extent="1-1"/>
+<wire x1="36.068" y1="13.528" x2="36.388" y2="13.528" width="0.4064" layer="1"/>
+<wire x1="36.388" y1="13.528" x2="38.1" y2="15.24" width="0.4064" layer="1"/>
+<via x="38.1" y="15.24" extent="1-16" drill="0.8" shape="square"/>
+<wire x1="38.1" y1="15.24" x2="43.18" y2="15.24" width="0.4064" layer="16"/>
+<wire x1="43.18" y1="15.24" x2="49.53" y2="21.59" width="0.4064" layer="16"/>
+<wire x1="49.53" y1="21.59" x2="49.53" y2="30.734" width="0.4064" layer="16"/>
+<wire x1="49.53" y1="30.734" x2="49.911" y2="31.115" width="0.4064" layer="16"/>
+<wire x1="49.911" y1="35.814" x2="49.911" y2="47.879" width="0.4064" layer="16"/>
+<wire x1="49.911" y1="47.879" x2="46.99" y2="50.8" width="0.4064" layer="16"/>
+<wire x1="46.99" y1="50.8" x2="26.67" y2="50.8" width="0.4064" layer="16"/>
+<wire x1="26.67" y1="50.8" x2="25.4" y2="49.53" width="0.4064" layer="16"/>
+<via x="25.4" y="49.53" extent="1-16" drill="0.8" shape="square"/>
+<wire x1="25.4" y1="49.53" x2="25.4" y2="47.498" width="0.4064" layer="1"/>
+<wire x1="25.4" y1="47.498" x2="25.908" y2="46.99" width="0.4064" layer="1"/>
 </signal>
 <signal name="PD2">
@@
 <wire x1="45.593" y1="38.862" x2="37.592" y2="30.861" width="0.6096" layer="16"/>
 <via x="37.592" y="30.861" extent="1-16" drill="0.9"/>
-<wire x1="37.592" y1="30.861" x2="30.988" y2="30.861" width="0.4064" layer="1"/>
 <wire x1="37.592" y1="30.861" x2="37.592" y2="28.448" width="0.4064" layer="1"/>
 <wire x1="37.592" y1="28.448" x2="37.846" y2="28.194" width="0.4064" layer="1"/>
@@
 <wire x1="37.273" y1="36.277" x2="37.273" y2="31.18" width="0.4064" layer="1"/>
 <wire x1="37.273" y1="31.18" x2="37.592" y2="30.861" width="0.4064" layer="1"/>
+<wire x1="30.988" y1="30.861" x2="30.988" y2="26.476959375" width="0.4064" layer="1"/>
+<wire x1="30.988" y1="26.476959375" x2="33.995359375" y2="23.4696" width="0.4064" layer="1"/>
+<wire x1="33.995359375" y1="23.4696" x2="35.2552" y2="23.4696" width="0.4064" layer="1"/>
+<wire x1="35.2552" y1="23.4696" x2="36.34231875" y2="24.55671875" width="0.4064" layer="1"/>
+<wire x1="36.34231875" y1="24.55671875" x2="36.34231875" y2="29.61131875" width="0.4064" layer="1"/>
+<wire x1="36.34231875" y1="29.61131875" x2="37.592" y2="30.861" width="0.4064" layer="1"/>
 </signal>
 <signal name="N$5">

Commit message: Updates
Routing:
- net GND: track 355.5 -> 440.4 mm, vias 7 -> 9
- net CANSTBY: track 12.8 -> 16.5 mm
- net N$5: track 14.5 -> 17.0 mm
- net RXCAN: track 33.6 -> 36.0 mm
- net N$6: track 14.9 -> 17.2 mm
Changed lines of the file:
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@@
 <vertex x="0" y="80"/>
 </polygon>
-<wire x1="11.5062" y1="8.509" x2="13.589" y2="8.509" width="0.4064" layer="1"/>
 <wire x1="13.589" y1="8.509" x2="14.732" y2="9.652" width="0.4064" layer="1"/>
 <wire x1="13.081" y1="14.113" x2="13.319" y2="14.113" width="0.4064" layer="1"/>
@@
 <wire x1="44.9072" y1="24.902159375" x2="44.9072" y2="28.4988" width="0.4064" layer="1"/>
 <wire x1="44.9072" y1="28.4988" x2="41.656" y2="31.75" width="0.4064" layer="1"/>
+<wire x1="6.589" y1="15.466" x2="6.589" y2="15.479" width="0.4064" layer="1"/>
+<wire x1="6.589" y1="15.479" x2="19.05" y2="27.94" width="0.4064" layer="1"/>
+<wire x1="19.05" y1="27.94" x2="19.05" y2="50.419" width="0.4064" layer="1"/>
+<wire x1="19.05" y1="50.419" x2="22.86" y2="54.229" width="0.4064" layer="1"/>
+<wire x1="6.6" y1="31.97" x2="4.86" y2="31.97" width="0.8128" layer="16"/>
+<wire x1="4.86" y1="31.97" x2="3.81" y2="33.02" width="0.8128" layer="16"/>
+<wire x1="3.81" y1="33.02" x2="3.81" y2="50.09" width="0.8128" layer="16"/>
+<wire x1="3.81" y1="50.09" x2="6.6" y2="52.88" width="0.8128" layer="16"/>
+<wire x1="17.272" y1="4.384" x2="17.272" y2="3.302" width="0.4064" layer="1"/>
+<wire x1="17.272" y1="3.302" x2="16.51" y2="2.54" width="0.4064" layer="1"/>
+<via x="16.51" y="2.54" extent="1-16" drill="0.6" shape="square"/>
+<wire x1="16.51" y1="2.54" x2="13.97" y2="2.54" width="0.4064" layer="16"/>
+<wire x1="13.97" y1="2.54" x2="11.43" y2="5.08" width="0.4064" layer="16"/>
+<via x="11.43" y="5.08" extent="1-16" drill="0.6" shape="square"/>
+<wire x1="11.43" y1="5.08" x2="9.704753125" y2="5.08" width="0.4064" layer="1"/>
+<wire x1="11.5062" y1="8.509" x2="9.71898125" y2="8.509" width="0.4064" layer="1"/>
+<wire x1="9.71898125" y1="8.509" x2="9.704753125" y2="5.08" width="0.4064" layer="1"/>
 <wire x1="60.452" y1="10.922" x2="60.512" y2="10.818" width="0" layer="19" extent="1-1"/>
-<wire x1="13.589" y1="8.509" x2="17.272" y2="4.384" width="0" layer="19" extent="1-1"/>
-<wire x1="25.08" y1="54.229" x2="37.446" y2="50.273" width="0" layer="19" extent="1-1"/>
-<wire x1="6.6" y1="31.97" x2="6.589" y2="15.466" width="0" layer="19" extent="1-1"/>
+<wire x1="13.589" y1="8.509" x2="11.5062" y2="8.509" width="0.4064" layer="1"/>
 </signal>
 <signal name="VCC">
@@
 <wire x1="22.606" y1="14.478" x2="23.368" y2="13.716" width="0.4064" layer="1"/>
 <wire x1="23.368" y1="13.716" x2="23.368" y2="11.9761" width="0.4064" layer="1"/>
-<wire x1="23.368" y1="11.9761" x2="23.368" y2="9.652" width="0.4064" layer="1"/>
-<wire x1="23.368" y1="9.652" x2="22.098" y2="8.382" width="0.4064" layer="1"/>
-<wire x1="11.5062" y1="11.049" x2="9.271" y2="11.049" width="0.4064" layer="1"/>
-<wire x1="9.271" y1="11.049" x2="9.144" y2="10.922" width="0.4064" layer="1"/>
-<wire x1="9.144" y1="10.922" x2="9.144" y2="6.35" width="0.4064" layer="1"/>
-<wire x1="9.144" y1="6.35" x2="9.906" y2="5.588" width="0.4064" layer="1"/>
-<wire x1="9.906" y1="5.588" x2="13.716" y2="5.588" width="0.4064" layer="1"/>
-<wire x1="13.716" y1="5.588" x2="16.51" y2="8.382" width="0.4064" layer="1"/>
-<wire x1="16.51" y1="8.382" x2="22.098" y2="8.382" width="0.4064" layer="1"/>
+<wire x1="11.5062" y1="11.049" x2="9.779" y2="11.049" width="0.4064" layer="1"/>
+<wire x1="9.779" y1="11.049" x2="8.89" y2="10.16" width="0.4064" layer="1"/>
+<wire x1="8.89" y1="10.16" x2="8.89" y2="5.08" width="0.4064" layer="1"/>
+<wire x1="8.89" y1="5.08" x2="10.16" y2="3.81" width="0.4064" layer="1"/>
+<wire x1="10.16" y1="3.81" x2="12.7" y2="3.81" width="0.4064" layer="1"/>
+<wire x1="12.7" y1="3.81" x2="13.97" y2="5.08" width="0.4064" layer="1"/>
+<wire x1="13.97" y1="5.08" x2="13.97" y2="6.35" width="0.4064" layer="1"/>
+<wire x1="13.97" y1="6.35" x2="16.51" y2="8.89" width="0.4064" layer="1"/>
+<wire x1="16.51" y1="8.89" x2="21.59" y2="8.89" width="0.4064" layer="1"/>
+<wire x1="21.59" y1="8.89" x2="23.368" y2="10.668" width="0.4064" layer="1"/>
+<wire x1="23.368" y1="11.9761" x2="23.368" y2="10.668" width="0.4064" layer="1"/>
 </signal>
 <signal name="TXCAN">
@@
 <contactref element="U2" pad="8"/>
 <contactref element="R8" pad="1"/>
-<wire x1="17.272" y1="6.284" x2="16.19" y2="6.284" width="0.4064" layer="1"/>
-<wire x1="16.19" y1="6.284" x2="14.478" y2="4.572" width="0.4064" layer="1"/>
-<wire x1="14.478" y1="4.572" x2="8.9408" y2="4.572" width="0.4064" layer="1"/>
-<wire x1="8.9408" y1="4.572" x2="6.2738" y2="7.239" width="0.4064" layer="1"/>
+<wire x1="17.272" y1="6.284" x2="16.444" y2="6.284" width="0.4064" layer="1"/>
+<wire x1="16.444" y1="6.284" x2="12.7" y2="2.54" width="0.4064" layer="1"/>
+<wire x1="12.7" y1="2.54" x2="7.62" y2="2.54" width="0.4064" layer="1"/>
+<wire x1="7.62" y1="2.54" x2="6.35" y2="3.81" width="0.4064" layer="1"/>
+<wire x1="6.35" y1="3.81" x2="6.35" y2="7.1628" width="0.4064" layer="1"/>
+<wire x1="6.35" y1="7.1628" x2="6.2738" y2="7.239" width="0.4064" layer="1"/>
 </signal>
 <signal name="CANH">
@@
 <contactref element="U3" pad="7"/>
 <contactref element="C3" pad="2"/>
-<wire x1="44.831" y1="56.703" x2="38.161" y2="56.068" width="0.4064" layer="1"/>
-<wire x1="38.161" y1="56.068" x2="37.211" y2="55.118" width="0.4064" layer="1"/>
 <wire x1="35.846" y1="49.2506" x2="35.846" y2="53.753" width="0.4064" layer="1"/>
-<wire x1="35.846" y1="53.753" x2="37.211" y2="55.118" width="0.4064" layer="1"/>
 <contactref element="Q4" pad="2"/>
-<wire x1="39.497" y1="55.118" x2="35.846" y2="49.2506" width="0" layer="19" extent="1-1"/>
+<wire x1="39.497" y1="55.118" x2="37.211" y2="55.118" width="0.4064" layer="1"/>
+<wire x1="37.211" y1="55.118" x2="36.7665" y2="54.6735" width="0.4064" layer="1"/>
+<wire x1="36.7665" y1="54.6735" x2="35.846" y2="53.753" width="0.4064" layer="1"/>
+<wire x1="44.831" y1="56.703" x2="38.796" y2="56.703" width="0.4064" layer="1"/>
+<wire x1="38.796" y1="56.703" x2="37.211" y2="55.118" width="0.4064" layer="1"/>
 </signal>
 <signal name="N$6">
@@
 <wire x1="31.054" y1="56.195" x2="32.131" y2="55.118" width="0.4064" layer="1"/>
 <wire x1="35.046" y1="49.2506" x2="35.046" y2="52.203" width="0.4064" layer="1"/>
-<wire x1="35.046" y1="52.203" x2="32.131" y2="55.118" width="0.4064" layer="1"/>
+<wire x1="35.046" y1="52.203" x2="34.7345" y2="52.5145" width="0.4064" layer="1"/>
 <contactref element="Q4" pad="1"/>
-<wire x1="29.845" y1="55.118" x2="35.046" y2="49.2506" width="0" layer="19" extent="1-1"/>
+<wire x1="29.845" y1="55.118" x2="32.131" y2="55.118" width="0.4064" layer="1"/>
+<wire x1="32.131" y1="55.118" x2="34.7345" y2="52.5145" width="0.4064" layer="1"/>
 </signal>
 <signal name="HE1">

Commit message: Terayzas PCBS etched...
Parts:
- added U$5, U$8, U$9: MMBZ5V6ALT1G, RobThePyro:SOT23
- moved C1 31.5 mm to (43.7, 52.2), turned to 90 degrees
- moved C9 21.4 mm to (37.2, 38.2), turned to 180 degrees
- moved R16 6.65 mm to (54.2, 35.6)
- moved S4 2.75 mm to (40.1, 28.4)
- moved R1 2.71 mm to (38.2, 34.7)
- moved C2 1.56 mm to (24.4, 56.8), turned to 0 degrees
- moved R9 1.17 mm to (75.2, 25.9)
- moved C3 1.02 mm to (44.9, 56.8), turned to 180 degrees
Connections:
- net A0: now also U$9.2
- net A1: now also U$9.1
- net GND: now also U$5.3, U$8.3, U$9.3
- net HE1: now also U$5.2
- net HE2: now also U$5.1
- net VCC: now also U$8.1, U$8.2
Routing:
- net GND: track 440.4 -> 197.1 mm, vias 9 -> 6
- net VCC: track 242.2 -> 330.9 mm, vias 6 -> 0
- net RST: track 52.9 -> 41.8 mm
- net HE1: track 27.3 -> 35.1 mm
- net A1: track 64.1 -> 69.2 mm
- net N$11: track 8.52 -> 11.9 mm
- net N$6: track 17.2 -> 14.5 mm
- net N$5: track 17.0 -> 14.9 mm
- net HE2: track 24.1 -> 26.0 mm
- net N$3: track 13.9 -> 12.1 mm
- net A0IN: track 8.32 -> 7.58 mm
- net A0: track 31.1 -> 31.9 mm
- net N$4: track 5.80 -> 5.13 mm
Other:
- board text added: "HE1"
- board text added: "HE2"
- board text added: "INT"
- board text added: "MTSPD"
- board text added: "RST"
- board text removed: "C:/Users/Terayza/Desktop/teacup.bmp"
- board text removed: "Hall Effect Sensors"
- board text removed: "Motor"

Commit message: Working
Parts:
- added U$10: HEADER-5WAY, con-TE-EP:1744426-5
Connections:
- removed net N$11: S1.2, U3.27
- new net INT: U$10.P$1
- new net SCL: U$10.P$3, U3.28
- new net SDA: U$10.P$2, U3.27
- net GND: now also U$10.P$4, U3.19
- net VCC: now also U$10.P$5
Routing:
- net N$11: track 11.9 -> 0.00 mm

Commit message: Terayza Work
Parts:
- moved U$10 104.2 mm to (99.5, 35.5), turned to 90 degrees
Changed lines of the file:
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@@
 <element name="U$8" library="RobThePyro" package="SOT23" value="MMBZ5V6ALT1G" x="63.3095" y="61.087" rot="R180"/>
 <element name="U$9" library="RobThePyro" package="SOT23" value="MMBZ5V6ALT1G" x="52.7685" y="23.1775" rot="R90"/>
-<element name="U$10" library="con-TE-EP" package="1744426-5" value="HEADER-5WAY" x="6.5" y="-11.5"/>
+<element name="U$10" library="con-TE-EP" package="1744426-5" value="HEADER-5WAY" x="99.5" y="35.5" rot="R90"/>
 </elements>
 <signals>
@@
 <contactref element="U$10" pad="P$4"/>
 <contactref element="U3" pad="19"/>
-<wire x1="50.199" y1="51.247" x2="53.467" y2="50.546" width="0" layer="19" extent="1-1"/>
+<wire x1="67.16" y1="32.552" x2="93" y2="38" width="0" layer="19" extent="1-1"/>
 <wire x1="36.646" y1="40.6654" x2="38.227" y2="40.6844" width="0" layer="19" extent="1-1"/>
+<wire x1="53.467" y1="50.546" x2="50.199" y2="51.247" width="0" layer="19" extent="1-1"/>
 <wire x1="53.467" y1="46.736" x2="53.467" y2="50.546" width="0" layer="19" extent="1-1"/>
-<wire x1="9" y1="-5" x2="17.272" y2="4.384" width="0" layer="19" extent="1-1"/>
 </signal>
 <signal name="VCC">
@@
 <wire x1="77.47" y1="29.2735" x2="76.0095" y2="30.734" width="0.8128" layer="1"/>
 <contactref element="U$10" pad="P$5"/>
-<wire x1="11.5" y1="-5" x2="11.5062" y2="9.779" width="0" layer="19" extent="1-1"/>
+<wire x1="76.1365" y1="48.8315" x2="93" y2="40.5" width="0" layer="19" extent="1-1"/>
 </signal>
 <signal name="PD2">
@@
 <contactref element="U$10" pad="P$3"/>
 <contactref element="U3" pad="28"/>
-<wire x1="6.5" y1="-5" x2="42.1386" y2="44.558" width="0" layer="19" extent="1-1"/>
+<wire x1="42.1386" y1="44.558" x2="93" y2="35.5" width="0" layer="19" extent="1-1"/>
 </signal>
 <signal name="SDA">
 <contactref element="U$10" pad="P$2"/>
 <contactref element="U3" pad="27"/>
-<wire x1="4" y1="-5" x2="42.1386" y2="43.758" width="0" layer="19" extent="1-1"/>
+<wire x1="42.1386" y1="43.758" x2="93" y2="33" width="0" layer="19" extent="1-1"/>
 </signal>
 <signal name="INT">

Commit message: Thingies
Connections:
- new net N$11: U3.12
Changed lines of the file:
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@@
 <contactref element="U$10" pad="P$1"/>
+</signal>
+<signal name="N$11">
+<contactref element="U3" pad="12"/>
 </signal>
 </signals>

Commit message: Board things
Parts:
- added U$11, U$12: MMBZ5V6ALT1G, RobThePyro:SOT23
- added U$13: HEADER-3WAY, con-TE-EP:1744426-3
- moved U$10 25.7 mm to (74.0, 38.5)
- moved U$1 17.5 mm to (74.2, 52.6)
- moved U$2 17.5 mm to (74.2, 63.7)
- moved F1 13.4 mm to (74.2, 71.7), turned to 0 degrees
- moved U$8 11.4 mm to (67.8, 71.6)
- moved U$5 10.0 mm to (61.8, 50.8)
- moved R3 10.0 mm to (61.8, 45.1)
- moved R4 9.00 mm to (61.7, 55.2)
- moved S1 4.53 mm to (50.4, 53.1)
- moved R16 2.50 mm to (51.7, 35.6)
- moved LED4 1.66 mm to (49.1, 41.4)
- moved LED5 1.53 mm to (49.3, 39.6)
- moved R11 1.52 mm to (53.2, 39.6)
- moved R10 1.14 mm to (53.2, 41.9)
- moved C1 0.50 mm to (43.7, 52.7)
Connections:
- new net RXD: U$13.P$3, U3.30
- new net TXD: U$13.P$2, U3.31
- net GND: now also U$11.3, U$12.3, U$13.P$1; no longer S1.1, U3.19
- net INT: now also U$12.1, U3.9
- net MTSPD: now also U3.12; no longer U3.30
- net N$11: now also S1.1, S1.2, U3.2; no longer U3.12
- net SCL: now also U$10.P$2, U$11.1; no longer U$10.P$3
- net SDA: now also U$10.P$3, U$11.2; no longer U$10.P$2
Routing:
- net INT: track 0.00 -> 52.1 mm, vias 0 -> 2
- net SDA: track 0.00 -> 46.1 mm
- net TXD: track 0.00 -> 44.7 mm, vias 0 -> 1
- net RXD: track 0.00 -> 40.7 mm, vias 0 -> 1
- net SCL: track 0.00 -> 33.0 mm
- net GND: track 197.1 -> 226.2 mm, vias 6 -> 7
- net VCC: track 330.9 -> 349.0 mm
- net MTSPD: track 38.1 -> 53.0 mm, vias 0 -> 2
- net N$11: track 0.00 -> 14.3 mm
- net FUSEDVCC: track 59.0 -> 71.1 mm
- net HE1: track 35.1 -> 24.8 mm
- net PD2: track 4.36 -> 14.4 mm
- net PD3: track 4.49 -> 12.7 mm
- net HE2: track 26.0 -> 27.3 mm
- net RST: track 41.8 -> 42.7 mm
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Other:
- board text added: "MPU6050"
- board text added: "RXD"
- board text added: "TXD"
