File: Eagle Projects/Terayza/D3/Speed.brd (EAGLE design)
At the start: 80 x 80 mm, 59 parts, among them Q2 16MHz, Q3 16MHz, Q4 16MHz, U2 MCP2551, U3 ATMEGA328P_TQFP, X1 5566-6, X2 5566-6

Commit message: Hack internet job using weakest internet in the world
Parts:
- removed C8: (no value), resistor:C0805
- R16: value 10K -> 1K
Connections:
- net GND: no longer C8.1
- net MTSPD: no longer C8.2
Routing:
- net GND: track 226.2 -> 221.8 mm
Changed lines of the file:
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@@
 </element>
 <element name="U$4" library="RobThePyro" package="SMPSBOARD" value="SMPSBOARD" x="17.176" y="58.724"/>
-<element name="C8" library="resistor" package="C0805" value="" x="58.674" y="27.051" rot="R270"/>
 <element name="U$6" library="con-TE-EP" package="1744426-2" value="HEADER-2WAY" x="73.914" y="19.304" rot="R90"/>
 <element name="R9" library="resistor" package="M0805" value="680E" x="75.184" y="25.908" rot="R90"/>
@@
 <attribute name="OC_FARNELL" value="unknown" x="66.802" y="26.924" size="1.778" layer="27" rot="R90" display="off"/>
 </element>
-<element name="R16" library="resistor" package="M0805" value="10K" x="51.6655" y="35.6235" rot="R90"/>
+<element name="R16" library="resistor" package="M0805" value="1K" x="51.6655" y="35.6235" rot="R90"/>
 <element name="D1" library="diode" package="SMB" value="" x="25.908" y="40.386" rot="R270"/>
 <element name="Q4" library="crystal" package="HC49UP" value="16MHz" x="34.671" y="55.118">
@@
 <contactref element="R15" pad="1"/>
 <contactref element="R14" pad="1"/>
-<contactref element="C8" pad="1"/>
 <contactref element="OK1" pad="3"/>
 <wire x1="38.227" y1="47.244" x2="38.227" y2="40.6844" width="0.4064" layer="1"/>
@@
 <contactref element="S1" pad="4"/>
 <contactref element="S1" pad="3"/>
-<wire x1="62.992" y1="28.194" x2="58.867" y2="28.194" width="0.4064" layer="1"/>
-<wire x1="58.867" y1="28.194" x2="58.674" y2="28.001" width="0.4064" layer="1"/>
 <wire x1="38.989" y1="49.3076" x2="39.046" y2="49.2506" width="0.4064" layer="1"/>
 <wire x1="55.753" y1="16.703" x2="52.578" y2="16.703" width="0.4064" layer="1"/>
@@
 <contactref element="R16" pad="1"/>
 <contactref element="OK1" pad="4"/>
-<contactref element="C8" pad="2"/>
-<wire x1="62.992" y1="25.654" x2="58.674" y2="25.654" width="0.4064" layer="1"/>
-<wire x1="58.674" y1="25.654" x2="58.674" y2="26.101" width="0.4064" layer="1"/>
-<wire x1="58.674" y1="26.101" x2="57.592" y2="26.101" width="0.4064" layer="1"/>
-<wire x1="51.6655" y1="32.0275" x2="57.592" y2="26.101" width="0.4064" layer="1"/>
+<wire x1="51.6655" y1="32.0275" x2="58.039" y2="25.654" width="0.4064" layer="1"/>
 <contactref element="U3" pad="12"/>
 <wire x1="51.6655" y1="34.6735" x2="48.8265" y2="34.6735" width="0.4064" layer="1"/>
@@
 <wire x1="33.4114" y1="45.5" x2="33.5534" y2="45.358" width="0.4064" layer="1"/>
 <wire x1="51.6655" y1="34.6735" x2="51.6655" y2="32.0275" width="0.4064" layer="1"/>
+<wire x1="62.992" y1="25.654" x2="58.039" y2="25.654" width="0.4064" layer="1"/>
 </signal>
 <signal name="N$7">
