File: Eagle Projects/Terayza/D3/MPU.sch (EAGLE design)
At the start: 10 parts, among them U1 ATMEGA328P-AU

Commit message: Added connectors for T's board: *Molex x2 CAN_IN and CAN_OUT *CAN interface from Ben on Schematic *Con TE EP connector added for sensor
Parts:
- removed JP1: (no value), pinhead:PINHD-1X5
- added C3, C4: 22pF, resistor:C-EUC0805K
- added C5, C6: 100nF, resistor:C-EUC0805K
- added LED1: RX, led:LEDCHIP-LED0805
- added LED2: TX, led:LEDCHIP-LED0805
- added LED3: INT, led:LEDCHIP-LED0805
- added Q2: 16MHz, crystal:CRYSTALHC49S
- added Q3: 16MHz, crystal:CRYSTALHC49UP
- added R5, R6, R7: 1k, resistor:R-US_R0805
- added R8, R9: 100k, resistor:R-US_R0805
- added U$1: HEADER-5WAY, con-TE-EP:HEADER-5WAY
- added U$2: MCP2515SO, RobThePyro:MCP2515SO
- added U$3: SMPSBOARD, RobThePyro:SMPSBOARD
- added U2: MCP2551, SparkFun:MCP2551
- added X1, X2: 5566-6, con-molex:5566-6
- added Z1, Z2: TVS-UD-SOD323, supressor:TVS-UD-SOD323
- R1: value (none) -> 50k
Connections:
- net N$3 renamed RST
- new net +5V: C5.2, C6.2, R5.2, R6.2, R7.2, R8.1, U$2G$2.VDD, U2.VDD
- new net CANCS: U$2G$1.!CS
- new net CANH: U2.CANH, X1-1.S, X2-1.S, Z1.C
- new net CANINT: LED3.C, U$2G$1.!INT
- new net CANL: U2.CANL, X1-4.S, X2-4.S, Z2.C
- new net CANRST: R8.2, U$2G$1.!RESET
- new net CANSTBY: R9.1, U2.RS
- new net MISO: JP2.1, U$2G$1.SO, U1.PB4
- new net MOSI: JP2.4, U$2G$1.SI, U1.PB3
- new net N$13: C4.1, Q2.1, Q3.1, U$2G$1.OSC2
- new net N$3: LED3.A, R7.1
- new net RXCAN: LED1.C, U$2G$1.RXCAN, U2.RXD
- new net SCK: JP2.3, U$2G$1.SCK, U1.PB5
- new net SPARE1: X1-5.S, X2-5.S
- new net SPARE2: X1-6.S, X2-6.S
- new net TXCAN: LED2.C, U$2G$1.TXCAN, U2.TXD
- new net VIN: U$3.VIN, X1-3.S, X2-3.S
- new net VOUT: U$3.VOUT
- net GND: now also C3.2, C4.2, C5.1, C6.1, R9.2, U$1.P$4, U$2G$2.VSS, U$3.GND, U$3.GND@1, U2.VSS, X1-2.S, X2-2.S, Z1.A, Z2.A; no longer JP1.2
- net N$1: now also LED1.A, R5.1; no longer JP2.1, U1.PB4
- net N$10: now also U$1.P$3; no longer JP1.3
- net N$11: now also U$1.P$2; no longer JP1.4
- net N$12: now also U$1.P$1; no longer JP1.5
- net N$2: now also LED2.A, R6.1; no longer JP2.4, U1.PB3
- net N$4: now also C3.1, Q2.2, Q3.2, U$2G$1.OSC1; no longer JP2.3, U1.PB5
- net VCC: now also U$1.P$5; no longer JP1.1
Other:
- note added: "16MHz Crystal"
- note added: "CAN Interface"
- note added: "ICSP Header"
- note added: "MPU-6050 Header"
- note added: "SMPS Board"

Commit message: MPU almost happy
Parts:
- removed JP2: AVR-ISP-6, avr-6:AVR-ISP-6
- added ISP1: AVRISP-BOX, adafruit:AVRISP-BOX
- added U$4: HEADER-2WAY, con-TE-EP:HEADER-2WAY
Connections:
- net N$10 renamed SCL
- net N$11 renamed SDA
- net N$12 renamed INT
- new net OUTPUT: U$4.P$1, U1.PC1
- net GND: now also ISP1.GND; no longer JP2.6
- net MISO: now also ISP1.MISO; no longer JP2.1
- net MOSI: now also ISP1.MOSI; no longer JP2.4
- net RST: now also ISP1.RST; no longer JP2.5
- net SCK: now also ISP1.SCK; no longer JP2.3
- net VCC: now also ISP1.VCC; no longer JP2.2
Other:
- note added: "OUTPUT to CAN"
Changed lines of the file:
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@@
 <layer number="113" name="IDFDebug" color="4" fill="1" visible="yes" active="yes"/>
 <layer number="116" name="Patch_BOT" color="9" fill="4" visible="yes" active="yes"/>
+<layer number="118" name="Rect_Pads" color="7" fill="1" visible="no" active="no"/>
 <layer number="121" name="_tsilk" color="7" fill="1" visible="yes" active="yes"/>
 <layer number="122" name="_bsilk" color="7" fill="1" visible="yes" active="yes"/>
@@
 <layer number="230" name="230bmp" color="7" fill="1" visible="yes" active="yes"/>
 <layer number="231" name="231bmp" color="7" fill="1" visible="yes" active="yes"/>
+<layer number="232" name="Eagle3D_PG2" color="7" fill="1" visible="no" active="no"/>
+<layer number="233" name="Eagle3D_PG3" color="7" fill="1" visible="no" active="no"/>
 <layer number="248" name="Housing" color="7" fill="1" visible="yes" active="yes"/>
 <layer number="249" name="Edge" color="7" fill="1" visible="yes" active="yes"/>
@@
 <part name="SUPPLY2" library="supply2" deviceset="VCC" device=""/>
 <part name="Q1" library="crystal" deviceset="CRYSTAL" device="HC49S"/>
-<part name="JP2" library="avr-6" deviceset="AVR-ISP-6" device=""/>
 <part name="R1" library="resistor" deviceset="R-US_" device="M0805" value="50k"/>
 <part name="R2" library="resistor" deviceset="R-US_" device="M0805"/>
@@
 <part name="C2" library="resistor" deviceset="C-EU" device="C0805"/>
 <part name="SUPPLY4" library="supply2" deviceset="GND" device=""/>
-<part name="GND1" library="SparkFun-Aesthetics" deviceset="GND" device=""/>
 <part name="GND2" library="SparkFun-Aesthetics" deviceset="GND" device=""/>
 <part name="U$1" library="con-TE-EP" deviceset="HEADER-5WAY" device=""/>
@@
 <part name="GND7" library="SparkFun-Aesthetics" deviceset="GND" device=""/>
 <part name="GND8" library="SparkFun-Aesthetics" deviceset="GND" device=""/>
+<part name="U$4" library="con-TE-EP" deviceset="HEADER-2WAY" device=""/>
+<part name="ISP1" library="adafruit" deviceset="AVRISP" device="-BOX"/>
+<part name="GND9" library="SparkFun-Aesthetics" deviceset="GND" device=""/>
+<part name="SUPPLY5" library="SparkFun-Aesthetics" deviceset="VCC" device=""/>
 </parts>
 <sheets>
@@
 <wire x1="132.08" y1="35.56" x2="81.28" y2="35.56" width="0.254" layer="94"/>
 <text x="109.22" y="9.144" size="1.778" layer="94">SMPS Board</text>
+<text x="58.42" y="86.36" size="1.778" layer="91">OUTPUT to CAN</text>
 </plain>
 <instances>
@@
 <instance part="SUPPLY2" gate="G$1" x="-17.78" y="91.44"/>
 <instance part="Q1" gate="G$1" x="-48.26" y="40.64" rot="R90"/>
-<instance part="JP2" gate="G$1" x="104.14" y="88.9"/>
 <instance part="R1" gate="G$1" x="45.72" y="66.04"/>
 <instance part="R2" gate="G$1" x="53.34" y="58.42"/>
@@
 <instance part="C2" gate="G$1" x="-58.42" y="35.56" rot="R90"/>
 <instance part="SUPPLY4" gate="GND" x="-66.04" y="27.94"/>
-<instance part="GND1" gate="1" x="91.44" y="78.74"/>
 <instance part="GND2" gate="1" x="86.36" y="45.72"/>
 <instance part="U$1" gate="G$1" x="104.14" y="58.42"/>
@@
 <instance part="GND7" gate="1" x="127" y="15.24"/>
 <instance part="GND8" gate="1" x="86.36" y="15.24"/>
+<instance part="U$4" gate="G$1" x="68.58" y="81.28"/>
+<instance part="ISP1" gate="G$1" x="106.68" y="88.9" rot="MR0"/>
+<instance part="GND9" gate="1" x="86.36" y="78.74"/>
+<instance part="SUPPLY5" gate="G$1" x="86.36" y="93.98"/>
 </instances>
 <busses>
@@
 </segment>
 <segment>
-<pinref part="JP2" gate="G$1" pin="6"/>
-<pinref part="GND1" gate="1" pin="GND"/>
-<wire x1="99.06" y1="86.36" x2="91.44" y2="86.36" width="0.1524" layer="91"/>
-<wire x1="91.44" y1="86.36" x2="91.44" y2="81.28" width="0.1524" layer="91"/>
-</segment>
-<segment>
 <wire x1="99.06" y1="60.96" x2="86.36" y2="60.96" width="0.1524" layer="91"/>
 <wire x1="86.36" y1="60.96" x2="86.36" y2="48.26" width="0.1524" layer="91"/>
@@
 <pinref part="GND8" gate="1" pin="GND"/>
 <wire x1="86.36" y1="20.32" x2="86.36" y2="17.78" width="0.1524" layer="91"/>
+</segment>
+<segment>
+<pinref part="ISP1" gate="G$1" pin="GND"/>
+<pinref part="GND9" gate="1" pin="GND"/>
+<wire x1="91.44" y1="86.36" x2="86.36" y2="86.36" width="0.1524" layer="91"/>
+<wire x1="86.36" y1="86.36" x2="86.36" y2="81.28" width="0.1524" layer="91"/>
 </segment>
 </net>
@@
 </segment>
 <segment>
-<pinref part="JP2" gate="G$1" pin="2"/>
-<wire x1="99.06" y1="91.44" x2="88.9" y2="91.44" width="0.1524" layer="91"/>
-<label x="83.058" y="91.44" size="1.778" layer="95"/>
-</segment>
-<segment>
 <label x="91.44" y="63.5" size="1.778" layer="95"/>
 <pinref part="U$1" gate="G$1" pin="P$5"/>
@@
 <pinref part="SUPPLY3" gate="G$1" pin="VCC"/>
 </segment>
+<segment>
+<pinref part="ISP1" gate="G$1" pin="VCC"/>
+<pinref part="SUPPLY5" gate="G$1" pin="VCC"/>
+<wire x1="91.44" y1="91.44" x2="86.36" y2="91.44" width="0.1524" layer="91"/>
+<wire x1="86.36" y1="91.44" x2="86.36" y2="93.98" width="0.1524" layer="91"/>
+</segment>
 </net>
 <net name="RST" class="0">
@@
 </segment>
 <segment>
-<pinref part="JP2" gate="G$1" pin="5"/>
-<wire x1="99.06" y1="88.9" x2="88.9" y2="88.9" width="0.1524" layer="91"/>
-<label x="83.058" y="88.9" size="1.778" layer="95"/>
+<pinref part="ISP1" gate="G$1" pin="RST"/>
+<wire x1="119.38" y1="86.36" x2="124.46" y2="86.36" width="0.1524" layer="91"/>
 </segment>
 </net>
@@
 </segment>
 <segment>
-<pinref part="JP2" gate="G$1" pin="1"/>
-<wire x1="109.22" y1="91.44" x2="116.84" y2="91.44" width="0.1524" layer="91"/>
-<label x="118.364" y="91.44" size="1.778" layer="95"/>
+<pinref part="ISP1" gate="G$1" pin="MISO"/>
+<wire x1="119.38" y1="91.44" x2="124.46" y2="91.44" width="0.1524" layer="91"/>
 </segment>
 </net>
 <net name="MOSI" class="0">
-<segment>
-<pinref part="JP2" gate="G$1" pin="4"/>
-<wire x1="109.22" y1="88.9" x2="116.84" y2="88.9" width="0.1524" layer="91"/>
-<label x="118.11" y="88.9" size="1.778" layer="95"/>
-</segment>
 <segment>
 <pinref part="U1" gate="A" pin="PB3"/>
@@
 <label x="-16.51" y="50.8" size="1.778" layer="95"/>
 </segment>
+<segment>
+<pinref part="ISP1" gate="G$1" pin="MOSI"/>
+<wire x1="91.44" y1="88.9" x2="86.36" y2="88.9" width="0.1524" layer="91"/>
+</segment>
 </net>
 <net name="SCK" class="0">
@@
 </segment>
 <segment>
-<pinref part="JP2" gate="G$1" pin="3"/>
-<wire x1="109.22" y1="86.36" x2="116.84" y2="86.36" width="0.1524" layer="91"/>
-<label x="118.11" y="86.36" size="1.778" layer="95"/>
+<pinref part="ISP1" gate="G$1" pin="SCK"/>
+<wire x1="119.38" y1="88.9" x2="124.46" y2="88.9" width="0.1524" layer="91"/>
 </segment>
 </net>
@@
 </segment>
 </net>
-<net name="N$10" class="0">
+<net name="SCL" class="0">
 <segment>
 <wire x1="99.06" y1="58.42" x2="58.42" y2="58.42" width="0.1524" layer="91"/>
@@
 </segment>
 </net>
-<net name="N$11" class="0">
+<net name="SDA" class="0">
 <segment>
 <wire x1="99.06" y1="55.88" x2="58.42" y2="55.88" width="0.1524" layer="91"/>
@@
 </segment>
 </net>
-<net name="N$12" class="0">
+<net name="INT" class="0">
 <segment>
 <wire x1="99.06" y1="53.34" x2="58.42" y2="53.34" width="0.1524" layer="91"/>
@@
 </segment>
 </net>
+<net name="OUTPUT" class="0">
+<segment>
+<pinref part="U1" gate="A" pin="PC1"/>
+<wire x1="33.02" y1="78.74" x2="63.5" y2="78.74" width="0.1524" layer="91"/>
+<pinref part="U$4" gate="G$1" pin="P$1"/>
+</segment>
+</net>

Commit message: Updates
Parts:
- removed ISP1: AVRISP-BOX, adafruit:AVRISP-BOX
- removed U$4: HEADER-2WAY, con-TE-EP:HEADER-2WAY
- removed U1: ATMEGA328P-AU, Atmel_By_element14_Batch_1-00:ATMEGA328P-AU
- added C7, C8: 100nF, resistor:C-EUC0805
- added JP1: AVR-ISP6-75869-131, atmel-avr:AVR-ISP6-75869-131
- added LED4, LED5: (no value), led:LEDCHIP-LED0805
- added Q4: (no value), special:XTAL/S
- added R10, R12: 560E, resistor:R-US_M0805
- added S1, S2: (no value), SparkFun:TAC_SWITCHSMD
- added U3: ATMEGA328P_TQFP, SparkFun-DigitalIC:ATMEGA328P_TQFP
- Q1: device crystal:CRYSTALHC49S -> crystal:CRYSTALHC49UP
Connections:
- removed net OUTPUT: U$4.P$1, U1.PC1
- removed net VCC: ISP1.VCC, R1.2, U$1.P$5, U1.AREF, U1.AVCC, U1.VCC, U1.VCC_2
- new net CANINIT: U3.PB1(OC1A)
- new net N$10: S2.1, S2.2, U3.PD5(T1)
- new net N$11: R1.2, U3.PC6(/RESET)
- new net N$12: LED4.A, R10.1
- new net N$14: LED5.A, R12.1
- new net N$15: LED4.C, U3.PC3(ADC3)
- new net N$17: C1.2, Q1.2, Q4.2, U3.PB7(XTAL2/TOSC2)
- net +5V: now also C7.2, C8.2, JP1.2, R1.1, R10.2, R12.2, U$1.P$5, U3.AREF, U3.AVCC, U3.VCC@4, U3.VCC@6
- net CANCS: now also U3.PB2(SS/OC1B)
- net GND: now also C7.1, C8.1, JP1.6, S1.3, S1.4, S2.3, S2.4, U3.AGND, U3.GND@3, U3.GND@5; no longer ISP1.GND, U1.GND, U1.GND_2, U1.GND_3
- net MISO: now also JP1.1, U3.PB4(MISO); no longer ISP1.MISO, U1.PB4
- net MOSI: now also JP1.4, U3.PB3(MOSI/OC2); no longer ISP1.MOSI, U1.PB3
- net N$5: now also U3.PC5(ADC5/SCL); no longer U1.PC5
- net N$6: now also U3.PC4(ADC4/SDA); no longer U1.PC4
- net N$7: now also U3.PD2(INT0); no longer U1.PD2
- net N$8: now also LED5.C, U3.PC2(ADC2); no longer C2.2, Q1.1, U1.PB6
- net N$9: now also C2.2, Q1.1, Q4.1, U3.PB6(XTAL1/TOSC1); no longer C1.2, Q1.2, U1.PB7
- net RST: now also JP1.5, S1.1, S1.2; no longer ISP1.RST, R1.1, U1.PC6
- net SCK: now also JP1.3, U3.PB5(SCK); no longer ISP1.SCK, U1.PB5
Other:
- note removed: "OUTPUT to CAN"
- moved on the sheet: C1, C2, Q1, R1, R2, R3, R4, U$1, U$3

Commit message: Done
Parts:
- added D1: (no value), diode:SCHOTTKY-DIODESMD
Connections:
- removed net VOUT: U$3.VOUT
- new net N$16: D1.A, JP1.2
- net +5V: now also D1.C, U$3.VOUT; no longer JP1.2
Changed lines of the file:
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@@
 <part name="SUPPLY3" library="supply2" deviceset="GND" device=""/>
 <part name="P+5" library="supply1" deviceset="+5V" device=""/>
+<part name="P+7" library="supply1" deviceset="+5V" device=""/>
+<part name="D1" library="diode" deviceset="SCHOTTKY-DIODE" device="SMD"/>
 </parts>
 <sheets>
@@
 <instance part="SUPPLY3" gate="GND" x="-17.78" y="-63.5"/>
 <instance part="P+5" gate="1" x="-25.4" y="2.54"/>
+<instance part="P+7" gate="1" x="172.72" y="-38.1"/>
+<instance part="D1" gate="G$1" x="144.78" y="-10.16"/>
 </instances>
 <busses>
@@
 </segment>
 </net>
-<net name="VOUT" class="0">
-<segment>
-<pinref part="U$3" gate="G$1" pin="VOUT"/>
-<wire x1="170.18" y1="-40.64" x2="172.72" y2="-40.64" width="0.254" layer="91"/>
-<label x="167.894" y="-39.624" size="1.778" layer="95"/>
-</segment>
-</net>
 <net name="CANCS" class="0">
 <segment>
@@
 </segment>
 <segment>
-<pinref part="JP1" gate="G$1" pin="2"/>
 <pinref part="P+9" gate="1" pin="+5V"/>
-<wire x1="139.7" y1="-10.16" x2="152.4" y2="-10.16" width="0.1524" layer="91"/>
 <wire x1="152.4" y1="-10.16" x2="152.4" y2="-2.54" width="0.1524" layer="91"/>
+<pinref part="D1" gate="G$1" pin="C"/>
+<wire x1="147.32" y1="-10.16" x2="152.4" y2="-10.16" width="0.1524" layer="91"/>
 </segment>
 <segment>
@@
 <junction x="-63.5" y="5.08"/>
 </segment>
+<segment>
+<pinref part="U$3" gate="G$1" pin="VOUT"/>
+<wire x1="170.18" y1="-40.64" x2="172.72" y2="-40.64" width="0.254" layer="91"/>
+<label x="167.894" y="-39.624" size="1.778" layer="95"/>
+<pinref part="P+7" gate="1" pin="+5V"/>
+</segment>
 </net>
 <net name="N$12" class="0">
@@
 </segment>
 </net>
+<net name="N$16" class="0">
+<segment>
+<pinref part="JP1" gate="G$1" pin="2"/>
+<pinref part="D1" gate="G$1" pin="A"/>
+<wire x1="139.7" y1="-10.16" x2="142.24" y2="-10.16" width="0.1524" layer="91"/>
+</segment>
+</net>
