File: Eagle Projects/Terayza/D3/Speed.sch (EAGLE design)
At the start: 16 parts, among them U1 ATMEGA328P-AU

Commit message: Added CAN I/O, Connectors, SMPS block to T's Speed Board
Parts:
- removed JP1, JP3: (no value), pinhead:PINHD-1X3
- added C4, C5: 22pF, resistor:C-EUC0805K
- added C6, C7: 100nF, resistor:C-EUC0805K
- added LED1: RX, led:LEDCHIP-LED0805
- added LED2: TX, led:LEDCHIP-LED0805
- added LED3: INT, led:LEDCHIP-LED0805
- added Q2: 16MHz, crystal:CRYSTALHC49S
- added Q3: 16MHz, crystal:CRYSTALHC49UP
- added R2, R5, R6: 1k, resistor:R-US_R0805
- added R7, R8: 100k, resistor:R-US_R0805
- added U$1, U$2: HEADER-3WAY, con-TE-EP:HEADER-3WAY
- added U$3: MCP2515SO, RobThePyro:MCP2515SO
- added U$4: SMPSBOARD, RobThePyro:SMPSBOARD
- added U2: MCP2551, SparkFun:MCP2551
- added X1, X2: 5566-6, con-molex:5566-6
- added Z1, Z2: TVS-UD-SOD323, supressor:TVS-UD-SOD323
Connections:
- removed net N$10: JP1.2, R3.2
- removed net N$13: JP3.2, R4.2
- new net +5V: C6.2, C7.2, R2.2, R5.2, R6.2, R7.1, U$3G$2.VDD, U2.VDD
- new net CANCS: U$3G$1.!CS
- new net CANH: U2.CANH, X1-1.S, X2-1.S, Z1.C
- new net CANINT: LED3.C, U$3G$1.!INT
- new net CANL: U2.CANL, X1-4.S, X2-4.S, Z2.C
- new net CANRST: R7.2, U$3G$1.!RESET
- new net CANSTBY: R8.1, U2.RS
- new net MISO: U$3G$1.SO
- new net MOSI: U$3G$1.SI
- new net N$15: LED1.A, R2.1
- new net N$16: LED2.A, R5.1
- new net N$17: LED3.A, R6.1
- new net N$18: C4.1, Q2.2, Q3.2, U$3G$1.OSC1
- new net N$19: C5.1, Q2.1, Q3.1, U$3G$1.OSC2
- new net PD2: R3.1, R3.2, U$1.P$2, U1.PD2
- new net PD3: R4.1, R4.2, U$2.P$2, U1.PD3
- new net RXCAN: LED1.C, U$3G$1.RXCAN, U2.RXD
- new net SCK: U$3G$1.SCK
- new net SPARE1: X1-5.S, X2-5.S
- new net SPARE2: X1-6.S, X2-6.S
- new net TXCAN: LED2.C, U$3G$1.TXCAN, U2.TXD
- new net VIN: X1-3.S, X2-3.S
- net GND: now also C4.2, C5.2, C6.1, C7.1, R8.2, U$1.P$1, U$2.P$1, U$3G$2.VSS, U$4.GND, U$4.GND@1, U2.VSS, X1-2.S, X2-2.S, Z1.A, Z2.A; no longer JP1.3, JP3.3
- net N$11: now also U$4.VIN; no longer R3.1, U1.PD2
- net N$12: now also U$4.VOUT; no longer R4.1, U1.PD3
- net VCC: now also U$1.P$3, U$2.P$3; no longer JP1.1, JP3.1
Other:
- note added: "CAN Interface"
- note added: "Hall Effect Sensor Headers"
- note added: "SMPS Header"

Commit message: Board things
Parts:
- removed C1: (no value), resistor:C-EUC0805
- removed D1: (no value), diode:DIODE-SOD110-R
- removed D2, D3: (no value), diode:ZENER-DIODESOT23
- removed JP2, JP4: (no value), pinhead:PINHD-1X1
- added C8: (no value), resistor:C-EUC0805
- added R9: (no value), resistor:R-US_M0805
- added U$5: DRTR5V0U1SO, RobThePyro:DRTR5V0U1SO
- added U$6, U$7: HEADER-2WAY, con-TE-EP:HEADER-2WAY
Connections:
- net N$4 renamed RST
- removed net N$1: C1.1, D1.C, D2.A, D3.C, U1.PB0
- removed net N$14: JP5.4, U1.PB3
- removed net N$5: JP4.1, U1.PC1
- removed net N$6: JP5.3, U1.PB5
- removed net N$9: JP5.1, U1.PB4
- new net N$4: U$7.P$1, U1.PC1
- new net PB0: R9.2, U1.PB0
- net GND: now also C8.1, U$5.GND; no longer C1.2, D3.A
- net MISO: now also JP5.1, U1.PB4
- net MOSI: now also JP5.4, U1.PB3
- net N$3: now also C8.2, R9.1, U$5.I/O, U$6.P$1; no longer D1.A, JP2.1
- net SCK: now also JP5.3, U1.PB5
- net VCC: now also U$5.VCC; no longer D2.C
Other:
- note added: "ICSP HEADER"
- note added: "Input from motor controller - rpm"
- note added: "OUTPUT from board to CAN"
- note removed: "Input from motor controller"
- note removed: "OUTPUT from board"
- moved on the sheet: JP5

Commit message: Helped with T board
Parts:
- removed JP5: AVR-ISP-6, avr-6:AVR-ISP-6
- removed U$5: DRTR5V0U1SO, RobThePyro:DRTR5V0U1SO
- removed U1: ATMEGA328P-AU, Atmel_By_element14_Batch_1-00:ATMEGA328P-AU
- added C1, C9: 100nF, resistor:C-EUC0805
- added D1: (no value), diode:SCHOTTKY-DIODESMD
- added F1: MF-MSMF014-2, adafruit:PTCFUSE-1812
- added JP1: AVR-ISP6-75869-131, atmel-avr:AVR-ISP6-75869-131
- added LED4, LED5: (no value), led:LEDCHIP-LED0805
- added OK1: LTV816, optocoupler:LTV816
- added R10, R11: 560E, resistor:R-US_M0805
- added R12, R13, R14, R15: (no value), resistor:R-US_M0805
- added R16: 10K, resistor:R-US_M0805
- added S1: BTN3, SparkFun:TAC_SWITCHSMD
- added S4: RST, SparkFun:TAC_SWITCHSMD
- added U3: ATMEGA328P_TQFP, SparkFun-DigitalIC:ATMEGA328P_TQFP
- R9: value (none) -> 680E
- U$7: value HEADER-2WAY -> HEADER-4WAY; device con-TE-EP:HEADER-2WAY -> con-TE-EP:HEADER-4WAY
Connections:
- removed net PB0: R9.2, U1.PB0
- new net A0: R12.1, R14.2, U3.PC1(ADC1)
- new net A0IN: R12.2, U$7.P$3
- new net A1: R13.1, R15.2, U3.PC0(ADC0)
- new net A1IN: R13.2, U$7.P$2
- new net FUSEDVCC: F1.1, U$1.P$3, U$2.P$3, U$7.P$4
- new net HE1: R3.1, U3.PD2(INT0)
- new net HE2: R4.1, U3.PD3(INT1)
- new net MTSPD: C8.2, OK1.COL, R16.1, U3.PD0(RXD)
- new net N$10: LED5.C, U3.PC3(ADC3)
- new net N$2: D1.A, JP1.2
- new net N$5: C3.2, Q1.2, U3.PB6(XTAL1/TOSC1)
- new net N$6: C2.2, Q1.1, U3.PB7(XTAL2/TOSC2)
- new net N$9: LED4.C, U3.PC2(ADC2)
- net CANCS: now also U3.PB2(SS/OC1B)
- net CANINT: now also U3.PB1(OC1A)
- net GND: now also C1.1, C9.1, JP1.6, OK1.EMIT, R14.1, R15.1, S1.3, S1.4, S4.3, S4.4, U$7.P$1, U3.AGND, U3.GND@3, U3.GND@5; no longer JP5.6, U$5.GND, U1.GND, U1.GND_2, U1.GND_3
- net MISO: now also JP1.1, U3.PB4(MISO); no longer JP5.1, U1.PB4
- net MOSI: now also JP1.4, U3.PB3(MOSI/OC2); no longer JP5.4, U1.PB3
- net N$11: now also S1.1, S1.2, U3.PC4(ADC4/SDA); no longer U$4.VIN
- net N$12: now also OK1.C, U$6.P$2; no longer U$4.VOUT
- net N$3: no longer C8.2, U$5.I/O
- net N$4: now also OK1.A, R9.2; no longer U$7.P$1, U1.PC1
- net N$7: now also LED4.A, R10.1; no longer C3.2, Q1.2, U1.PB7
- net N$8: now also LED5.A, R11.1; no longer C2.2, Q1.1, U1.PB6
- net PD2: no longer R3.1, U1.PD2
- net PD3: no longer R4.1, U1.PD3
- net RST: now also JP1.5, S4.1, S4.2, U3.PC6(/RESET); no longer JP5.5, U1.PC6
- net SCK: now also JP1.3, U3.PB5(SCK); no longer JP5.3, U1.PB5
- net VCC: now also C1.2, C9.2, D1.C, F1.2, R10.2, R11.2, R16.2, U$4.VOUT, U3.AREF, U3.AVCC, U3.VCC@4, U3.VCC@6; no longer JP5.2, U$1.P$3, U$2.P$3, U$5.VCC, U1.AREF, U1.AVCC, U1.VCC, U1.VCC_2
- net VIN: now also U$4.VIN
Other:
- note added: "ISOLATED"
- note removed: "OUTPUT from board to CAN"
- moved on the sheet: C2, C3, C8, Q1, R1, R3, R4, R9, U$1, U$2, U$4, U$6

Commit message: Speed basically done
Connections:
- net A0IN: now also R13.2; no longer R12.2
- net A1IN: now also R12.2; no longer R13.2
- net GND: now also S1.1
- net N$10: now also LED4.C; no longer LED5.C
- net N$11: no longer S1.1
- net N$9: now also LED5.C; no longer LED4.C
Changed lines of the file:
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@@
 <?xml version="1.0" encoding="utf-8"?>
 <!DOCTYPE eagle SYSTEM "eagle.dtd">
-<eagle version="7.2.0">
+<eagle version="6.5.0">
 <drawing>
 <settings>
@@
 </segment>
 <segment>
-<pinref part="S1" gate="S" pin="3"/>
-<pinref part="SUPPLY13" gate="GND" pin="GND"/>
-<wire x1="40.64" y1="7.62" x2="40.64" y2="2.54" width="0.1524" layer="91"/>
-<pinref part="S1" gate="S" pin="4"/>
-<wire x1="40.64" y1="5.08" x2="40.64" y2="7.62" width="0.1524" layer="91"/>
-<junction x="40.64" y="7.62"/>
-</segment>
-<segment>
 <pinref part="U$7" gate="G$1" pin="P$1"/>
 <wire x1="104.14" y1="55.88" x2="91.44" y2="55.88" width="0.1524" layer="91"/>
@@
 <wire x1="58.42" y1="27.94" x2="66.04" y2="27.94" width="0.1524" layer="91"/>
 <junction x="66.04" y="27.94"/>
+</segment>
+<segment>
+<pinref part="SUPPLY13" gate="GND" pin="GND"/>
+<pinref part="S1" gate="S" pin="4"/>
+<wire x1="40.64" y1="2.54" x2="40.64" y2="5.08" width="0.1524" layer="91"/>
+<pinref part="S1" gate="S" pin="1"/>
+<wire x1="30.48" y1="7.62" x2="30.48" y2="17.78" width="0.1524" layer="91"/>
+<wire x1="30.48" y1="17.78" x2="45.72" y2="17.78" width="0.1524" layer="91"/>
+<wire x1="45.72" y1="17.78" x2="45.72" y2="5.08" width="0.1524" layer="91"/>
+<wire x1="45.72" y1="5.08" x2="40.64" y2="5.08" width="0.1524" layer="91"/>
+<junction x="40.64" y="5.08"/>
+<wire x1="30.48" y1="7.62" x2="30.48" y2="5.08" width="0.1524" layer="91"/>
+<junction x="30.48" y="7.62"/>
+<pinref part="S1" gate="S" pin="3"/>
+<wire x1="40.64" y1="7.62" x2="40.64" y2="5.08" width="0.1524" layer="91"/>
 </segment>
 </net>
@@
 <net name="N$9" class="0">
 <segment>
-<pinref part="LED4" gate="G$1" pin="C"/>
-<wire x1="20.32" y1="35.56" x2="20.32" y2="10.16" width="0.1524" layer="91"/>
 <pinref part="U3" gate="U$1" pin="PC2(ADC2)"/>
 <wire x1="20.32" y1="10.16" x2="10.16" y2="10.16" width="0.1524" layer="91"/>
+<wire x1="20.32" y1="10.16" x2="20.32" y2="20.32" width="0.1524" layer="91"/>
+<wire x1="20.32" y1="20.32" x2="25.4" y2="20.32" width="0.1524" layer="91"/>
+<wire x1="25.4" y1="20.32" x2="25.4" y2="33.02" width="0.1524" layer="91"/>
+<pinref part="LED5" gate="G$1" pin="C"/>
+<wire x1="25.4" y1="33.02" x2="27.94" y2="33.02" width="0.1524" layer="91"/>
+<wire x1="27.94" y1="33.02" x2="27.94" y2="35.56" width="0.1524" layer="91"/>
 </segment>
 </net>
 <net name="N$10" class="0">
 <segment>
-<pinref part="LED5" gate="G$1" pin="C"/>
-<wire x1="27.94" y1="35.56" x2="27.94" y2="7.62" width="0.1524" layer="91"/>
 <pinref part="U3" gate="U$1" pin="PC3(ADC3)"/>
 <wire x1="27.94" y1="7.62" x2="10.16" y2="7.62" width="0.1524" layer="91"/>
+<wire x1="27.94" y1="7.62" x2="27.94" y2="27.94" width="0.1524" layer="91"/>
+<pinref part="LED4" gate="G$1" pin="C"/>
+<wire x1="27.94" y1="27.94" x2="20.32" y2="27.94" width="0.1524" layer="91"/>
+<wire x1="20.32" y1="27.94" x2="20.32" y2="35.56" width="0.1524" layer="91"/>
 </segment>
 </net>
@@
 <pinref part="S1" gate="S" pin="2"/>
 <wire x1="10.16" y1="5.08" x2="30.48" y2="5.08" width="0.1524" layer="91"/>
-<pinref part="S1" gate="S" pin="1"/>
-<wire x1="30.48" y1="7.62" x2="30.48" y2="5.08" width="0.1524" layer="91"/>
-<junction x="30.48" y="5.08"/>
 </segment>
 </net>
@@
 <pinref part="U$7" gate="G$1" pin="P$2"/>
 <label x="86.36" y="58.42" size="1.778" layer="95"/>
-<pinref part="R13" gate="G$1" pin="2"/>
-<wire x1="104.14" y1="58.42" x2="76.2" y2="58.42" width="0.1524" layer="91"/>
-<wire x1="76.2" y1="58.42" x2="76.2" y2="50.8" width="0.1524" layer="91"/>
+<wire x1="104.14" y1="58.42" x2="63.5" y2="58.42" width="0.1524" layer="91"/>
+<pinref part="R12" gate="G$1" pin="2"/>
+<wire x1="58.42" y1="50.8" x2="63.5" y2="50.8" width="0.1524" layer="91"/>
+<wire x1="63.5" y1="50.8" x2="63.5" y2="58.42" width="0.1524" layer="91"/>
 </segment>
 </net>
@@
 <pinref part="U$7" gate="G$1" pin="P$3"/>
 <label x="86.36" y="60.96" size="1.778" layer="95"/>
-<pinref part="R12" gate="G$1" pin="2"/>
-<wire x1="58.42" y1="50.8" x2="58.42" y2="60.96" width="0.1524" layer="91"/>
 <wire x1="58.42" y1="60.96" x2="104.14" y2="60.96" width="0.1524" layer="91"/>
-</segment>
-</net>
+<wire x1="58.42" y1="60.96" x2="58.42" y2="55.88" width="0.1524" layer="91"/>
+<wire x1="58.42" y1="55.88" x2="76.2" y2="55.88" width="0.1524" layer="91"/>
+<pinref part="R13" gate="G$1" pin="2"/>
+<wire x1="76.2" y1="55.88" x2="76.2" y2="50.8" width="0.1524" layer="91"/>
+</segment>
+</net>

Commit message: fixed some T things/
Parts:
- added Q4: 16MHz, crystal:CRYSTALHC49UP
Connections:
- removed net +5V: C6.2, C7.2, R2.2, R5.2, R6.2, R7.1, U$3G$2.VDD, U2.VDD
- net N$5: now also Q4.2
- net N$6: now also Q4.1
- net VCC: now also C6.2, C7.2, R2.2, R5.2, R6.2, R7.1, U$3G$2.VDD, U2.VDD
Changed lines of the file:
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@@
 <?xml version="1.0" encoding="utf-8"?>
 <!DOCTYPE eagle SYSTEM "eagle.dtd">
-<eagle version="6.5.0">
+<eagle version="7.2.0">
 <drawing>
 <settings>
@@
 <part name="U$3" library="RobThePyro" deviceset="MCP2515" device="SO"/>
 <part name="U2" library="SparkFun" deviceset="MCP2551" device=""/>
-<part name="P+1" library="supply1" deviceset="+5V" device=""/>
 <part name="GND1" library="supply1" deviceset="GND" device=""/>
 <part name="GND2" library="supply1" deviceset="GND" device=""/>
-<part name="P+2" library="supply1" deviceset="+5V" device=""/>
 <part name="Q2" library="crystal" deviceset="CRYSTAL" device="HC49S" value="16MHz"/>
 <part name="Q3" library="crystal" deviceset="CRYSTAL" device="HC49UP" value="16MHz"/>
@@
 <part name="LED2" library="led" deviceset="LED" device="CHIP-LED0805" value="TX"/>
 <part name="LED3" library="led" deviceset="LED" device="CHIP-LED0805" value="INT"/>
-<part name="P+3" library="supply1" deviceset="+5V" device=""/>
 <part name="R7" library="resistor" deviceset="R-US_" device="R0805" value="100k"/>
-<part name="P+4" library="supply1" deviceset="+5V" device=""/>
 <part name="R8" library="resistor" deviceset="R-US_" device="R0805" value="100k"/>
 <part name="Z1" library="supressor" deviceset="TVS-UD-" device="SOD323"/>
@@
 <part name="R16" library="resistor" deviceset="R-US_" device="M0805" value="10K"/>
 <part name="D1" library="diode" deviceset="SCHOTTKY-DIODE" device="SMD"/>
+<part name="SUPPLY16" library="supply2" deviceset="VCC" device=""/>
+<part name="SUPPLY17" library="supply2" deviceset="VCC" device=""/>
+<part name="SUPPLY18" library="supply2" deviceset="VCC" device=""/>
+<part name="SUPPLY19" library="supply2" deviceset="VCC" device=""/>
+<part name="Q4" library="crystal" deviceset="CRYSTAL" device="HC49UP" value="16MHz"/>
 </parts>
 <sheets>
@@
 <instance part="R16" gate="G$1" x="-104.14" y="43.18" rot="R90"/>
 <instance part="D1" gate="G$1" x="-132.08" y="-22.86"/>
+<instance part="Q4" gate="G$1" x="-45.72" y="-12.7" rot="R90"/>
 </instances>
 <busses>
@@
 <pinref part="Q1" gate="G$1" pin="2"/>
 <pinref part="U3" gate="U$1" pin="PB6(XTAL1/TOSC1)"/>
-<wire x1="-50.8" y1="-7.62" x2="-38.1" y2="-7.62" width="0.1524" layer="91"/>
+<wire x1="-50.8" y1="-7.62" x2="-45.72" y2="-7.62" width="0.1524" layer="91"/>
+<wire x1="-45.72" y1="-7.62" x2="-38.1" y2="-7.62" width="0.1524" layer="91"/>
 <wire x1="-38.1" y1="-7.62" x2="-38.1" y2="-10.16" width="0.1524" layer="91"/>
 <pinref part="C3" gate="G$1" pin="2"/>
 <wire x1="-60.96" y1="-7.62" x2="-50.8" y2="-7.62" width="0.1524" layer="91"/>
 <junction x="-50.8" y="-7.62"/>
+<pinref part="Q4" gate="G$1" pin="2"/>
+<wire x1="-45.72" y1="-10.16" x2="-45.72" y2="-7.62" width="0.1524" layer="91"/>
+<junction x="-45.72" y="-7.62"/>
 </segment>
 </net>
@@
 <pinref part="Q1" gate="G$1" pin="1"/>
 <pinref part="U3" gate="U$1" pin="PB7(XTAL2/TOSC2)"/>
-<wire x1="-50.8" y1="-17.78" x2="-38.1" y2="-17.78" width="0.1524" layer="91"/>
+<wire x1="-50.8" y1="-17.78" x2="-45.72" y2="-17.78" width="0.1524" layer="91"/>
+<wire x1="-45.72" y1="-17.78" x2="-38.1" y2="-17.78" width="0.1524" layer="91"/>
 <wire x1="-38.1" y1="-17.78" x2="-38.1" y2="-15.24" width="0.1524" layer="91"/>
 <pinref part="C2" gate="G$1" pin="2"/>
 <wire x1="-60.96" y1="-17.78" x2="-50.8" y2="-17.78" width="0.1524" layer="91"/>
 <junction x="-50.8" y="-17.78"/>
+<pinref part="Q4" gate="G$1" pin="1"/>
+<wire x1="-45.72" y1="-17.78" x2="-45.72" y2="-15.24" width="0.1524" layer="91"/>
+<junction x="-45.72" y="-17.78"/>
 </segment>
 </net>
@@
 <instance part="U$3" gate="G$1" x="0" y="0"/>
 <instance part="U2" gate="G$1" x="71.12" y="0"/>
-<instance part="P+1" gate="1" x="-15.24" y="58.42"/>
 <instance part="GND1" gate="1" x="5.08" y="33.02"/>
 <instance part="GND2" gate="1" x="48.26" y="-2.54"/>
-<instance part="P+2" gate="1" x="55.88" y="10.16"/>
 <instance part="Q2" gate="G$1" x="-30.48" y="17.78" rot="R90"/>
 <instance part="Q3" gate="G$1" x="-25.4" y="17.78" rot="R90"/>
@@
 <instance part="LED2" gate="G$1" x="22.86" y="27.94"/>
 <instance part="LED3" gate="G$1" x="27.94" y="27.94"/>
-<instance part="P+3" gate="1" x="22.86" y="50.8"/>
 <instance part="R7" gate="G$1" x="-25.4" y="-12.7" rot="R90"/>
-<instance part="P+4" gate="1" x="-25.4" y="-25.4" rot="R180"/>
 <instance part="R8" gate="G$1" x="76.2" y="25.4" rot="R180"/>
 <instance part="Z1" gate="G$1" x="99.06" y="-12.7" rot="R90"/>
@@
 <instance part="X2" gate="-5" x="91.44" y="45.72" rot="R90"/>
 <instance part="X2" gate="-6" x="93.98" y="45.72" rot="R90"/>
+<instance part="SUPPLY16" gate="G$1" x="-15.24" y="58.42"/>
+<instance part="SUPPLY17" gate="G$1" x="22.86" y="50.8"/>
+<instance part="SUPPLY18" gate="G$1" x="55.88" y="10.16"/>
+<instance part="SUPPLY19" gate="G$1" x="-25.4" y="-25.4" rot="R180"/>
 </instances>
 <busses>
@@
 <wire x1="22.86" y1="22.86" x2="22.86" y2="5.08" width="0.1524" layer="91"/>
 <junction x="22.86" y="5.08"/>
-</segment>
-</net>
-<net name="+5V" class="0">
-<segment>
-<pinref part="U2" gate="G$1" pin="VDD"/>
-<pinref part="P+2" gate="1" pin="+5V"/>
-<wire x1="60.96" y1="2.54" x2="55.88" y2="2.54" width="0.1524" layer="91"/>
-<wire x1="55.88" y1="2.54" x2="55.88" y2="7.62" width="0.1524" layer="91"/>
-</segment>
-<segment>
-<pinref part="P+1" gate="1" pin="+5V"/>
-<wire x1="-15.24" y1="55.88" x2="-15.24" y2="50.8" width="0.1524" layer="91"/>
-<pinref part="U$3" gate="G$2" pin="VDD"/>
-<wire x1="-12.7" y1="50.8" x2="-15.24" y2="50.8" width="0.1524" layer="91"/>
-<wire x1="-15.24" y1="50.8" x2="-15.24" y2="45.72" width="0.1524" layer="91"/>
-<junction x="-15.24" y="50.8"/>
-<pinref part="C6" gate="G$1" pin="2"/>
-<wire x1="-15.24" y1="45.72" x2="-10.16" y2="45.72" width="0.1524" layer="91"/>
-<wire x1="-15.24" y1="45.72" x2="-15.24" y2="38.1" width="0.1524" layer="91"/>
-<junction x="-15.24" y="45.72"/>
-<pinref part="C7" gate="G$1" pin="2"/>
-<wire x1="-15.24" y1="38.1" x2="-10.16" y2="38.1" width="0.1524" layer="91"/>
-</segment>
-<segment>
-<pinref part="R2" gate="G$1" pin="2"/>
-<pinref part="R5" gate="G$1" pin="2"/>
-<wire x1="17.78" y1="43.18" x2="22.86" y2="43.18" width="0.1524" layer="91"/>
-<pinref part="R6" gate="G$1" pin="2"/>
-<wire x1="22.86" y1="43.18" x2="27.94" y2="43.18" width="0.1524" layer="91"/>
-<junction x="22.86" y="43.18"/>
-<pinref part="P+3" gate="1" pin="+5V"/>
-<wire x1="22.86" y1="43.18" x2="22.86" y2="48.26" width="0.1524" layer="91"/>
-</segment>
-<segment>
-<pinref part="R7" gate="G$1" pin="1"/>
-<pinref part="P+4" gate="1" pin="+5V"/>
-<wire x1="-25.4" y1="-17.78" x2="-25.4" y2="-22.86" width="0.1524" layer="91"/>
 </segment>
 </net>
@@
 </segment>
 </net>
+<net name="VCC" class="0">
+<segment>
+<wire x1="-15.24" y1="55.88" x2="-15.24" y2="50.8" width="0.1524" layer="91"/>
+<pinref part="U$3" gate="G$2" pin="VDD"/>
+<wire x1="-12.7" y1="50.8" x2="-15.24" y2="50.8" width="0.1524" layer="91"/>
+<wire x1="-15.24" y1="50.8" x2="-15.24" y2="45.72" width="0.1524" layer="91"/>
+<junction x="-15.24" y="50.8"/>
+<pinref part="C6" gate="G$1" pin="2"/>
+<wire x1="-15.24" y1="45.72" x2="-10.16" y2="45.72" width="0.1524" layer="91"/>
+<wire x1="-15.24" y1="45.72" x2="-15.24" y2="38.1" width="0.1524" layer="91"/>
+<junction x="-15.24" y="45.72"/>
+<pinref part="C7" gate="G$1" pin="2"/>
+<wire x1="-15.24" y1="38.1" x2="-10.16" y2="38.1" width="0.1524" layer="91"/>
+<pinref part="SUPPLY16" gate="G$1" pin="VCC"/>
+</segment>
+<segment>
+<pinref part="R2" gate="G$1" pin="2"/>
+<pinref part="R5" gate="G$1" pin="2"/>
+<wire x1="17.78" y1="43.18" x2="22.86" y2="43.18" width="0.1524" layer="91"/>
+<pinref part="R6" gate="G$1" pin="2"/>
+<wire x1="22.86" y1="43.18" x2="27.94" y2="43.18" width="0.1524" layer="91"/>
+<junction x="22.86" y="43.18"/>
+<wire x1="22.86" y1="43.18" x2="22.86" y2="48.26" width="0.1524" layer="91"/>
+<pinref part="SUPPLY17" gate="G$1" pin="VCC"/>
+</segment>
+<segment>
+<pinref part="U2" gate="G$1" pin="VDD"/>
+<wire x1="60.96" y1="2.54" x2="55.88" y2="2.54" width="0.1524" layer="91"/>
+<wire x1="55.88" y1="2.54" x2="55.88" y2="7.62" width="0.1524" layer="91"/>
+<pinref part="SUPPLY18" gate="G$1" pin="VCC"/>
+</segment>
+<segment>
+<pinref part="R7" gate="G$1" pin="1"/>
+<wire x1="-25.4" y1="-17.78" x2="-25.4" y2="-22.86" width="0.1524" layer="91"/>
+<pinref part="SUPPLY19" gate="G$1" pin="VCC"/>
+</segment>
+</net>
