File: Eagle Projects/Terayza/D3/Speed.sch (EAGLE design)
At the start: 52 parts, among them Q2 16MHz, Q3 16MHz, Q4 16MHz, U2 MCP2551, U3 ATMEGA328P_TQFP, X1 5566-6, X2 5566-6

Commit message: Terayzas PCBS etched...
Parts:
- added U$5, U$8, U$9: MMBZ5V6ALT1G, RobThePyro:MMBZ5V6ALT1G
Connections:
- net A0: now also U$9.A2
- net A1: now also U$9.A1
- net GND: now also U$5.C, U$8.C, U$9.C
- net HE1: now also U$5.A2
- net HE2: now also U$5.A1
- net VCC: now also U$8.A1, U$8.A2
Other:
- moved on the sheet: R4
Changed lines of the file:
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@@
 <part name="SUPPLY19" library="supply2" deviceset="VCC" device=""/>
 <part name="Q4" library="crystal" deviceset="CRYSTAL" device="HC49UP" value="16MHz"/>
+<part name="U$5" library="RobThePyro" deviceset="MMBZ5V6ALT1G" device=""/>
+<part name="U$8" library="RobThePyro" deviceset="MMBZ5V6ALT1G" device=""/>
+<part name="SUPPLY20" library="supply2" deviceset="VCC" device=""/>
+<part name="SUPPLY21" library="supply2" deviceset="GND" device=""/>
+<part name="U$9" library="RobThePyro" deviceset="MMBZ5V6ALT1G" device=""/>
 </parts>
 <sheets>
@@
 <instance part="R1" gate="G$1" x="-50.8" y="22.86" rot="R90"/>
 <instance part="R3" gate="G$1" x="116.84" y="2.54"/>
-<instance part="R4" gate="G$1" x="116.84" y="-12.7"/>
+<instance part="R4" gate="G$1" x="116.84" y="-10.16"/>
 <instance part="SUPPLY2" gate="GND" x="-71.12" y="-30.48"/>
 <instance part="SUPPLY4" gate="GND" x="129.54" y="-22.86"/>
@@
 <instance part="D1" gate="G$1" x="-132.08" y="-22.86"/>
 <instance part="Q4" gate="G$1" x="-45.72" y="-12.7" rot="R90"/>
+<instance part="U$5" gate="G$1" x="78.74" y="-20.32"/>
+<instance part="U$8" gate="G$1" x="-43.18" y="48.26"/>
+<instance part="SUPPLY20" gate="G$1" x="-38.1" y="60.96"/>
+<instance part="SUPPLY21" gate="GND" x="-38.1" y="33.02"/>
+<instance part="U$9" gate="G$1" x="43.18" y="27.94"/>
 </instances>
 <busses>
@@
 <wire x1="129.54" y1="-15.24" x2="139.7" y2="-15.24" width="0.1524" layer="91"/>
 <pinref part="SUPPLY4" gate="GND" pin="GND"/>
-<wire x1="129.54" y1="-20.32" x2="129.54" y2="-15.24" width="0.1524" layer="91"/>
 <junction x="129.54" y="-15.24"/>
 <pinref part="U$1" gate="G$1" pin="P$1"/>
 <pinref part="U$2" gate="G$1" pin="P$1"/>
+<wire x1="129.54" y1="-20.32" x2="129.54" y2="-17.78" width="0.1524" layer="91"/>
+<pinref part="U$5" gate="G$1" pin="C"/>
+<wire x1="129.54" y1="-17.78" x2="129.54" y2="-15.24" width="0.1524" layer="91"/>
+<wire x1="83.82" y1="-27.94" x2="121.92" y2="-27.94" width="0.1524" layer="91"/>
+<wire x1="121.92" y1="-27.94" x2="121.92" y2="-17.78" width="0.1524" layer="91"/>
+<wire x1="121.92" y1="-17.78" x2="129.54" y2="-17.78" width="0.1524" layer="91"/>
+<junction x="129.54" y="-17.78"/>
 </segment>
 <segment>
@@
 <pinref part="SUPPLY15" gate="GND" pin="GND"/>
 <wire x1="76.2" y1="27.94" x2="66.04" y2="27.94" width="0.1524" layer="91"/>
-<wire x1="66.04" y1="27.94" x2="66.04" y2="22.86" width="0.1524" layer="91"/>
+<wire x1="66.04" y1="27.94" x2="66.04" y2="25.4" width="0.1524" layer="91"/>
 <pinref part="R14" gate="G$1" pin="1"/>
+<wire x1="66.04" y1="25.4" x2="66.04" y2="22.86" width="0.1524" layer="91"/>
 <wire x1="58.42" y1="27.94" x2="66.04" y2="27.94" width="0.1524" layer="91"/>
 <junction x="66.04" y="27.94"/>
+<pinref part="U$9" gate="G$1" pin="C"/>
+<wire x1="48.26" y1="20.32" x2="60.96" y2="20.32" width="0.1524" layer="91"/>
+<wire x1="60.96" y1="20.32" x2="60.96" y2="25.4" width="0.1524" layer="91"/>
+<wire x1="60.96" y1="25.4" x2="66.04" y2="25.4" width="0.1524" layer="91"/>
+<junction x="66.04" y="25.4"/>
 </segment>
 <segment>
@@
 <pinref part="S1" gate="S" pin="3"/>
 <wire x1="40.64" y1="7.62" x2="40.64" y2="5.08" width="0.1524" layer="91"/>
+</segment>
+<segment>
+<pinref part="SUPPLY21" gate="GND" pin="GND"/>
+<pinref part="U$8" gate="G$1" pin="C"/>
+<wire x1="-38.1" y1="35.56" x2="-38.1" y2="40.64" width="0.1524" layer="91"/>
 </segment>
 </net>
@@
 <wire x1="-124.46" y1="-22.86" x2="-124.46" y2="-20.32" width="0.1524" layer="91"/>
 </segment>
+<segment>
+<pinref part="U$8" gate="G$1" pin="A1"/>
+<pinref part="SUPPLY20" gate="G$1" pin="VCC"/>
+<wire x1="-35.56" y1="55.88" x2="-38.1" y2="55.88" width="0.1524" layer="91"/>
+<wire x1="-38.1" y1="55.88" x2="-38.1" y2="58.42" width="0.1524" layer="91"/>
+<pinref part="U$8" gate="G$1" pin="A2"/>
+<wire x1="-40.64" y1="55.88" x2="-38.1" y2="55.88" width="0.1524" layer="91"/>
+<junction x="-38.1" y="55.88"/>
+</segment>
 </net>
 <net name="PD2" class="0">
@@
 <net name="PD3" class="0">
 <segment>
-<wire x1="121.92" y1="-12.7" x2="139.7" y2="-12.7" width="0.1524" layer="91"/>
+<wire x1="121.92" y1="-10.16" x2="139.7" y2="-12.7" width="0.1524" layer="91"/>
 <pinref part="R4" gate="G$1" pin="2"/>
 <pinref part="U$2" gate="G$1" pin="P$2"/>
@@
 </segment>
 <segment>
-<wire x1="106.68" y1="2.54" x2="111.76" y2="2.54" width="0.1524" layer="91"/>
 <pinref part="R3" gate="G$1" pin="1"/>
 <label x="101.6" y="2.54" size="1.778" layer="95"/>
+<pinref part="U$5" gate="G$1" pin="A2"/>
+<wire x1="111.76" y1="2.54" x2="81.28" y2="2.54" width="0.1524" layer="91"/>
+<wire x1="81.28" y1="2.54" x2="81.28" y2="-12.7" width="0.1524" layer="91"/>
 </segment>
 </net>
@@
 </segment>
 <segment>
-<wire x1="106.68" y1="-12.7" x2="111.76" y2="-12.7" width="0.1524" layer="91"/>
 <pinref part="R4" gate="G$1" pin="1"/>
 <label x="101.6" y="-12.7" size="1.778" layer="95"/>
+<pinref part="U$5" gate="G$1" pin="A1"/>
+<wire x1="111.76" y1="-10.16" x2="86.36" y2="-10.16" width="0.1524" layer="91"/>
+<wire x1="86.36" y1="-10.16" x2="86.36" y2="-12.7" width="0.1524" layer="91"/>
 </segment>
 </net>
@@
 <pinref part="R14" gate="G$1" pin="2"/>
 <wire x1="58.42" y1="40.64" x2="58.42" y2="38.1" width="0.1524" layer="91"/>
-<wire x1="58.42" y1="40.64" x2="53.34" y2="40.64" width="0.1524" layer="91"/>
 <junction x="58.42" y="40.64"/>
 <label x="48.26" y="40.64" size="1.778" layer="95"/>
+<pinref part="U$9" gate="G$1" pin="A2"/>
+<wire x1="58.42" y1="40.64" x2="45.72" y2="40.64" width="0.1524" layer="91"/>
+<wire x1="45.72" y1="40.64" x2="45.72" y2="35.56" width="0.1524" layer="91"/>
 </segment>
 <segment>
@@
 <pinref part="R15" gate="G$1" pin="2"/>
 <wire x1="76.2" y1="40.64" x2="76.2" y2="38.1" width="0.1524" layer="91"/>
-<wire x1="76.2" y1="40.64" x2="71.12" y2="40.64" width="0.1524" layer="91"/>
+<wire x1="76.2" y1="40.64" x2="68.58" y2="40.64" width="0.1524" layer="91"/>
 <junction x="76.2" y="40.64"/>
 <label x="66.04" y="40.64" size="1.778" layer="95"/>
-</segment>
-<segment>
+<wire x1="68.58" y1="40.64" x2="68.58" y2="38.1" width="0.1524" layer="91"/>
+<pinref part="U$9" gate="G$1" pin="A1"/>
+<wire x1="68.58" y1="38.1" x2="50.8" y2="38.1" width="0.1524" layer="91"/>
+<wire x1="50.8" y1="38.1" x2="50.8" y2="35.56" width="0.1524" layer="91"/>
+</segment>
+<segment>

Commit message: Working
Parts:
- added U$10: HEADER-5WAY, con-TE-EP:HEADER-5WAY
Connections:
- removed net N$11: S1.2, U3.PC4(ADC4/SDA)
- new net INT: U$10.P$1
- new net SCL: U$10.P$3, U3.PC5(ADC5/SCL)
- new net SDA: U$10.P$2, U3.PC4(ADC4/SDA)
- net GND: now also U$10.P$4, U3.ADC6
- net VCC: now also U$10.P$5
Other:
- note added: "Add protection to the inputs"
- note added: "Connect int still Look at datasheet for pin"
- note added: "Ensure button can go on pin19"
- note added: "MPU6050 Header"
- moved on the sheet: F1, R3, R4, U$1, U$2, U$4, U$5

Commit message: Thingies
Connections:
- new net N$11: U3.PB0(ICP)
Changed lines of the file:
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@@
+</segment>
+</net>
+<net name="N$11" class="0">
+<segment>
+<pinref part="U3" gate="U$1" pin="PB0(ICP)"/>
+<wire x1="10.16" y1="-30.48" x2="15.24" y2="-30.48" width="0.1524" layer="91"/>
 </segment>
 </net>
