File: Eagle Projects/Terayza/D3/Speed.sch (EAGLE design)
At the start: 56 parts, among them Q2 16MHz, Q3 16MHz, Q4 16MHz, U2 MCP2551, U3 ATMEGA328P_TQFP, X1 5566-6, X2 5566-6

Commit message: Board things
Parts:
- added U$11, U$12: MMBZ5V6ALT1G, RobThePyro:MMBZ5V6ALT1G
- added U$13: HEADER-3WAY, con-TE-EP:HEADER-3WAY
Connections:
- new net RXD: U$13.P$3, U3.PD0(RXD)
- new net TXD: U$13.P$2, U3.PD1(TXD)
- net GND: now also U$11.C, U$12.C, U$13.P$1; no longer S1.1, U3.ADC6
- net INT: now also U$12.A1, U3.PD5(T1)
- net MTSPD: now also U3.PB0(ICP); no longer U3.PD0(RXD)
- net N$11: now also S1.1, S1.2, U3.PD4(XCK/T0); no longer U3.PB0(ICP)
- net SCL: now also U$10.P$2, U$11.A1; no longer U$10.P$3
- net SDA: now also U$10.P$3, U$11.A2; no longer U$10.P$2
Other:
- note removed: "Add protection to the inputs"
- note removed: "Connect int still Look at datasheet for pin"
- note removed: "Ensure button can go on pin19"
- moved on the sheet: S1, U$10

Commit message: Hack internet job using weakest internet in the world
Parts:
- removed C8: (no value), resistor:C-EUC0805
- R16: value 10K -> 1K
Connections:
- net GND: no longer C8.1
- net MTSPD: no longer C8.2
Changed lines of the file:
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@@
 <part name="SUPPLY10" library="supply2" deviceset="GND" device=""/>
 <part name="SUPPLY11" library="supply2" deviceset="VCC" device=""/>
-<part name="C8" library="resistor" deviceset="C-EU" device="C0805"/>
 <part name="U$6" library="con-TE-EP" deviceset="HEADER-2WAY" device=""/>
 <part name="R9" library="resistor" deviceset="R-US_" device="M0805" value="680E"/>
@@
 <part name="SUPPLY15" library="supply2" deviceset="GND" device=""/>
 <part name="OK1" library="optocoupler" deviceset="LTV816" device=""/>
-<part name="R16" library="resistor" deviceset="R-US_" device="M0805" value="10K"/>
+<part name="R16" library="resistor" deviceset="R-US_" device="M0805" value="1K"/>
 <part name="D1" library="diode" deviceset="SCHOTTKY-DIODE" device="SMD"/>
 <part name="SUPPLY16" library="supply2" deviceset="VCC" device=""/>
@@
 <instance part="SUPPLY10" gate="GND" x="-104.14" y="17.78"/>
 <instance part="SUPPLY11" gate="G$1" x="-96.52" y="50.8"/>
-<instance part="C8" gate="G$1" x="-96.52" y="25.4" rot="R180"/>
 <instance part="U$6" gate="G$1" x="-144.78" y="30.48" rot="R180"/>
 <instance part="R9" gate="G$1" x="-129.54" y="33.02"/>
@@
 <segment>
 <pinref part="SUPPLY10" gate="GND" pin="GND"/>
-<wire x1="-104.14" y1="20.32" x2="-104.14" y2="22.86" width="0.1524" layer="91"/>
-<pinref part="C8" gate="G$1" pin="1"/>
-<wire x1="-104.14" y1="22.86" x2="-96.52" y2="22.86" width="0.1524" layer="91"/>
 <pinref part="OK1" gate="G$1" pin="EMIT"/>
-<wire x1="-104.14" y1="22.86" x2="-104.14" y2="27.94" width="0.1524" layer="91"/>
-<junction x="-104.14" y="22.86"/>
+<wire x1="-104.14" y1="20.32" x2="-104.14" y2="27.94" width="0.1524" layer="91"/>
 </segment>
 <segment>
@@
 <wire x1="-104.14" y1="38.1" x2="-104.14" y2="35.56" width="0.1524" layer="91"/>
 <wire x1="-104.14" y1="35.56" x2="-104.14" y2="33.02" width="0.1524" layer="91"/>
-<wire x1="-104.14" y1="35.56" x2="-96.52" y2="35.56" width="0.1524" layer="91"/>
+<wire x1="-104.14" y1="35.56" x2="-93.98" y2="35.56" width="0.1524" layer="91"/>
 <junction x="-104.14" y="35.56"/>
-<pinref part="C8" gate="G$1" pin="2"/>
-<wire x1="-96.52" y1="35.56" x2="-93.98" y2="35.56" width="0.1524" layer="91"/>
-<wire x1="-96.52" y1="30.48" x2="-96.52" y2="35.56" width="0.1524" layer="91"/>
-<junction x="-96.52" y="35.56"/>
 <label x="-93.98" y="38.1" size="1.778" layer="95"/>
 </segment>
